Commit message: added: yaml rosparam loading

File: eTaSL/moveit_plan_compact/test_assets/custom_robots.urdf (robot description, URDF)
Before this commit: robot custom_robots, 21 links, 20 joints
Links:
- link panda1_hand: geometry collision cylinder length=0.05 radius=0.01; collision cylinder length=0.055 radius=0.02
- link panda1_link6: geometry collision cylinder length=0.08 radius=0.04; collision cylinder length=0.09 radius=0.065
Joints:
- removed joint indy0_joint_base
- removed joint panda1_joint_base
- added joint indy0_joint_base_link: type fixed, parent base_link, child indy0_link0, origin xyz=-0.446480512619 0.251528263092 0.00979518890381 rpy=7.72251143907e-05 0.012837732858 -1.58433052921
- added joint panda1_joint_base_link: type fixed, parent base_link, child panda1_link0, origin xyz=0.511702060699 0.168303191662 0.014661192894 rpy=0.00371903837049 0.0130669918716 -1.60510658312

File: eTaSL/robots/custom_robots.urdf (robot description, URDF)
Before this commit: robot custom_robots, 21 links, 20 joints
Joints:
- joint indy0_joint_base_link: origin xyz=-0.446480512619 0.251528263092 0.00979518890381 rpy=7.72251143907e-05 0.012837732858 -1.58433052921 -> xyz=1.48274451419 0.452685329639 0.188611320622 rpy=0.0 0.0 0.340886585646
- joint panda1_joint_base_link: origin xyz=0.511702060699 0.168303191662 0.014661192894 rpy=0.00371903837049 0.0130669918716 -1.60510658312 -> xyz=0.5035655925 1.68277256243 0.325530553938 rpy=0.0 0.0 1.33622974449

File: eTaSL/robots/custom_robots.urdf.xacro (robot description, xacro)
@@ -6,6 +6,6 @@
 <link name="base_link"/>
 <!-- BODY BEGIN -->
-<xacro:indy7_robot robot_id="0" xyz="-0.446480512619 0.251528263092 0.00979518890381" rpy="7.72251143907e-05 0.012837732858 -1.58433052921" connected_to="base_link"/>
-<xacro:panda_robot robot_id="1" xyz="0.511702060699 0.168303191662 0.014661192894" rpy="0.00371903837049 0.0130669918716 -1.60510658312" connected_to="base_link"/>
+<xacro:indy7_robot robot_id="0" xyz="1.48274451419 0.452685329639 0.188611320622" rpy="0 0 0.340886585646" connected_to="base_link"/>
+<xacro:panda_robot robot_id="1" xyz="0.5035655925 1.68277256243 0.325530553938" rpy="0 0 1.33622974449" connected_to="base_link"/>
 <!-- BODY END -->
 </robot>
