Commit message: custom robot setting - indy7

File: eTaSL/robots/custom_robots.urdf (robot description, URDF)
Before this commit: robot panda, 25 links, 24 joints
Links:
- removed link panda0_hand
- removed link panda0_leftfinger
- removed link panda0_link0
- removed link panda0_link1
- removed link panda0_link2
- removed link panda0_link3
- removed link panda0_link4
- removed link panda0_link5
- removed link panda0_link6
- removed link panda0_link7
- removed link panda0_link8
- removed link panda0_rightfinger
- removed link panda1_hand
- removed link panda1_leftfinger
- removed link panda1_link0
- removed link panda1_link1
- removed link panda1_link2
- removed link panda1_link3
- removed link panda1_link4
- removed link panda1_link5
- removed link panda1_link6
- removed link panda1_link7
- removed link panda1_link8
- removed link panda1_rightfinger
- added link indy0_link0, mass 1.59306955; collision cylinder length=0.075 radius=0.102; visual mesh filename=package://indy7_description/meshes/stl/Indy7_0.stl
- added link indy0_link1, mass 11.8030102; collision cylinder length=0.109 radius=0.075; collision cylinder length=0.222 radius=0.075
- added link indy0_link2, mass 7.99292141; collision cylinder length=0.09 radius=0.075; collision cylinder length=0.1205 radius=0.045
- added link indy0_link3, mass 2.99134127; collision cylinder length=0.075 radius=0.045; collision cylinder length=0.267 radius=0.045
- added link indy0_link4, mass 2.12317035; collision cylinder length=0.083 radius=0.045; collision cylinder length=0.114 radius=0.045
- added link indy0_link5, mass 2.28865091; collision cylinder length=0.069 radius=0.045; collision cylinder length=0.168 radius=0.045
- added link indy0_link6, mass 0.40083918; collision cylinder length=0.06 radius=0.045; visual mesh filename=package://indy7_description/meshes/stl/Indy7_6.stl
- added link indy0_tcp
- added link indy1_link0, mass 1.59306955; collision cylinder length=0.075 radius=0.102; visual mesh filename=package://indy7_description/meshes/stl/Indy7_0.stl
- added link indy1_link1, mass 11.8030102; collision cylinder length=0.109 radius=0.075; collision cylinder length=0.222 radius=0.075
- added link indy1_link2, mass 7.99292141; collision cylinder length=0.09 radius=0.075; collision cylinder length=0.1205 radius=0.045
- added link indy1_link3, mass 2.99134127; collision cylinder length=0.075 radius=0.045; collision cylinder length=0.267 radius=0.045
- added link indy1_link4, mass 2.12317035; collision cylinder length=0.083 radius=0.045; collision cylinder length=0.114 radius=0.045
- added link indy1_link5, mass 2.28865091; collision cylinder length=0.069 radius=0.045; collision cylinder length=0.168 radius=0.045
- added link indy1_link6, mass 0.40083918; collision cylinder length=0.06 radius=0.045; visual mesh filename=package://indy7_description/meshes/stl/Indy7_6.stl
- added link indy1_tcp
Joints:
- removed joint panda0_finger_joint1
- removed joint panda0_finger_joint2
- removed joint panda0_hand_joint
- removed joint panda0_joint1
- removed joint panda0_joint2
- removed joint panda0_joint3
- removed joint panda0_joint4
- removed joint panda0_joint5
- removed joint panda0_joint6
- removed joint panda0_joint7
- removed joint panda0_joint8
- removed joint panda0_joint_world
- removed joint panda1_finger_joint1
- removed joint panda1_finger_joint2
- removed joint panda1_hand_joint
- removed joint panda1_joint1
- removed joint panda1_joint2
- removed joint panda1_joint3
- removed joint panda1_joint4
- removed joint panda1_joint5
- removed joint panda1_joint6
- removed joint panda1_joint7
- removed joint panda1_joint8
- removed joint panda1_joint_world
- added joint indy0_joint0: type revolute, parent indy0_link0, child indy0_link1, origin xyz=0 0 0.0775 rpy=0 0 0, axis 0 0 1, limit lower=-3.05432619099 upper=3.05432619099 effort=10 velocity=1
- added joint indy0_joint1: type revolute, parent indy0_link1, child indy0_link2, origin xyz=0 -0.10900000 0.22200000 rpy=1.57079632679 1.57079632679 0, axis 0 0 1, limit lower=-3.05432619099 upper=3.05432619099 effort=10 velocity=1
- added joint indy0_joint2: type revolute, parent indy0_link2, child indy0_link3, origin xyz=-0.45000000 +0.00000000 -0.03050000 rpy=0 0 0, axis 0 0 1, limit lower=-3.05432619099 upper=3.05432619099 effort=10 velocity=1
- added joint indy0_joint3: type revolute, parent indy0_link3, child indy0_link4, origin xyz=-0.26700000 +0.00000000 -0.07500000 rpy=-1.57079632679 0 1.57079632679, axis 0 0 1, limit lower=-3.05432619099 upper=3.05432619099 effort=10 velocity=1
- added joint indy0_joint4: type revolute, parent indy0_link4, child indy0_link5, origin xyz=+0.00000000 -0.11400000 +0.08300000 rpy=1.57079632679 1.57079632679 0, axis 0 0 1, limit lower=-3.05432619099 upper=3.05432619099 effort=10 velocity=1
- added joint indy0_joint5: type revolute, parent indy0_link5, child indy0_link6, origin xyz=-0.16800000 +0.00000000 +0.06900000 rpy=-1.57079632679 0 1.57079632679, axis 0 0 1, limit lower=-3.75245789179 upper=3.75245789179 effort=10 velocity=1
- added joint indy0_joint_world: type fixed, parent world, child indy0_link0, origin xyz=0 0.5 0 rpy=0 0 0
- added joint indy0_tcp: type fixed, parent indy0_link6, child indy0_tcp, origin xyz=0 0 0.06 rpy=0 0 0
- added joint indy1_joint0: type revolute, parent indy1_link0, child indy1_link1, origin xyz=0 0 0.0775 rpy=0 0 0, axis 0 0 1, limit lower=-3.05432619099 upper=3.05432619099 effort=10 velocity=1
- added joint indy1_joint1: type revolute, parent indy1_link1, child indy1_link2, origin xyz=0 -0.10900000 0.22200000 rpy=1.57079632679 1.57079632679 0, axis 0 0 1, limit lower=-3.05432619099 upper=3.05432619099 effort=10 velocity=1
- added joint indy1_joint2: type revolute, parent indy1_link2, child indy1_link3, origin xyz=-0.45000000 +0.00000000 -0.03050000 rpy=0 0 0, axis 0 0 1, limit lower=-3.05432619099 upper=3.05432619099 effort=10 velocity=1
- added joint indy1_joint3: type revolute, parent indy1_link3, child indy1_link4, origin xyz=-0.26700000 +0.00000000 -0.07500000 rpy=-1.57079632679 0 1.57079632679, axis 0 0 1, limit lower=-3.05432619099 upper=3.05432619099 effort=10 velocity=1
- added joint indy1_joint4: type revolute, parent indy1_link4, child indy1_link5, origin xyz=+0.00000000 -0.11400000 +0.08300000 rpy=1.57079632679 1.57079632679 0, axis 0 0 1, limit lower=-3.05432619099 upper=3.05432619099 effort=10 velocity=1
- added joint indy1_joint5: type revolute, parent indy1_link5, child indy1_link6, origin xyz=-0.16800000 +0.00000000 +0.06900000 rpy=-1.57079632679 0 1.57079632679, axis 0 0 1, limit lower=-3.75245789179 upper=3.75245789179 effort=10 velocity=1
- added joint indy1_joint_world: type fixed, parent world, child indy1_link0, origin xyz=0 -0.5 0 rpy=0 0 0
- added joint indy1_tcp: type fixed, parent indy1_link6, child indy1_tcp, origin xyz=0 0 0.06 rpy=0 0 0

File: eTaSL/robots/custom_robots.urdf.xacro (robot description, xacro)
@@ -1,7 +1,9 @@
 <?xml version="1.0" encoding="utf-8"?>
-<robot xmlns:xacro="http://www.ros.org/wiki/xacro" name="panda">
+<robot xmlns:xacro="http://www.ros.org/wiki/xacro" name="custom_robots">
+  <xacro:include filename="$(find indy7_description)/urdf/materials.xacro"/>
   <xacro:include filename="$(env TF_GMT_ETASL_DIR)/robots/panda_robot.xacro"/>
+  <xacro:include filename="$(env TF_GMT_ETASL_DIR)/robots/indy7_robot.xacro"/>
   <link name="world"/>
-  <xacro:panda_robot robot_id="0" xyz="0 0.5 0" connected_to="world"/>
-  <xacro:panda_robot robot_id="1" xyz="0 -0.5 0" connected_to="world"/>
+  <xacro:indy7_robot robot_id="0" xyz="0 0.5 0" connected_to="world"/>
+  <xacro:indy7_robot robot_id="1" xyz="0 -0.5 0" connected_to="world"/>
 </robot>

Commit message: custom robot urdf loading done

File: eTaSL/robots/custom_robots.urdf (robot description, URDF)
Before this commit: robot custom_robots, 17 links, 16 joints
Links:
- removed link indy0_link0
- removed link indy0_link1
- removed link indy0_link2
- removed link indy0_link3
- removed link indy0_link4
- removed link indy0_link5
- removed link indy0_link6
- removed link indy0_tcp
- added link panda0_hand; collision mesh filename=package://franka_description/meshes/collision/hand.stl; visual mesh filename=package://franka_description/meshes/visual/hand.dae
- added link panda0_leftfinger; collision mesh filename=package://franka_description/meshes/collision/finger.stl; visual mesh filename=package://franka_description/meshes/visual/finger.dae
- added link panda0_link0; collision mesh filename=package://franka_description/meshes/collision/link0.stl; visual mesh filename=package://franka_description/meshes/visual/link0.dae
- added link panda0_link1; collision mesh filename=package://franka_description/meshes/collision/link1.stl; visual mesh filename=package://franka_description/meshes/visual/link1.dae
- added link panda0_link2; collision mesh filename=package://franka_description/meshes/collision/link2.stl; visual mesh filename=package://franka_description/meshes/visual/link2.dae
- added link panda0_link3; collision mesh filename=package://franka_description/meshes/collision/link3.stl; visual mesh filename=package://franka_description/meshes/visual/link3.dae
- added link panda0_link4; collision mesh filename=package://franka_description/meshes/collision/link4.stl; visual mesh filename=package://franka_description/meshes/visual/link4.dae
- added link panda0_link5; collision mesh filename=package://franka_description/meshes/collision/link5.stl; visual mesh filename=package://franka_description/meshes/visual/link5.dae
- added link panda0_link6; collision mesh filename=package://franka_description/meshes/collision/link6.stl; visual mesh filename=package://franka_description/meshes/visual/link6.dae
- added link panda0_link7; collision mesh filename=package://franka_description/meshes/collision/link7.stl; visual mesh filename=package://franka_description/meshes/visual/link7.dae
- added link panda0_link8
- added link panda0_rightfinger; collision mesh filename=package://franka_description/meshes/collision/finger.stl; visual mesh filename=package://franka_description/meshes/visual/finger.dae
Joints:
- removed joint indy0_joint0
- removed joint indy0_joint1
- removed joint indy0_joint2
- removed joint indy0_joint3
- removed joint indy0_joint4
- removed joint indy0_joint5
- removed joint indy0_joint_world
- removed joint indy0_tcp
- added joint panda0_finger_joint1: type prismatic, parent panda0_hand, child panda0_leftfinger, origin xyz=0 0 0.0584 rpy=0 0 0, axis 0 1 0, limit lower=0.0 upper=0.04 effort=20 velocity=0.2
- added joint panda0_finger_joint2: type prismatic, parent panda0_hand, child panda0_rightfinger, origin xyz=0 0 0.0584 rpy=0 0 0, axis 0 -1 0, limit lower=0.0 upper=0.04 effort=20 velocity=0.2, mimic joint=panda0_finger_joint1
- added joint panda0_hand_joint: type fixed, parent panda0_link8, child panda0_hand, origin xyz=0 0 0 rpy=0 0 -0.785398163397
- added joint panda0_joint1: type revolute, parent panda0_link0, child panda0_link1, origin xyz=0 0 0.333 rpy=0 0 0, axis 0 0 1, limit lower=-2.8973 upper=2.8973 effort=87 velocity=2.1750
- added joint panda0_joint2: type revolute, parent panda0_link1, child panda0_link2, origin xyz=0 0 0 rpy=-1.57079632679 0 0, axis 0 0 1, limit lower=-1.7628 upper=1.7628 effort=87 velocity=2.1750
- added joint panda0_joint3: type revolute, parent panda0_link2, child panda0_link3, origin xyz=0 -0.316 0 rpy=1.57079632679 0 0, axis 0 0 1, limit lower=-2.8973 upper=2.8973 effort=87 velocity=2.1750
- added joint panda0_joint4: type revolute, parent panda0_link3, child panda0_link4, origin xyz=0.0825 0 0 rpy=1.57079632679 0 0, axis 0 0 1, limit lower=-3.0718 upper=-0.0698 effort=87 velocity=2.1750
- added joint panda0_joint5: type revolute, parent panda0_link4, child panda0_link5, origin xyz=-0.0825 0.384 0 rpy=-1.57079632679 0 0, axis 0 0 1, limit lower=-2.8973 upper=2.8973 effort=12 velocity=2.6100
- added joint panda0_joint6: type revolute, parent panda0_link5, child panda0_link6, origin xyz=0 0 0 rpy=1.57079632679 0 0, axis 0 0 1, limit lower=-0.0175 upper=3.7525 effort=12 velocity=2.6100
- added joint panda0_joint7: type revolute, parent panda0_link6, child panda0_link7, origin xyz=0.088 0 0 rpy=1.57079632679 0 0, axis 0 0 1, limit lower=-2.8973 upper=2.8973 effort=12 velocity=2.6100
- added joint panda0_joint8: type fixed, parent panda0_link7, child panda0_link8, origin xyz=0 0 0.107 rpy=0 0 0, axis 0 0 0
- added joint panda0_joint_world: type fixed, parent world, child panda0_link0, origin xyz=0 0.5 0 rpy=0 0 0

File: eTaSL/robots/custom_robots.urdf.xacro (robot description, xacro)
@@ -5,5 +5,5 @@
   <xacro:include filename="$(env TF_GMT_ETASL_DIR)/robots/indy7_robot.xacro"/>
   <link name="world"/>
-  <xacro:indy7_robot robot_id="0" xyz="0 0.5 0" connected_to="world"/>
+  <xacro:panda_robot robot_id="0" xyz="0 0.5 0" connected_to="world"/>
   <xacro:indy7_robot robot_id="1" xyz="0 -0.5 0" connected_to="world"/>
 </robot>

Commit message: xacro auto generation, rviz autostart, graph running tested

File: eTaSL/robots/custom_robots.urdf (robot description, URDF)
Before this commit: robot custom_robots, 21 links, 20 joints
Links:
- removed link indy1_link0
- removed link indy1_link1
- removed link indy1_link2
- removed link indy1_link3
- removed link indy1_link4
- removed link indy1_link5
- removed link indy1_link6
- removed link indy1_tcp
- removed link panda0_hand
- removed link panda0_leftfinger
- removed link panda0_link0
- removed link panda0_link1
- removed link panda0_link2
- removed link panda0_link3
- removed link panda0_link4
- removed link panda0_link5
- removed link panda0_link6
- removed link panda0_link7
- removed link panda0_link8
- removed link panda0_rightfinger
- added link indy0_link0, mass 1.59306955; collision cylinder length=0.075 radius=0.102; visual mesh filename=package://indy7_description/meshes/stl/Indy7_0.stl
- added link indy0_link1, mass 11.8030102; collision cylinder length=0.109 radius=0.075; collision cylinder length=0.222 radius=0.075
- added link indy0_link2, mass 7.99292141; collision cylinder length=0.09 radius=0.075; collision cylinder length=0.1205 radius=0.045
- added link indy0_link3, mass 2.99134127; collision cylinder length=0.075 radius=0.045; collision cylinder length=0.267 radius=0.045
- added link indy0_link4, mass 2.12317035; collision cylinder length=0.083 radius=0.045; collision cylinder length=0.114 radius=0.045
- added link indy0_link5, mass 2.28865091; collision cylinder length=0.069 radius=0.045; collision cylinder length=0.168 radius=0.045
- added link indy0_link6, mass 0.40083918; collision cylinder length=0.06 radius=0.045; visual mesh filename=package://indy7_description/meshes/stl/Indy7_6.stl
- added link indy0_tcp
- added link panda1_hand; collision mesh filename=package://franka_description/meshes/collision/hand.stl; visual mesh filename=package://franka_description/meshes/visual/hand.dae
- added link panda1_leftfinger; collision mesh filename=package://franka_description/meshes/collision/finger.stl; visual mesh filename=package://franka_description/meshes/visual/finger.dae
- added link panda1_link0; collision mesh filename=package://franka_description/meshes/collision/link0.stl; visual mesh filename=package://franka_description/meshes/visual/link0.dae
- added link panda1_link1; collision mesh filename=package://franka_description/meshes/collision/link1.stl; visual mesh filename=package://franka_description/meshes/visual/link1.dae
- added link panda1_link2; collision mesh filename=package://franka_description/meshes/collision/link2.stl; visual mesh filename=package://franka_description/meshes/visual/link2.dae
- added link panda1_link3; collision mesh filename=package://franka_description/meshes/collision/link3.stl; visual mesh filename=package://franka_description/meshes/visual/link3.dae
- added link panda1_link4; collision mesh filename=package://franka_description/meshes/collision/link4.stl; visual mesh filename=package://franka_description/meshes/visual/link4.dae
- added link panda1_link5; collision mesh filename=package://franka_description/meshes/collision/link5.stl; visual mesh filename=package://franka_description/meshes/visual/link5.dae
- added link panda1_link6; collision mesh filename=package://franka_description/meshes/collision/link6.stl; visual mesh filename=package://franka_description/meshes/visual/link6.dae
- added link panda1_link7; collision mesh filename=package://franka_description/meshes/collision/link7.stl; visual mesh filename=package://franka_description/meshes/visual/link7.dae
- added link panda1_link8
- added link panda1_rightfinger; collision mesh filename=package://franka_description/meshes/collision/finger.stl; visual mesh filename=package://franka_description/meshes/visual/finger.dae
Joints:
- removed joint indy1_joint0
- removed joint indy1_joint1
- removed joint indy1_joint2
- removed joint indy1_joint3
- removed joint indy1_joint4
- removed joint indy1_joint5
- removed joint indy1_joint_world
- removed joint indy1_tcp
- removed joint panda0_finger_joint1
- removed joint panda0_finger_joint2
- removed joint panda0_hand_joint
- removed joint panda0_joint1
- removed joint panda0_joint2
- removed joint panda0_joint3
- removed joint panda0_joint4
- removed joint panda0_joint5
- removed joint panda0_joint6
- removed joint panda0_joint7
- removed joint panda0_joint8
- removed joint panda0_joint_world
- added joint indy0_joint0: type revolute, parent indy0_link0, child indy0_link1, origin xyz=0.0 0.0 0.0775 rpy=0.0 0.0 0.0, axis 0.0 0.0 1.0, limit lower=-3.05432619099 upper=3.05432619099 effort=10.0 velocity=1.0
- added joint indy0_joint1: type revolute, parent indy0_link1, child indy0_link2, origin xyz=0.0 -0.109 0.222 rpy=1.57079632679 1.57079632679 0.0, axis 0.0 0.0 1.0, limit lower=-3.05432619099 upper=3.05432619099 effort=10.0 velocity=1.0
- added joint indy0_joint2: type revolute, parent indy0_link2, child indy0_link3, origin xyz=-0.45 0.0 -0.0305 rpy=0.0 0.0 0.0, axis 0.0 0.0 1.0, limit lower=-3.05432619099 upper=3.05432619099 effort=10.0 velocity=1.0
- added joint indy0_joint3: type revolute, parent indy0_link3, child indy0_link4, origin xyz=-0.267 0.0 -0.075 rpy=-1.57079632679 0.0 1.57079632679, axis 0.0 0.0 1.0, limit lower=-3.05432619099 upper=3.05432619099 effort=10.0 velocity=1.0
- added joint indy0_joint4: type revolute, parent indy0_link4, child indy0_link5, origin xyz=0.0 -0.114 0.083 rpy=1.57079632679 1.57079632679 0.0, axis 0.0 0.0 1.0, limit lower=-3.05432619099 upper=3.05432619099 effort=10.0 velocity=1.0
- added joint indy0_joint5: type revolute, parent indy0_link5, child indy0_link6, origin xyz=-0.168 0.0 0.069 rpy=-1.57079632679 0.0 1.57079632679, axis 0.0 0.0 1.0, limit lower=-3.75245789179 upper=3.75245789179 effort=10.0 velocity=1.0
- added joint indy0_joint_world: type fixed, parent world, child indy0_link0, origin xyz=0.0 -0.5 0.0 rpy=0.0 0.0 0.0
- added joint indy0_tcp: type fixed, parent indy0_link6, child indy0_tcp, origin xyz=0.0 0.0 0.06 rpy=0.0 0.0 0.0
- added joint panda1_finger_joint1: type fixed, parent panda1_hand, child panda1_leftfinger, origin xyz=0.0 0.04 0.0584 rpy=0.0 0.0 0.0, axis 0.0 1.0 0.0, limit lower=0.0 upper=0.04 effort=20.0 velocity=0.2
- added joint panda1_finger_joint2: type fixed, parent panda1_hand, child panda1_rightfinger, origin xyz=0.0 -0.04 0.0584 rpy=0.0 0.0 0.0, axis 0.0 -1.0 0.0, limit lower=0.0 upper=0.04 effort=20.0 velocity=0.2, mimic joint=panda1_finger_joint1
- added joint panda1_hand_joint: type fixed, parent panda1_link8, child panda1_hand, origin xyz=0.0 0.0 0.0 rpy=0.0 0.0 -0.785398163397
- added joint panda1_joint1: type revolute, parent panda1_link0, child panda1_link1, origin xyz=0.0 0.0 0.333 rpy=0.0 0.0 0.0, axis 0.0 0.0 1.0, limit lower=-2.8973 upper=2.8973 effort=87.0 velocity=2.175
- added joint panda1_joint2: type revolute, parent panda1_link1, child panda1_link2, origin xyz=0.0 0.0 0.0 rpy=-1.57079632679 0.0 0.0, axis 0.0 0.0 1.0, limit lower=-1.7628 upper=1.7628 effort=87.0 velocity=2.175
- added joint panda1_joint3: type revolute, parent panda1_link2, child panda1_link3, origin xyz=0.0 -0.316 0.0 rpy=1.57079632679 0.0 0.0, axis 0.0 0.0 1.0, limit lower=-2.8973 upper=2.8973 effort=87.0 velocity=2.175
- added joint panda1_joint4: type revolute, parent panda1_link3, child panda1_link4, origin xyz=0.0825 0.0 0.0 rpy=1.57079632679 0.0 0.0, axis 0.0 0.0 1.0, limit lower=-3.0718 upper=-0.0698 effort=87.0 velocity=2.175
- added joint panda1_joint5: type revolute, parent panda1_link4, child panda1_link5, origin xyz=-0.0825 0.384 0.0 rpy=-1.57079632679 0.0 0.0, axis 0.0 0.0 1.0, limit lower=-2.8973 upper=2.8973 effort=12.0 velocity=2.61
- added joint panda1_joint6: type revolute, parent panda1_link5, child panda1_link6, origin xyz=0.0 0.0 0.0 rpy=1.57079632679 0.0 0.0, axis 0.0 0.0 1.0, limit lower=-0.0175 upper=3.7525 effort=12.0 velocity=2.61
- added joint panda1_joint7: type revolute, parent panda1_link6, child panda1_link7, origin xyz=0.088 0.0 0.0 rpy=1.57079632679 0.0 0.0, axis 0.0 0.0 1.0, limit lower=-2.8973 upper=2.8973 effort=12.0 velocity=2.61
- added joint panda1_joint8: type fixed, parent panda1_link7, child panda1_link8, origin xyz=0.0 0.0 0.107 rpy=0.0 0.0 0.0, axis 0.0 0.0 0.0
- added joint panda1_joint_world: type fixed, parent world, child panda1_link0, origin xyz=0.0 0.5 0.0 rpy=0.0 0.0 0.0

File: eTaSL/robots/custom_robots.urdf.xacro (robot description, xacro)
@@ -1,9 +1,11 @@
 <?xml version="1.0" encoding="utf-8"?>
 <robot xmlns:xacro="http://www.ros.org/wiki/xacro" name="custom_robots">
-  <xacro:include filename="$(find indy7_description)/urdf/materials.xacro"/>
-  <xacro:include filename="$(env TF_GMT_ETASL_DIR)/robots/panda_robot.xacro"/>
-  <xacro:include filename="$(env TF_GMT_ETASL_DIR)/robots/indy7_robot.xacro"/>
-  <link name="world"/>
-  <xacro:panda_robot robot_id="0" xyz="0 0.5 0" connected_to="world"/>
-  <xacro:indy7_robot robot_id="1" xyz="0 -0.5 0" connected_to="world"/>
+<xacro:include filename="$(find indy7_description)/urdf/materials.xacro"/>
+<xacro:include filename="$(env TF_GMT_ETASL_DIR)/robots/panda_robot.xacro"/>
+<xacro:include filename="$(env TF_GMT_ETASL_DIR)/robots/indy7_robot.xacro"/>
+<link name="world"/>
+<!-- BODY BEGIN -->
+<xacro:indy7_robot robot_id="0" xyz="0 -0.5 0" rpy="0 0 0" connected_to="world"/>
+<xacro:panda_robot robot_id="1" xyz="0 0.5 0" rpy="0 0 0" connected_to="world"/>
+<!-- BODY END -->
 </robot>

Commit message: add - initialize error debug - panda mesh refinement, mesh collision

File: eTaSL/robots/custom_robots.urdf (robot description, URDF)
Before this commit: robot custom_robots, 21 links, 20 joints
Joints:
- joint panda1_finger_joint1: axis 0.0 1.0 0.0 -> (none); limit lower=0.0 upper=0.04 effort=20.0 velocity=0.2 -> (none)
- joint panda1_finger_joint2: axis 0.0 -1.0 0.0 -> (none); limit lower=0.0 upper=0.04 effort=20.0 velocity=0.2 -> (none)
