Commit message: add velocity limit

File: eTaSL/robots/custom_robots.urdf (robot description, URDF)
Before this commit: robot custom_robots, 21 links, 20 joints
Joints:
- joint indy0_joint0: limit lower=-3.05432619099 upper=3.05432619099 effort=10.0 velocity=1.0 -> lower=-3.05432619099 upper=3.05432619099 effort=10.0 velocity=1.3089969389957472
- joint indy0_joint1: limit lower=-3.05432619099 upper=3.05432619099 effort=10.0 velocity=1.0 -> lower=-3.05432619099 upper=3.05432619099 effort=10.0 velocity=1.3089969389957472
- joint indy0_joint2: limit lower=-3.05432619099 upper=3.05432619099 effort=10.0 velocity=1.0 -> lower=-3.05432619099 upper=3.05432619099 effort=10.0 velocity=1.3089969389957472
- joint indy0_joint3: limit lower=-3.05432619099 upper=3.05432619099 effort=10.0 velocity=1.0 -> lower=-3.05432619099 upper=3.05432619099 effort=10.0 velocity=1.5707963267948966
- joint indy0_joint4: limit lower=-3.05432619099 upper=3.05432619099 effort=10.0 velocity=1.0 -> lower=-3.05432619099 upper=3.05432619099 effort=10.0 velocity=1.5707963267948966
- joint indy0_joint5: limit lower=-3.75245789179 upper=3.75245789179 effort=10.0 velocity=1.0 -> lower=-3.75245789179 upper=3.75245789179 effort=10.0 velocity=1.5707963267948966
- joint panda1_joint1: limit lower=-2.8973 upper=2.8973 effort=87.0 velocity=2.175 -> lower=-2.8973 upper=2.8973 effort=87.0 velocity=1.3089969389957472
- joint panda1_joint2: limit lower=-1.7628 upper=1.7628 effort=87.0 velocity=2.175 -> lower=-1.7628 upper=1.7628 effort=87.0 velocity=1.3089969389957472
- joint panda1_joint3: limit lower=-2.8973 upper=2.8973 effort=87.0 velocity=2.175 -> lower=-2.8973 upper=2.8973 effort=87.0 velocity=1.3089969389957472
- joint panda1_joint4: limit lower=-3.0718 upper=-0.0698 effort=87.0 velocity=2.175 -> lower=-3.0718 upper=-0.0698 effort=87.0 velocity=1.3089969389957472
- joint panda1_joint5: limit lower=-2.8973 upper=2.8973 effort=12.0 velocity=2.61 -> lower=-2.8973 upper=2.8973 effort=12.0 velocity=1.5707963267948966
- joint panda1_joint6: limit lower=-0.0175 upper=3.7525 effort=12.0 velocity=2.61 -> lower=-0.0175 upper=3.7525 effort=12.0 velocity=1.5707963267948966
- joint panda1_joint7: limit lower=-2.8973 upper=2.8973 effort=12.0 velocity=2.61 -> lower=-2.8973 upper=2.8973 effort=12.0 velocity=1.5707963267948966

Commit message: constraints optimized

File: eTaSL/robots/custom_robots.urdf (robot description, URDF)
Before this commit: robot custom_robots, 21 links, 20 joints
Links:
- link indy0_link0: geometry visual mesh filename=package://indy7_description/meshes/stl/Indy7_0.stl
- link indy0_link1: geometry collision cylinder length=0.3 radius=0.1; visual mesh filename=package://indy7_description/meshes/stl/Indy7_1.stl
- link indy0_link2: geometry collision cylinder length=0.2 radius=0.085; collision cylinder length=0.45 radius=0.073
- link indy0_link3: geometry collision cylinder length=0.2 radius=0.055; visual mesh filename=package://indy7_description/meshes/stl/Indy7_3.stl
- link indy0_link4: geometry collision cylinder length=0.35 radius=0.055; visual mesh filename=package://indy7_description/meshes/stl/Indy7_4.stl
- link indy0_link5: geometry collision cylinder length=0.183 radius=0.055; visual mesh filename=package://indy7_description/meshes/stl/Indy7_5.stl
- link indy0_link6: geometry collision cylinder length=0.218 radius=0.05; visual mesh filename=package://indy7_description/meshes/stl/Indy7_6.stl

File: eTaSL/robots/indy7_robot-bak.xacro (robot description, xacro)
@@ -20,4 +20,10 @@
 			<material name="${indy_material}"/>
 		</visual>
+		<collision>
+			<origin xyz="0 0 0" rpy="0 0 0"/>
+			<geometry>
+				<cylinder length="0.075" radius="0.102"/>
+			</geometry>
+		</collision>
 		<inertial>
 			<origin xyz="0 0 0" rpy="0 0 0"/>
@@ -35,7 +41,13 @@
 		</visual>
 		<collision>
-			<origin xyz="0 0 0.072" rpy="0 0 0"/>
-			<geometry>
-				<cylinder length="0.3" radius="0.1"/>
+			<origin xyz="0 0 0.111" rpy="0 0 0"/>
+			<geometry>
+				<cylinder length="0.222" radius="0.075"/>
+			</geometry>
+		</collision>
+		<collision>
+			<origin xyz="0 -0.0545 0.222" rpy="${PI/2} 0 0"/>
+			<geometry>
+				<cylinder length="0.109" radius="0.075"/>
 			</geometry>
 		</collision>
@@ -57,11 +69,17 @@
 			<origin xyz="-0.225 0 0.09" rpy="${PI/2} 0 -${PI/2}"/>
 			<geometry>
-				<cylinder length="0.450" radius="0.073"/>
-			</geometry>
-		</collision>
-		<collision>
-			<origin xyz="0 0 -0.01" rpy="0 0 0"/>
-			<geometry>
-				<cylinder length="0.2" radius="0.085"/>
+				<cylinder length="0.450" radius="0.063"/>
+			</geometry>
+		</collision>
+		<collision>
+			<origin xyz="0 0 0.045" rpy="0 0 0"/>
+			<geometry>
+				<cylinder length="0.09" radius="0.075"/>
+			</geometry>
+		</collision>
+		<collision>
+			<origin xyz="-0.45 0 0.02975 " rpy="0 0 0"/>
+			<geometry>
+				<cylinder length="0.1205" radius="0.045"/>
 			</geometry>
 		</collision>
@@ -81,7 +99,13 @@
 		</visual>
 		<collision>
-			<origin xyz="0 0 0.03" rpy="0 0 0"/>
-			<geometry>
-				<cylinder length="0.2" radius="0.055"/>
+			<origin xyz="-0.1335 0 -0.075" rpy="${PI/2} 0 -${PI/2}"/>
+			<geometry>
+				<cylinder length="0.267" radius="0.045"/>
+			</geometry>
+		</collision>
+		<collision>
+			<origin xyz="0 0 -0.0375" rpy="0 0 0"/>
+			<geometry>
+				<cylinder length="0.075" radius="0.045"/>
 			</geometry>
 		</collision>
@@ -101,7 +125,19 @@
 		</visual>
 		<collision>
-			<origin xyz="0 0 -0.092" rpy="0 0 0"/>
-			<geometry>
-				<cylinder length="0.35" radius="0.055"/>
+			<origin xyz="0 -0.057 0.083" rpy="${PI/2} 0 0"/>
+			<geometry>
+				<cylinder length="0.114" radius="0.045"/>
+			</geometry>
+		</collision>
+		<collision>
+			<origin xyz="0 -0.057 0.083" rpy="${PI/2} 0 0"/>
+			<geometry>
+				<cylinder length="0.114" radius="0.045"/>
+			</geometry>
+		</collision>
+		<collision>
+			<origin xyz="0 0 0.0415" rpy="0 0 0"/>
+			<geometry>
+				<cylinder length="0.083" radius="0.045"/>
 			</geometry>
 		</collision>
@@ -121,7 +157,13 @@
 		</visual>
 		<collision>
-			<origin xyz="-0 0 -0.0225" rpy="0 0 0"/>
-			<geometry>
-				<cylinder length="0.183" radius="0.055"/>
+			<origin xyz="-0.084 0 0.069" rpy="${PI/2} 0 -${PI/2}"/>
+			<geometry>
+				<cylinder length="0.168" radius="0.045"/>
+			</geometry>
+		</collision>
+		<collision>
+			<origin xyz="-0 0 0.0345" rpy="0 0 0"/>
+			<geometry>
+				<cylinder length="0.069" radius="0.045"/>
 			</geometry>
 		</collision>
@@ -141,7 +183,7 @@
 		</visual>
 		<collision>
-			<origin xyz="0 0 -0.054" rpy="0 0 0"/>
-			<geometry>
-				<cylinder length="0.218" radius="0.050"/>
+			<origin xyz="0 0 0.03" rpy="0 0 0"/>
+			<geometry>
+				<cylinder length="0.06" radius="0.045"/>
 			</geometry>
 		</collision>

Commit message: done: kinect environment sync

File: eTaSL/robots/custom_robots.urdf (robot description, URDF)
Before this commit: robot custom_robots, 21 links, 20 joints
Joints:
- joint indy0_joint_world: origin xyz=0.0 -0.5 0.0 rpy=0.0 0.0 0.0 -> xyz=-0.328049600124 -0.0254697203636 0.0018418431282 rpy=-0.00952161836518 -0.00819341519378 1.54180969078
- joint panda1_joint_world: origin xyz=0.0 0.5 0.0 rpy=0.0 0.0 0.0 -> xyz=0.286244928837 0.429062277079 0.00359612703323 rpy=-0.101035998965 -0.0275128574156 -1.57501283665

File: eTaSL/robots/custom_robots.urdf.xacro (robot description, xacro)
@@ -6,6 +6,6 @@
 <link name="world"/>
 <!-- BODY BEGIN -->
-<xacro:indy7_robot robot_id="0" xyz="0 -0.5 0" rpy="0 0 0" connected_to="world"/>
-<xacro:panda_robot robot_id="1" xyz="0 0.5 0" rpy="0 0 0" connected_to="world"/>
+<xacro:indy7_robot robot_id="0" xyz="-0.328049600124 -0.0254697203636 0.0018418431282" rpy="-0.00952161836518 -0.00819341519378 1.54180969078" connected_to="world"/>
+<xacro:panda_robot robot_id="1" xyz="0.286244928837 0.429062277079 0.00359612703323" rpy="-0.101035998965 -0.0275128574156 -1.57501283665" connected_to="world"/>
 <!-- BODY END -->
 </robot>

Commit message: indy trajectory following initial version

File: eTaSL/robots/custom_robots.urdf (robot description, URDF)
Before this commit: robot custom_robots, 21 links, 20 joints
Joints:
- joint indy0_joint_world: origin xyz=-0.328049600124 -0.0254697203636 0.0018418431282 rpy=-0.00952161836518 -0.00819341519378 1.54180969078 -> xyz=-0.27338463068 -0.0145324468613 0.0511643886566 rpy=0.00732033205866 -0.00214329858802 1.51741749193
- joint panda1_joint_world: origin xyz=0.286244928837 0.429062277079 0.00359612703323 rpy=-0.101035998965 -0.0275128574156 -1.57501283665 -> xyz=0.664858281612 0.394209086895 0.0303395986557 rpy=7.10060861184e-05 0.00684849814155 -1.63456437701

File: eTaSL/robots/custom_robots.urdf.xacro (robot description, xacro)
@@ -6,6 +6,6 @@
 <link name="world"/>
 <!-- BODY BEGIN -->
-<xacro:indy7_robot robot_id="0" xyz="-0.328049600124 -0.0254697203636 0.0018418431282" rpy="-0.00952161836518 -0.00819341519378 1.54180969078" connected_to="world"/>
-<xacro:panda_robot robot_id="1" xyz="0.286244928837 0.429062277079 0.00359612703323" rpy="-0.101035998965 -0.0275128574156 -1.57501283665" connected_to="world"/>
+<xacro:indy7_robot robot_id="0" xyz="-0.27338463068 -0.0145324468613 0.0511643886566" rpy="0.00732033205866 -0.00214329858802 1.51741749193" connected_to="world"/>
+<xacro:panda_robot robot_id="1" xyz="0.664858281612 0.394209086895 0.0303395986557" rpy="7.10060861184e-05 0.00684849814155 -1.63456437701" connected_to="world"/>
 <!-- BODY END -->
 </robot>

Commit message: added acceleration, interpolation

File: eTaSL/robots/custom_robots.urdf (robot description, URDF)
Before this commit: robot custom_robots, 21 links, 20 joints
Joints:
- joint indy0_joint0: limit lower=-3.05432619099 upper=3.05432619099 effort=10.0 velocity=1.3089969389957472 -> lower=-3.05432619099 upper=3.05432619099 effort=3.141592653589793 velocity=1.3089969389957472
- joint indy0_joint1: limit lower=-3.05432619099 upper=3.05432619099 effort=10.0 velocity=1.3089969389957472 -> lower=-3.05432619099 upper=3.05432619099 effort=3.141592653589793 velocity=1.3089969389957472
- joint indy0_joint2: limit lower=-3.05432619099 upper=3.05432619099 effort=10.0 velocity=1.3089969389957472 -> lower=-3.05432619099 upper=3.05432619099 effort=3.141592653589793 velocity=1.3089969389957472
- joint indy0_joint3: limit lower=-3.05432619099 upper=3.05432619099 effort=10.0 velocity=1.5707963267948966 -> lower=-3.05432619099 upper=3.05432619099 effort=3.141592653589793 velocity=1.5707963267948966
- joint indy0_joint4: limit lower=-3.05432619099 upper=3.05432619099 effort=10.0 velocity=1.5707963267948966 -> lower=-3.05432619099 upper=3.05432619099 effort=3.141592653589793 velocity=1.5707963267948966
- joint indy0_joint5: limit lower=-3.75245789179 upper=3.75245789179 effort=10.0 velocity=1.5707963267948966 -> lower=-3.75245789179 upper=3.75245789179 effort=3.141592653589793 velocity=1.5707963267948966
- joint indy0_joint_world: origin xyz=-0.27338463068 -0.0145324468613 0.0511643886566 rpy=0.00732033205866 -0.00214329858802 1.51741749193 -> xyz=-0.270824670792 -0.0157505571842 0.0500493049622 rpy=0.0177146642508 0.00907266499533 1.52353711186
- joint panda1_joint1: limit lower=-2.8973 upper=2.8973 effort=87.0 velocity=1.3089969389957472 -> lower=-2.8973 upper=2.8973 effort=3.141592653589793 velocity=1.3089969389957472
- joint panda1_joint2: limit lower=-1.7628 upper=1.7628 effort=87.0 velocity=1.3089969389957472 -> lower=-1.7628 upper=1.7628 effort=3.141592653589793 velocity=1.3089969389957472
- joint panda1_joint3: limit lower=-2.8973 upper=2.8973 effort=87.0 velocity=1.3089969389957472 -> lower=-2.8973 upper=2.8973 effort=3.141592653589793 velocity=1.3089969389957472
- joint panda1_joint4: limit lower=-3.0718 upper=-0.0698 effort=87.0 velocity=1.3089969389957472 -> lower=-3.0718 upper=-0.0698 effort=3.141592653589793 velocity=1.3089969389957472
- joint panda1_joint5: limit lower=-2.8973 upper=2.8973 effort=12.0 velocity=1.5707963267948966 -> lower=-2.8973 upper=2.8973 effort=3.141592653589793 velocity=1.5707963267948966
- joint panda1_joint6: limit lower=-0.0175 upper=3.7525 effort=12.0 velocity=1.5707963267948966 -> lower=-0.0175 upper=3.7525 effort=3.141592653589793 velocity=1.5707963267948966
- joint panda1_joint7: limit lower=-2.8973 upper=2.8973 effort=12.0 velocity=1.5707963267948966 -> lower=-2.8973 upper=2.8973 effort=3.141592653589793 velocity=1.5707963267948966
- joint panda1_joint_world: origin xyz=0.664858281612 0.394209086895 0.0303395986557 rpy=7.10060861184e-05 0.00684849814155 -1.63456437701 -> xyz=0.649404883385 0.399997353554 0.00985872745514 rpy=-0.0341424216818 -0.0145806313008 -1.63646380558

File: eTaSL/robots/custom_robots.urdf.xacro (robot description, xacro)
@@ -6,6 +6,6 @@
 <link name="world"/>
 <!-- BODY BEGIN -->
-<xacro:indy7_robot robot_id="0" xyz="-0.27338463068 -0.0145324468613 0.0511643886566" rpy="0.00732033205866 -0.00214329858802 1.51741749193" connected_to="world"/>
-<xacro:panda_robot robot_id="1" xyz="0.664858281612 0.394209086895 0.0303395986557" rpy="7.10060861184e-05 0.00684849814155 -1.63456437701" connected_to="world"/>
+<xacro:indy7_robot robot_id="0" xyz="-0.270824670792 -0.0157505571842 0.0500493049622" rpy="0.0177146642508 0.00907266499533 1.52353711186" connected_to="world"/>
+<xacro:panda_robot robot_id="1" xyz="0.649404883385 0.399997353554 0.00985872745514" rpy="-0.0341424216818 -0.0145806313008 -1.63646380558" connected_to="world"/>
 <!-- BODY END -->
 </robot>

Commit message: finished trajectory

File: eTaSL/robots/custom_robots.urdf (robot description, URDF)
Before this commit: robot custom_robots, 21 links, 20 joints
Joints:
- joint indy0_joint_world: origin xyz=-0.270824670792 -0.0157505571842 0.0500493049622 rpy=0.0177146642508 0.00907266499533 1.52353711186 -> xyz=-0.2701998353 -0.015514627099 0.0508535504341 rpy=0.0159077957519 0.00442104645988 1.52100187385
- joint panda1_joint_world: origin xyz=0.649404883385 0.399997353554 0.00985872745514 rpy=-0.0341424216818 -0.0145806313008 -1.63646380558 -> xyz=0.650361061096 0.399778693914 0.0142936110497 rpy=-0.0317647354784 -0.0116640282806 -1.6370816388

File: eTaSL/robots/custom_robots.urdf.xacro (robot description, xacro)
@@ -6,6 +6,6 @@
 <link name="world"/>
 <!-- BODY BEGIN -->
-<xacro:indy7_robot robot_id="0" xyz="-0.270824670792 -0.0157505571842 0.0500493049622" rpy="0.0177146642508 0.00907266499533 1.52353711186" connected_to="world"/>
-<xacro:panda_robot robot_id="1" xyz="0.649404883385 0.399997353554 0.00985872745514" rpy="-0.0341424216818 -0.0145806313008 -1.63646380558" connected_to="world"/>
+<xacro:indy7_robot robot_id="0" xyz="-0.2701998353 -0.015514627099 0.0508535504341" rpy="0.0159077957519 0.00442104645988 1.52100187385" connected_to="world"/>
+<xacro:panda_robot robot_id="1" xyz="0.650361061096 0.399778693914 0.0142936110497" rpy="-0.0317647354784 -0.0116640282806 -1.6370816388" connected_to="world"/>
 <!-- BODY END -->
 </robot>

Commit message: prepare sync trajectory done

File: eTaSL/robots/custom_robots.urdf (robot description, URDF)
Before this commit: robot custom_robots, 21 links, 20 joints
Joints:
- joint indy0_joint_world: origin xyz=-0.2701998353 -0.015514627099 0.0508535504341 rpy=0.0159077957519 0.00442104645988 1.52100187385 -> xyz=-0.271527409554 -0.0154553800821 0.0499985814095 rpy=0.0153188939223 0.0053701700303 1.52145857
- joint panda1_joint_world: origin xyz=0.650361061096 0.399778693914 0.0142936110497 rpy=-0.0317647354784 -0.0116640282806 -1.6370816388 -> xyz=0.648643374443 0.399706482887 0.0143700242043 rpy=-0.0285099029659 -0.0172426985423 -1.63094361292

File: eTaSL/robots/custom_robots.urdf.xacro (robot description, xacro)
@@ -6,6 +6,6 @@
 <link name="world"/>
 <!-- BODY BEGIN -->
-<xacro:indy7_robot robot_id="0" xyz="-0.2701998353 -0.015514627099 0.0508535504341" rpy="0.0159077957519 0.00442104645988 1.52100187385" connected_to="world"/>
-<xacro:panda_robot robot_id="1" xyz="0.650361061096 0.399778693914 0.0142936110497" rpy="-0.0317647354784 -0.0116640282806 -1.6370816388" connected_to="world"/>
+<xacro:indy7_robot robot_id="0" xyz="-0.271527409554 -0.0154553800821 0.0499985814095" rpy="0.0153188939223 0.0053701700303 1.52145857" connected_to="world"/>
+<xacro:panda_robot robot_id="1" xyz="0.648643374443 0.399706482887 0.0143700242043" rpy="-0.0285099029659 -0.0172426985423 -1.63094361292" connected_to="world"/>
 <!-- BODY END -->
 </robot>

Commit message: sync motion initial ver.

File: eTaSL/robots/custom_robots.urdf (robot description, URDF)
Before this commit: robot custom_robots, 21 links, 20 joints
Joints:
- joint indy0_joint_world: origin xyz=-0.271527409554 -0.0154553800821 0.0499985814095 rpy=0.0153188939223 0.0053701700303 1.52145857 -> xyz=-0.50934612751 -0.0140069276094 0.0138622522354 rpy=0.0134274033876 0.000418877622475 1.54826227309
- joint panda1_joint_world: origin xyz=0.648643374443 0.399706482887 0.0143700242043 rpy=-0.0285099029659 -0.0172426985423 -1.63094361292 -> xyz=0.00160580873489 0.436583042145 0.00706601142883 rpy=-0.00661957175964 0.00636852325315 -1.59232471466

File: eTaSL/robots/custom_robots.urdf.xacro (robot description, xacro)
@@ -6,6 +6,6 @@
 <link name="world"/>
 <!-- BODY BEGIN -->
-<xacro:indy7_robot robot_id="0" xyz="-0.271527409554 -0.0154553800821 0.0499985814095" rpy="0.0153188939223 0.0053701700303 1.52145857" connected_to="world"/>
-<xacro:panda_robot robot_id="1" xyz="0.648643374443 0.399706482887 0.0143700242043" rpy="-0.0285099029659 -0.0172426985423 -1.63094361292" connected_to="world"/>
+<xacro:indy7_robot robot_id="0" xyz="-0.50934612751 -0.0140069276094 0.0138622522354" rpy="0.0134274033876 0.000418877622475 1.54826227309" connected_to="world"/>
+<xacro:panda_robot robot_id="1" xyz="0.00160580873489 0.436583042145 0.00706601142883" rpy="-0.00661957175964 0.00636852325315 -1.59232471466" connected_to="world"/>
 <!-- BODY END -->
 </robot>

Commit message: calc_offset initial ver.

File: eTaSL/robots/custom_robots.urdf (robot description, URDF)
Before this commit: robot custom_robots, 21 links, 20 joints
Joints:
- joint indy0_joint_world: origin xyz=-0.50934612751 -0.0140069276094 0.0138622522354 rpy=0.0134274033876 0.000418877622475 1.54826227309 -> xyz=-0.517569541931 0.241169840097 -0.013944029808 rpy=-0.0439173793565 0.0341804011987 1.08908952516
- joint panda1_joint_world: origin xyz=0.00160580873489 0.436583042145 0.00706601142883 rpy=-0.00661957175964 0.00636852325315 -1.59232471466 -> xyz=0.188743054867 0.398934483528 0.00163584947586 rpy=-0.00774259098144 -0.00478142806801 -2.04887347232

File: eTaSL/robots/custom_robots.urdf.xacro (robot description, xacro)
@@ -6,6 +6,6 @@
 <link name="world"/>
 <!-- BODY BEGIN -->
-<xacro:indy7_robot robot_id="0" xyz="-0.50934612751 -0.0140069276094 0.0138622522354" rpy="0.0134274033876 0.000418877622475 1.54826227309" connected_to="world"/>
-<xacro:panda_robot robot_id="1" xyz="0.00160580873489 0.436583042145 0.00706601142883" rpy="-0.00661957175964 0.00636852325315 -1.59232471466" connected_to="world"/>
+<xacro:indy7_robot robot_id="0" xyz="-0.517569541931 0.241169840097 -0.013944029808" rpy="-0.0439173793565 0.0341804011987 1.08908952516" connected_to="world"/>
+<xacro:panda_robot robot_id="1" xyz="0.188743054867 0.398934483528 0.00163584947586" rpy="-0.00774259098144 -0.00478142806801 -2.04887347232" connected_to="world"/>
 <!-- BODY END -->
 </robot>

Commit message: cleaned

File: eTaSL/robots/custom_robots.urdf (robot description, URDF)
Before this commit: robot custom_robots, 21 links, 20 joints
Joints:
- joint indy0_joint_world: origin xyz=-0.517569541931 0.241169840097 -0.013944029808 rpy=-0.0439173793565 0.0341804011987 1.08908952516 -> xyz=-0.52249443531 0.10203795135 0.0125234127045 rpy=0.00833006380493 0.0172834411121 1.27034759964
- joint panda1_joint_world: origin xyz=0.188743054867 0.398934483528 0.00163584947586 rpy=-0.00774259098144 -0.00478142806801 -2.04887347232 -> xyz=0.0970267355442 0.390915095806 0.00331979990005 rpy=-0.00937373930552 -0.00443786923144 -1.87606356043

File: eTaSL/robots/custom_robots.urdf.xacro (robot description, xacro)
@@ -6,6 +6,6 @@
 <link name="world"/>
 <!-- BODY BEGIN -->
-<xacro:indy7_robot robot_id="0" xyz="-0.517569541931 0.241169840097 -0.013944029808" rpy="-0.0439173793565 0.0341804011987 1.08908952516" connected_to="world"/>
-<xacro:panda_robot robot_id="1" xyz="0.188743054867 0.398934483528 0.00163584947586" rpy="-0.00774259098144 -0.00478142806801 -2.04887347232" connected_to="world"/>
+<xacro:indy7_robot robot_id="0" xyz="-0.52249443531 0.10203795135 0.0125234127045" rpy="0.00833006380493 0.0172834411121 1.27034759964" connected_to="world"/>
+<xacro:panda_robot robot_id="1" xyz="0.0970267355442 0.390915095806 0.00331979990005" rpy="-0.00937373930552 -0.00443786923144 -1.87606356043" connected_to="world"/>
 <!-- BODY END -->
 </robot>

Commit message: calibration short tested w. panda

File: eTaSL/robots/custom_robots.urdf (robot description, URDF)
Before this commit: robot custom_robots, 21 links, 20 joints
Joints:
- joint indy0_joint_world: origin xyz=-0.52249443531 0.10203795135 0.0125234127045 rpy=0.00833006380493 0.0172834411121 1.27034759964 -> xyz=-0.520950078964 0.102396816015 0.0148023962975 rpy=0.0179848883694 0.0089306256948 1.26405232018
- joint panda1_hand_joint: origin xyz=0.0 0.0 0.0 rpy=0.0 0.0 -0.785398163397 -> xyz=0.0 0.0 0.0 rpy=0.0 -0.0 -0.785398163397
- joint panda1_joint_world: origin xyz=0.0970267355442 0.390915095806 0.00331979990005 rpy=-0.00937373930552 -0.00443786923144 -1.87606356043 -> xyz=0.0909019597926 0.395140539508 0.00399171533466 rpy=-0.011794190703 -0.00731106135215 -1.87625232935

File: eTaSL/robots/custom_robots.urdf.xacro (robot description, xacro)
@@ -6,6 +6,6 @@
 <link name="world"/>
 <!-- BODY BEGIN -->
-<xacro:indy7_robot robot_id="0" xyz="-0.52249443531 0.10203795135 0.0125234127045" rpy="0.00833006380493 0.0172834411121 1.27034759964" connected_to="world"/>
-<xacro:panda_robot robot_id="1" xyz="0.0970267355442 0.390915095806 0.00331979990005" rpy="-0.00937373930552 -0.00443786923144 -1.87606356043" connected_to="world"/>
+<xacro:indy7_robot robot_id="0" xyz="-0.520950078964 0.102396816015 0.0148023962975" rpy="0.0179848883694 0.0089306256948 1.26405232018" connected_to="world"/>
+<xacro:panda_robot robot_id="1" xyz="0.0909019597926 0.395140539508 0.00399171533466" rpy="-0.011794190703 -0.00731106135215 -1.87625232935" connected_to="world"/>
 <!-- BODY END -->
 </robot>
