Commit message: calibration w. indy

File: eTaSL/robots/custom_robots.urdf (robot description, URDF)
Before this commit: robot custom_robots, 21 links, 20 joints
Joints:
- joint indy0_joint_world: origin xyz=-0.520950078964 0.102396816015 0.0148023962975 rpy=0.0179848883694 0.0089306256948 1.26405232018 -> xyz=-0.532590679825 0.107710005063 0.0127092942974 rpy=0.0150965929123 0.00811313875957 1.27159046918
- joint indy0_tcp: origin xyz=0.0 0.0 0.06 rpy=0.0 0.0 0.0 -> xyz=-0.00590267304607 0.000456018937306 0.0602359141913 rpy=-0.0272346363883 -0.00977225860042 0.014358710505
- joint panda1_hand_joint: origin xyz=0.0 0.0 0.0 rpy=0.0 -0.0 -0.785398163397 -> xyz=0.0015538636864 0.00384081899101 0.00117409495442 rpy=0.00799966069138 -0.00551973919069 -0.794669530373
- joint panda1_joint6: limit lower=-0.0175 upper=3.7525 effort=3.141592653589793 velocity=1.5707963267948966 -> lower=0.5 upper=3.7525 effort=3.141592653589793 velocity=1.5707963267948966
- joint panda1_joint_world: origin xyz=0.0909019597926 0.395140539508 0.00399171533466 rpy=-0.011794190703 -0.00731106135215 -1.87625232935 -> xyz=0.0914257230014 0.395475427003 0.00427928960791 rpy=-0.0112616728328 -0.00702172347129 -1.87598923262

File: eTaSL/robots/custom_robots.urdf.xacro (robot description, xacro)
@@ -6,6 +6,6 @@
 <link name="world"/>
 <!-- BODY BEGIN -->
-<xacro:indy7_robot robot_id="0" xyz="-0.520950078964 0.102396816015 0.0148023962975" rpy="0.0179848883694 0.0089306256948 1.26405232018" connected_to="world"/>
-<xacro:panda_robot robot_id="1" xyz="0.0909019597926 0.395140539508 0.00399171533466" rpy="-0.011794190703 -0.00731106135215 -1.87625232935" connected_to="world"/>
+<xacro:indy7_robot robot_id="0" xyz="-0.532590679825 0.107710005063 0.0127092942974" rpy="0.0150965929123 0.00811313875957 1.27159046918" connected_to="world"/>
+<xacro:panda_robot robot_id="1" xyz="0.0914257230014 0.395475427003 0.00427928960791" rpy="-0.0112616728328 -0.00702172347129 -1.87598923262" connected_to="world"/>
 <!-- BODY END -->
 </robot>

Commit message: add triangulation examples

File: eTaSL/robots/custom_robots.urdf (robot description, URDF)
Before this commit: robot custom_robots, 21 links, 20 joints
Joints:
- joint indy0_joint_world: origin xyz=-0.532590679825 0.107710005063 0.0127092942974 rpy=0.0150965929123 0.00811313875957 1.27159046918 -> xyz=-0.217783391476 -0.393223285675 0.0167390704155 rpy=0.0109810741192 0.0144872136831 1.53302944723
- joint indy0_tcp: origin xyz=-0.00590267304607 0.000456018937306 0.0602359141913 rpy=-0.0272346363883 -0.00977225860042 0.014358710505 -> xyz=0.0 0.0 0.0599999986589 rpy=0.0 -0.0 0.0
- joint panda1_hand_joint: origin xyz=0.0015538636864 0.00384081899101 0.00117409495442 rpy=0.00799966069138 -0.00551973919069 -0.794669530373 -> xyz=0.0 0.0 0.0 rpy=0.0 -0.0 -0.785398163397
- joint panda1_joint6: limit lower=0.5 upper=3.7525 effort=3.141592653589793 velocity=1.5707963267948966 -> lower=-0.0175 upper=3.7525 effort=3.141592653589793 velocity=1.5707963267948966
- joint panda1_joint_world: origin xyz=0.0914257230014 0.395475427003 0.00427928960791 rpy=-0.0112616728328 -0.00702172347129 -1.87598923262 -> xyz=0.36877477169 0.0418559014797 -0.00364065170288 rpy=-0.00481223139387 -0.0115587399502 -1.63112361166

File: eTaSL/robots/custom_robots.urdf.xacro (robot description, xacro)
@@ -6,6 +6,6 @@
 <link name="world"/>
 <!-- BODY BEGIN -->
-<xacro:indy7_robot robot_id="0" xyz="-0.532590679825 0.107710005063 0.0127092942974" rpy="0.0150965929123 0.00811313875957 1.27159046918" connected_to="world"/>
-<xacro:panda_robot robot_id="1" xyz="0.0914257230014 0.395475427003 0.00427928960791" rpy="-0.0112616728328 -0.00702172347129 -1.87598923262" connected_to="world"/>
+<xacro:indy7_robot robot_id="0" xyz="-0.217783391476 -0.393223285675 0.0167390704155" rpy="0.0109810741192 0.0144872136831 1.53302944723" connected_to="world"/>
+<xacro:panda_robot robot_id="1" xyz="0.36877477169 0.0418559014797 -0.00364065170288" rpy="-0.00481223139387 -0.0115587399502 -1.63112361166" connected_to="world"/>
 <!-- BODY END -->
 </robot>

Commit message: recalibration-not good

File: eTaSL/robots/custom_robots.urdf (robot description, URDF)
Before this commit: robot custom_robots, 21 links, 20 joints
Joints:
- joint indy0_joint_world: origin xyz=-0.217783391476 -0.393223285675 0.0167390704155 rpy=0.0109810741192 0.0144872136831 1.53302944723 -> xyz=0.612544778056 0.0789817566548 0.0247673378352 rpy=0.0489630050924 0.000192864434053 -1.6388714317
- joint indy0_tcp: origin xyz=0.0 0.0 0.0599999986589 rpy=0.0 -0.0 0.0 -> xyz=0.000402975278853 -0.00066818685235 0.0588690187041 rpy=-0.0104108936784 -0.0160709183845 -0.0218111178257
- joint panda1_hand_joint: origin xyz=0.0 0.0 0.0 rpy=0.0 -0.0 -0.785398163397 -> xyz=0.0015538636864 0.00384081899101 0.00117409495442 rpy=0.00799966069138 -0.00551973919069 -0.794669530373
- joint panda1_joint_world: origin xyz=0.36877477169 0.0418559014797 -0.00364065170288 rpy=-0.00481223139387 -0.0115587399502 -1.63112361166 -> xyz=-0.0649315247183 -0.338550625397 -0.0015929573077 rpy=0.0353887261998 -0.0218884470509 1.48624490566

File: eTaSL/robots/custom_robots.urdf.xacro (robot description, xacro)
@@ -6,6 +6,6 @@
 <link name="world"/>
 <!-- BODY BEGIN -->
-<xacro:indy7_robot robot_id="0" xyz="-0.217783391476 -0.393223285675 0.0167390704155" rpy="0.0109810741192 0.0144872136831 1.53302944723" connected_to="world"/>
-<xacro:panda_robot robot_id="1" xyz="0.36877477169 0.0418559014797 -0.00364065170288" rpy="-0.00481223139387 -0.0115587399502 -1.63112361166" connected_to="world"/>
+<xacro:indy7_robot robot_id="0" xyz="0.612544778056 0.0789817566548 0.0247673378352" rpy="0.0489630050924 0.000192864434053 -1.6388714317" connected_to="world"/>
+<xacro:panda_robot robot_id="1" xyz="-0.0649315247183 -0.338550625397 -0.0015929573077" rpy="0.0353887261998 -0.0218884470509 1.48624490566" connected_to="world"/>
 <!-- BODY END -->
 </robot>

Commit message: Indy tracker tested on simulation

File: eTaSL/robots/custom_robots.urdf (robot description, URDF)
Before this commit: robot custom_robots, 21 links, 20 joints
Joints:
- joint indy0_joint_world: origin xyz=0.612544778056 0.0789817566548 0.0247673378352 rpy=0.0489630050924 0.000192864434053 -1.6388714317 -> xyz=0.367763519975 0.0285778110421 0.00270301862935 rpy=0.00581560357046 0.0145621496684 -1.49891262613
- joint indy0_tcp: origin xyz=0.000402975278853 -0.00066818685235 0.0588690187041 rpy=-0.0104108936784 -0.0160709183845 -0.0218111178257 -> xyz=-0.0125303795503 0.000417391292825 0.0652073328889 rpy=-0.0288878882228 -0.016886431851 -0.0403732322458
- joint panda1_joint_world: origin xyz=-0.0649315247183 -0.338550625397 -0.0015929573077 rpy=0.0353887261998 -0.0218884470509 1.48624490566 -> xyz=-0.291338219306 -0.435594861441 0.00447293881535 rpy=0.00352158178045 -0.00198499891338 1.56473166957

File: eTaSL/robots/custom_robots.urdf.xacro (robot description, xacro)
@@ -6,6 +6,6 @@
 <link name="world"/>
 <!-- BODY BEGIN -->
-<xacro:indy7_robot robot_id="0" xyz="0.612544778056 0.0789817566548 0.0247673378352" rpy="0.0489630050924 0.000192864434053 -1.6388714317" connected_to="world"/>
-<xacro:panda_robot robot_id="1" xyz="-0.0649315247183 -0.338550625397 -0.0015929573077" rpy="0.0353887261998 -0.0218884470509 1.48624490566" connected_to="world"/>
+<xacro:indy7_robot robot_id="0" xyz="0.367763519975 0.0285778110421 0.00270301862935" rpy="0.00581560357046 0.0145621496684 -1.49891262613" connected_to="world"/>
+<xacro:panda_robot robot_id="1" xyz="-0.291338219306 -0.435594861441 0.00447293881535" rpy="0.00352158178045 -0.00198499891338 1.56473166957" connected_to="world"/>
 <!-- BODY END -->
 </robot>

Commit message: online tracking indy homing tested

File: eTaSL/robots/custom_robots.urdf (robot description, URDF)
Before this commit: robot custom_robots, 21 links, 20 joints
Joints:
- joint indy0_joint_world: origin xyz=0.367763519975 0.0285778110421 0.00270301862935 rpy=0.00581560357046 0.0145621496684 -1.49891262613 -> xyz=-0.319578290246 -0.00410150076201 -0.000417835275873 rpy=0.00439442802347 0.0134426877365 1.6405039255
- joint panda1_joint_world: origin xyz=-0.291338219306 -0.435594861441 0.00447293881535 rpy=0.00352158178045 -0.00198499891338 1.56473166957 -> xyz=0.343492328869 0.459384615938 0.00433604585268 rpy=0.00305151779434 0.00181406569069 -1.57932698891

File: eTaSL/robots/custom_robots.urdf.xacro (robot description, xacro)
@@ -6,6 +6,6 @@
 <link name="world"/>
 <!-- BODY BEGIN -->
-<xacro:indy7_robot robot_id="0" xyz="0.367763519975 0.0285778110421 0.00270301862935" rpy="0.00581560357046 0.0145621496684 -1.49891262613" connected_to="world"/>
-<xacro:panda_robot robot_id="1" xyz="-0.291338219306 -0.435594861441 0.00447293881535" rpy="0.00352158178045 -0.00198499891338 1.56473166957" connected_to="world"/>
+<xacro:indy7_robot robot_id="0" xyz="-0.319578290246 -0.00410150076201 -0.000417835275873" rpy="0.00439442802347 0.0134426877365 1.6405039255" connected_to="world"/>
+<xacro:panda_robot robot_id="1" xyz="0.343492328869 0.459384615938 0.00433604585268" rpy="0.00305151779434 0.00181406569069 -1.57932698891" connected_to="world"/>
 <!-- BODY END -->
 </robot>

Commit message: stereo fixed

File: eTaSL/robots/custom_robots.urdf (robot description, URDF)
Before this commit: robot custom_robots, 21 links, 20 joints
Joints:
- joint indy0_joint_world: origin xyz=-0.319578290246 -0.00410150076201 -0.000417835275873 rpy=0.00439442802347 0.0134426877365 1.6405039255 -> xyz=-0.507298350334 0.0459206104279 0.00660020112991 rpy=-0.00641558405873 0.000878980837848 -1.58075939499
- joint indy0_tcp: origin xyz=-0.0125303795503 0.000417391292825 0.0652073328889 rpy=-0.0288878882228 -0.016886431851 -0.0403732322458 -> xyz=0.0 0.0 0.06 rpy=0.0 0.0 0.0
- joint panda1_hand_joint: origin xyz=0.0015538636864 0.00384081899101 0.00117409495442 rpy=0.00799966069138 -0.00551973919069 -0.794669530373 -> xyz=0.0 0.0 0.0 rpy=0.0 0.0 -0.785398163397
- joint panda1_joint_world: origin xyz=0.343492328869 0.459384615938 0.00433604585268 rpy=0.00305151779434 0.00181406569069 -1.57932698891 -> xyz=0.454326987267 -0.00940454006195 0.00411355495453 rpy=-0.00537314348419 -0.000365826033638 -1.57917701675

File: eTaSL/robots/custom_robots.urdf.xacro (robot description, xacro)
@@ -6,6 +6,6 @@
 <link name="world"/>
 <!-- BODY BEGIN -->
-<xacro:indy7_robot robot_id="0" xyz="-0.319578290246 -0.00410150076201 -0.000417835275873" rpy="0.00439442802347 0.0134426877365 1.6405039255" connected_to="world"/>
-<xacro:panda_robot robot_id="1" xyz="0.343492328869 0.459384615938 0.00433604585268" rpy="0.00305151779434 0.00181406569069 -1.57932698891" connected_to="world"/>
+<xacro:indy7_robot robot_id="0" xyz="-0.507298350334 0.0459206104279 0.00660020112991" rpy="-0.00641558405873 0.000878980837848 -1.58075939499" connected_to="world"/>
+<xacro:panda_robot robot_id="1" xyz="0.454326987267 -0.00940454006195 0.00411355495453" rpy="-0.00537314348419 -0.000365826033638 -1.57917701675" connected_to="world"/>
 <!-- BODY END -->
 </robot>

Commit message: task running tested w. panda

File: eTaSL/robots/custom_robots.urdf (robot description, URDF)
Before this commit: robot custom_robots, 21 links, 20 joints
Joints:
- joint indy0_joint_world: origin xyz=-0.507298350334 0.0459206104279 0.00660020112991 rpy=-0.00641558405873 0.000878980837848 -1.58075939499 -> xyz=-0.448628753424 0.0491750836372 0.0126187205315 rpy=-0.00559553685673 0.00815772775075 -1.5689325988
- joint panda1_joint_world: origin xyz=0.454326987267 -0.00940454006195 0.00411355495453 rpy=-0.00537314348419 -0.000365826033638 -1.57917701675 -> xyz=0.51068854332 -0.0208044052124 0.00980961322784 rpy=-0.00465814192854 0.00824846908983 -1.59513247343

File: eTaSL/robots/custom_robots.urdf.xacro (robot description, xacro)
@@ -6,6 +6,6 @@
 <link name="world"/>
 <!-- BODY BEGIN -->
-<xacro:indy7_robot robot_id="0" xyz="-0.507298350334 0.0459206104279 0.00660020112991" rpy="-0.00641558405873 0.000878980837848 -1.58075939499" connected_to="world"/>
-<xacro:panda_robot robot_id="1" xyz="0.454326987267 -0.00940454006195 0.00411355495453" rpy="-0.00537314348419 -0.000365826033638 -1.57917701675" connected_to="world"/>
+<xacro:indy7_robot robot_id="0" xyz="-0.448628753424 0.0491750836372 0.0126187205315" rpy="-0.00559553685673 0.00815772775075 -1.5689325988" connected_to="world"/>
+<xacro:panda_robot robot_id="1" xyz="0.51068854332 -0.0208044052124 0.00980961322784" rpy="-0.00465814192854 0.00824846908983 -1.59513247343" connected_to="world"/>
 <!-- BODY END -->
 </robot>

Commit message: online ongoing

File: eTaSL/robots/custom_robots.urdf (robot description, URDF)
Before this commit: robot custom_robots, 21 links, 20 joints
Joints:
- joint indy0_joint_world: origin xyz=-0.448628753424 0.0491750836372 0.0126187205315 rpy=-0.00559553685673 0.00815772775075 -1.5689325988 -> xyz=-0.449295699596 0.0486089587212 0.0127248167992 rpy=-0.00446359041577 0.00744673905369 -1.56694697228
- joint panda1_joint_world: origin xyz=0.51068854332 -0.0208044052124 0.00980961322784 rpy=-0.00465814192854 0.00824846908983 -1.59513247343 -> xyz=0.51137304306 -0.0204440951347 0.0105627775192 rpy=-0.00212708854677 0.00322777206705 -1.59515759283

File: eTaSL/robots/custom_robots.urdf.xacro (robot description, xacro)
@@ -6,6 +6,6 @@
 <link name="world"/>
 <!-- BODY BEGIN -->
-<xacro:indy7_robot robot_id="0" xyz="-0.448628753424 0.0491750836372 0.0126187205315" rpy="-0.00559553685673 0.00815772775075 -1.5689325988" connected_to="world"/>
-<xacro:panda_robot robot_id="1" xyz="0.51068854332 -0.0208044052124 0.00980961322784" rpy="-0.00465814192854 0.00824846908983 -1.59513247343" connected_to="world"/>
+<xacro:indy7_robot robot_id="0" xyz="-0.449295699596 0.0486089587212 0.0127248167992" rpy="-0.00446359041577 0.00744673905369 -1.56694697228" connected_to="world"/>
+<xacro:panda_robot robot_id="1" xyz="0.51137304306 -0.0204440951347 0.0105627775192" rpy="-0.00212708854677 0.00322777206705 -1.59515759283" connected_to="world"/>
 <!-- BODY END -->
 </robot>

Commit message: tested single object online handling

File: eTaSL/robots/custom_robots.urdf (robot description, URDF)
Before this commit: robot custom_robots, 21 links, 20 joints
Joints:
- joint indy0_joint_world: origin xyz=-0.449295699596 0.0486089587212 0.0127248167992 rpy=-0.00446359041577 0.00744673905369 -1.56694697228 -> xyz=-0.448984235525 0.0514437556267 0.0101051330566 rpy=-0.00502190446694 0.00910233737794 -1.57059582055
- joint panda1_joint_world: origin xyz=0.51137304306 -0.0204440951347 0.0105627775192 rpy=-0.00212708854677 0.00322777206705 -1.59515759283 -> xyz=0.509574532509 -0.0179131031036 0.010754108429 rpy=0.00301585594593 0.0083009924695 -1.59531413455

File: eTaSL/robots/custom_robots.urdf.xacro (robot description, xacro)
@@ -6,6 +6,6 @@
 <link name="world"/>
 <!-- BODY BEGIN -->
-<xacro:indy7_robot robot_id="0" xyz="-0.449295699596 0.0486089587212 0.0127248167992" rpy="-0.00446359041577 0.00744673905369 -1.56694697228" connected_to="world"/>
-<xacro:panda_robot robot_id="1" xyz="0.51137304306 -0.0204440951347 0.0105627775192" rpy="-0.00212708854677 0.00322777206705 -1.59515759283" connected_to="world"/>
+<xacro:indy7_robot robot_id="0" xyz="-0.448984235525 0.0514437556267 0.0101051330566" rpy="-0.00502190446694 0.00910233737794 -1.57059582055" connected_to="world"/>
+<xacro:panda_robot robot_id="1" xyz="0.509574532509 -0.0179131031036 0.010754108429" rpy="0.00301585594593 0.0083009924695 -1.59531413455" connected_to="world"/>
 <!-- BODY END -->
 </robot>

Commit message: onestep online execution tested

File: eTaSL/robots/custom_robots.urdf (robot description, URDF)
Before this commit: robot custom_robots, 21 links, 20 joints
Joints:
- joint indy0_joint_world: origin xyz=-0.448984235525 0.0514437556267 0.0101051330566 rpy=-0.00502190446694 0.00910233737794 -1.57059582055 -> xyz=-0.449337929487 0.050374686718 0.0131216645241 rpy=-0.00696492979457 0.00859379540227 -1.57054465153
- joint panda1_joint_world: origin xyz=0.509574532509 -0.0179131031036 0.010754108429 rpy=0.00301585594593 0.0083009924695 -1.59531413455 -> xyz=0.510402739048 -0.0169289112091 0.0088187456131 rpy=-0.00362093238276 0.00786177695094 -1.59182997756

File: eTaSL/robots/custom_robots.urdf.xacro (robot description, xacro)
@@ -6,6 +6,6 @@
 <link name="world"/>
 <!-- BODY BEGIN -->
-<xacro:indy7_robot robot_id="0" xyz="-0.448984235525 0.0514437556267 0.0101051330566" rpy="-0.00502190446694 0.00910233737794 -1.57059582055" connected_to="world"/>
-<xacro:panda_robot robot_id="1" xyz="0.509574532509 -0.0179131031036 0.010754108429" rpy="0.00301585594593 0.0083009924695 -1.59531413455" connected_to="world"/>
+<xacro:indy7_robot robot_id="0" xyz="-0.449337929487 0.050374686718 0.0131216645241" rpy="-0.00696492979457 0.00859379540227 -1.57054465153" connected_to="world"/>
+<xacro:panda_robot robot_id="1" xyz="0.510402739048 -0.0169289112091 0.0088187456131" rpy="-0.00362093238276 0.00786177695094 -1.59182997756" connected_to="world"/>
 <!-- BODY END -->
 </robot>

Commit message: dual robot process all tested, minor practical issues

File: eTaSL/robots/custom_robots.urdf (robot description, URDF)
Before this commit: robot custom_robots, 21 links, 20 joints
Joints:
- joint indy0_joint_world: origin xyz=-0.449337929487 0.050374686718 0.0131216645241 rpy=-0.00696492979457 0.00859379540227 -1.57054465153 -> xyz=-0.450414001942 0.063992023468 0.00961089134216 rpy=-0.00240906491853 0.0122450997011 -1.56613393589
- joint panda1_joint1: limit lower=-2.8973 upper=2.8973 effort=3.141592653589793 velocity=1.3089969389957472 -> lower=-2.75 upper=2.75 effort=3.141592653589793 velocity=1.3089969389957472
- joint panda1_joint5: limit lower=-2.8973 upper=2.8973 effort=3.141592653589793 velocity=1.5707963267948966 -> lower=-2.75 upper=2.75 effort=3.141592653589793 velocity=1.5707963267948966
- joint panda1_joint6: limit lower=-0.0175 upper=3.7525 effort=3.141592653589793 velocity=1.5707963267948966 -> lower=0.1 upper=3.6 effort=3.141592653589793 velocity=1.5707963267948966
- joint panda1_joint7: limit lower=-2.8973 upper=2.8973 effort=3.141592653589793 velocity=1.5707963267948966 -> lower=-2.75 upper=2.75 effort=3.141592653589793 velocity=1.5707963267948966
- joint panda1_joint_world: origin xyz=0.510402739048 -0.0169289112091 0.0088187456131 rpy=-0.00362093238276 0.00786177695094 -1.59182997756 -> xyz=0.510338068008 -0.00296866893768 0.0124877095222 rpy=-0.00118356485613 0.0103462362728 -1.58600016203

File: eTaSL/robots/custom_robots.urdf.xacro (robot description, xacro)
@@ -6,6 +6,6 @@
 <link name="world"/>
 <!-- BODY BEGIN -->
-<xacro:indy7_robot robot_id="0" xyz="-0.449337929487 0.050374686718 0.0131216645241" rpy="-0.00696492979457 0.00859379540227 -1.57054465153" connected_to="world"/>
-<xacro:panda_robot robot_id="1" xyz="0.510402739048 -0.0169289112091 0.0088187456131" rpy="-0.00362093238276 0.00786177695094 -1.59182997756" connected_to="world"/>
+<xacro:indy7_robot robot_id="0" xyz="-0.450414001942 0.063992023468 0.00961089134216" rpy="-0.00240906491853 0.0122450997011 -1.56613393589" connected_to="world"/>
+<xacro:panda_robot robot_id="1" xyz="0.510338068008 -0.00296866893768 0.0124877095222" rpy="-0.00118356485613 0.0103462362728 -1.58600016203" connected_to="world"/>
 <!-- BODY END -->
 </robot>

Commit message: threaded rviz visualization

File: eTaSL/robots/custom_robots.urdf (robot description, URDF)
Before this commit: robot custom_robots, 21 links, 20 joints
Joints:
- joint indy0_joint_world: origin xyz=-0.450414001942 0.063992023468 0.00961089134216 rpy=-0.00240906491853 0.0122450997011 -1.56613393589 -> xyz=-0.449715226889 0.0631829500198 0.0107617974281 rpy=-0.00316313563019 0.00660850819119 -1.56665778053
- joint panda1_joint_world: origin xyz=0.510338068008 -0.00296866893768 0.0124877095222 rpy=-0.00118356485613 0.0103462362728 -1.58600016203 -> xyz=0.511348485947 -0.00281500816345 0.0128458142281 rpy=-0.000780244967974 0.00471957512415 -1.58585239251

File: eTaSL/robots/custom_robots.urdf.xacro (robot description, xacro)
@@ -6,6 +6,6 @@
 <link name="world"/>
 <!-- BODY BEGIN -->
-<xacro:indy7_robot robot_id="0" xyz="-0.450414001942 0.063992023468 0.00961089134216" rpy="-0.00240906491853 0.0122450997011 -1.56613393589" connected_to="world"/>
-<xacro:panda_robot robot_id="1" xyz="0.510338068008 -0.00296866893768 0.0124877095222" rpy="-0.00118356485613 0.0103462362728 -1.58600016203" connected_to="world"/>
+<xacro:indy7_robot robot_id="0" xyz="-0.449715226889 0.0631829500198 0.0107617974281" rpy="-0.00316313563019 0.00660850819119 -1.56665778053" connected_to="world"/>
+<xacro:panda_robot robot_id="1" xyz="0.511348485947 -0.00281500816345 0.0128458142281" rpy="-0.000780244967974 0.00471957512415 -1.58585239251" connected_to="world"/>
 <!-- BODY END -->
 </robot>

Commit message: dual arm handover tested once

File: eTaSL/robots/custom_robots.urdf (robot description, URDF)
Before this commit: robot custom_robots, 21 links, 20 joints
Joints:
- joint indy0_joint_world: origin xyz=-0.449715226889 0.0631829500198 0.0107617974281 rpy=-0.00316313563019 0.00660850819119 -1.56665778053 -> xyz=-0.415481477976 0.255269497633 0.00683271884918 rpy=0.00328284253678 0.0106098371168 -1.52924587389
- joint panda1_joint_world: origin xyz=0.511348485947 -0.00281500816345 0.0128458142281 rpy=-0.000780244967974 0.00471957512415 -1.58585239251 -> xyz=0.54721313715 0.222797244787 0.0159376859665 rpy=0.00477876945711 0.00584773772488 -1.54915548774

File: eTaSL/robots/custom_robots.urdf.xacro (robot description, xacro)
@@ -6,6 +6,6 @@
 <link name="world"/>
 <!-- BODY BEGIN -->
-<xacro:indy7_robot robot_id="0" xyz="-0.449715226889 0.0631829500198 0.0107617974281" rpy="-0.00316313563019 0.00660850819119 -1.56665778053" connected_to="world"/>
-<xacro:panda_robot robot_id="1" xyz="0.511348485947 -0.00281500816345 0.0128458142281" rpy="-0.000780244967974 0.00471957512415 -1.58585239251" connected_to="world"/>
+<xacro:indy7_robot robot_id="0" xyz="-0.415481477976 0.255269497633 0.00683271884918" rpy="0.00328284253678 0.0106098371168 -1.52924587389" connected_to="world"/>
+<xacro:panda_robot robot_id="1" xyz="0.54721313715 0.222797244787 0.0159376859665" rpy="0.00477876945711 0.00584773772488 -1.54915548774" connected_to="world"/>
 <!-- BODY END -->
 </robot>
