Commit message: test done, remaining problem - singularity, vac offset

File: eTaSL/robots/custom_robots.urdf (robot description, URDF)
Before this commit: robot custom_robots, 21 links, 20 joints
Joints:
- joint indy0_joint_world: origin xyz=-0.415481477976 0.255269497633 0.00683271884918 rpy=0.00328284253678 0.0106098371168 -1.52924587389 -> xyz=-0.398579478264 0.333458960056 0.00808799266815 rpy=0.000299221039608 0.00837094631134 -1.55107055888
- joint panda1_joint2: limit lower=-1.7628 upper=1.7628 effort=3.141592653589793 velocity=1.3089969389957472 -> lower=-1.7 upper=1.7 effort=3.141592653589793 velocity=1.3089969389957472
- joint panda1_joint3: limit lower=-2.8973 upper=2.8973 effort=3.141592653589793 velocity=1.3089969389957472 -> lower=-2.75 upper=2.75 effort=3.141592653589793 velocity=1.3089969389957472
- joint panda1_joint4: limit lower=-3.0718 upper=-0.0698 effort=3.141592653589793 velocity=1.3089969389957472 -> lower=-2.9 upper=-0.1 effort=3.141592653589793 velocity=1.3089969389957472
- joint panda1_joint_world: origin xyz=0.54721313715 0.222797244787 0.0159376859665 rpy=0.00477876945711 0.00584773772488 -1.54915548774 -> xyz=0.564567565918 0.27959227562 0.0143544077873 rpy=-0.000821830428254 0.00567495683607 -1.56992275006

File: eTaSL/robots/custom_robots.urdf.xacro (robot description, xacro)
@@ -6,6 +6,6 @@
 <link name="world"/>
 <!-- BODY BEGIN -->
-<xacro:indy7_robot robot_id="0" xyz="-0.415481477976 0.255269497633 0.00683271884918" rpy="0.00328284253678 0.0106098371168 -1.52924587389" connected_to="world"/>
-<xacro:panda_robot robot_id="1" xyz="0.54721313715 0.222797244787 0.0159376859665" rpy="0.00477876945711 0.00584773772488 -1.54915548774" connected_to="world"/>
+<xacro:indy7_robot robot_id="0" xyz="-0.398579478264 0.333458960056 0.00808799266815" rpy="0.000299221039608 0.00837094631134 -1.55107055888" connected_to="world"/>
+<xacro:panda_robot robot_id="1" xyz="0.564567565918 0.27959227562 0.0143544077873" rpy="-0.000821830428254 0.00567495683607 -1.56992275006" connected_to="world"/>
 <!-- BODY END -->
 </robot>

Commit message: openGJK

File: eTaSL/robots/custom_robots.urdf (robot description, URDF)
Before this commit: robot custom_robots, 21 links, 20 joints
Joints:
- joint indy0_joint_world: origin xyz=-0.398579478264 0.333458960056 0.00808799266815 rpy=0.000299221039608 0.00837094631134 -1.55107055888 -> xyz=-0.398447275162 0.333022654057 -0.00535577535629 rpy=0.0181478442646 0.00132442069801 -1.55469574894
- joint panda1_joint_world: origin xyz=0.564567565918 0.27959227562 0.0143544077873 rpy=-0.000821830428254 0.00567495683607 -1.56992275006 -> xyz=0.565165519714 0.277357816696 0.0177581906319 rpy=0.0281038894439 -0.00787265079725 -1.5814208671

File: eTaSL/robots/custom_robots.urdf.xacro (robot description, xacro)
@@ -6,6 +6,6 @@
 <link name="world"/>
 <!-- BODY BEGIN -->
-<xacro:indy7_robot robot_id="0" xyz="-0.398579478264 0.333458960056 0.00808799266815" rpy="0.000299221039608 0.00837094631134 -1.55107055888" connected_to="world"/>
-<xacro:panda_robot robot_id="1" xyz="0.564567565918 0.27959227562 0.0143544077873" rpy="-0.000821830428254 0.00567495683607 -1.56992275006" connected_to="world"/>
+<xacro:indy7_robot robot_id="0" xyz="-0.398447275162 0.333022654057 -0.00535577535629" rpy="0.0181478442646 0.00132442069801 -1.55469574894" connected_to="world"/>
+<xacro:panda_robot robot_id="1" xyz="0.565165519714 0.277357816696 0.0177581906319" rpy="0.0281038894439 -0.00787265079725 -1.5814208671" connected_to="world"/>
 <!-- BODY END -->
 </robot>

Commit message: added swept volume test for joint move

File: eTaSL/robots/custom_robots.urdf (robot description, URDF)
Before this commit: robot custom_robots, 21 links, 20 joints
Joints:
- joint indy0_joint_world: origin xyz=-0.398447275162 0.333022654057 -0.00535577535629 rpy=0.0181478442646 0.00132442069801 -1.55469574894 -> xyz=-0.446902781725 0.281177520752 0.00863087177277 rpy=0.000503793281712 0.0107447201587 -1.57753520299
- joint panda1_joint_world: origin xyz=0.565165519714 0.277357816696 0.0177581906319 rpy=0.0281038894439 -0.00787265079725 -1.5814208671 -> xyz=0.513609230518 0.202775776386 0.0151824355125 rpy=0.00165491754746 0.00960060808645 -1.59814087216

File: eTaSL/robots/custom_robots.urdf.xacro (robot description, xacro)
@@ -6,6 +6,6 @@
 <link name="world"/>
 <!-- BODY BEGIN -->
-<xacro:indy7_robot robot_id="0" xyz="-0.398447275162 0.333022654057 -0.00535577535629" rpy="0.0181478442646 0.00132442069801 -1.55469574894" connected_to="world"/>
-<xacro:panda_robot robot_id="1" xyz="0.565165519714 0.277357816696 0.0177581906319" rpy="0.0281038894439 -0.00787265079725 -1.5814208671" connected_to="world"/>
+<xacro:indy7_robot robot_id="0" xyz="-0.446902781725 0.281177520752 0.00863087177277" rpy="0.000503793281712 0.0107447201587 -1.57753520299" connected_to="world"/>
+<xacro:panda_robot robot_id="1" xyz="0.513609230518 0.202775776386 0.0151824355125" rpy="0.00165491754746 0.00960060808645 -1.59814087216" connected_to="world"/>
 <!-- BODY END -->
 </robot>

Commit message: misc optimization

File: eTaSL/robots/custom_robots.urdf (robot description, URDF)
Before this commit: robot custom_robots, 21 links, 20 joints
Joints:
- joint indy0_joint_world: origin xyz=-0.446902781725 0.281177520752 0.00863087177277 rpy=0.000503793281712 0.0107447201587 -1.57753520299 -> xyz=-0.446954458952 0.281213283539 0.00830286741257 rpy=-1.90004858101e-05 0.00922117342013 -1.57713749711
- joint panda1_joint_world: origin xyz=0.513609230518 0.202775776386 0.0151824355125 rpy=0.00165491754746 0.00960060808645 -1.59814087216 -> xyz=0.513459861279 0.202846288681 0.0148251652718 rpy=0.00274363515123 0.00941330725316 -1.59848809756

File: eTaSL/robots/custom_robots.urdf.xacro (robot description, xacro)
@@ -6,6 +6,6 @@
 <link name="world"/>
 <!-- BODY BEGIN -->
-<xacro:indy7_robot robot_id="0" xyz="-0.446902781725 0.281177520752 0.00863087177277" rpy="0.000503793281712 0.0107447201587 -1.57753520299" connected_to="world"/>
-<xacro:panda_robot robot_id="1" xyz="0.513609230518 0.202775776386 0.0151824355125" rpy="0.00165491754746 0.00960060808645 -1.59814087216" connected_to="world"/>
+<xacro:indy7_robot robot_id="0" xyz="-0.446954458952 0.281213283539 0.00830286741257" rpy="-1.90004858101e-05 0.00922117342013 -1.57713749711" connected_to="world"/>
+<xacro:panda_robot robot_id="1" xyz="0.513459861279 0.202846288681 0.0148251652718" rpy="0.00274363515123 0.00941330725316 -1.59848809756" connected_to="world"/>
 <!-- BODY END -->
 </robot>

Commit message: arudo parameter update

File: eTaSL/robots/custom_robots.urdf (robot description, URDF)
Before this commit: robot custom_robots, 21 links, 20 joints
Joints:
- joint indy0_joint_world: origin xyz=-0.446954458952 0.281213283539 0.00830286741257 rpy=-1.90004858101e-05 0.00922117342013 -1.57713749711 -> xyz=-0.448677062988 0.283258587122 0.00913608074188 rpy=-0.000704484632721 0.0154524099057 -1.57827017697
- joint panda1_joint_world: origin xyz=0.513459861279 0.202846288681 0.0148251652718 rpy=0.00274363515123 0.00941330725316 -1.59848809756 -> xyz=0.513780832291 0.201571017504 0.0159308314323 rpy=-8.17645361403e-06 0.0124823842846 -1.59885212731

File: eTaSL/robots/custom_robots.urdf.xacro (robot description, xacro)
@@ -6,6 +6,6 @@
 <link name="world"/>
 <!-- BODY BEGIN -->
-<xacro:indy7_robot robot_id="0" xyz="-0.446954458952 0.281213283539 0.00830286741257" rpy="-1.90004858101e-05 0.00922117342013 -1.57713749711" connected_to="world"/>
-<xacro:panda_robot robot_id="1" xyz="0.513459861279 0.202846288681 0.0148251652718" rpy="0.00274363515123 0.00941330725316 -1.59848809756" connected_to="world"/>
+<xacro:indy7_robot robot_id="0" xyz="-0.448677062988 0.283258587122 0.00913608074188" rpy="-0.000704484632721 0.0154524099057 -1.57827017697" connected_to="world"/>
+<xacro:panda_robot robot_id="1" xyz="0.513780832291 0.201571017504 0.0159308314323" rpy="-8.17645361403e-06 0.0124823842846 -1.59885212731" connected_to="world"/>
 <!-- BODY END -->
 </robot>

Commit message: added binding matcher

File: eTaSL/robots/custom_robots.urdf (robot description, URDF)
Before this commit: robot custom_robots, 21 links, 20 joints
Joints:
- joint indy0_joint_world: origin xyz=-0.448677062988 0.283258587122 0.00913608074188 rpy=-0.000704484632721 0.0154524099057 -1.57827017697 -> xyz=-0.446637332439 0.281307071447 0.0100173950195 rpy=-0.00174475416079 0.0142583405311 -1.57746320792
- joint panda1_joint_world: origin xyz=0.513780832291 0.201571017504 0.0159308314323 rpy=-8.17645361403e-06 0.0124823842846 -1.59885212731 -> xyz=0.513214468956 0.203078538179 0.0138563513756 rpy=7.93323960496e-05 0.00979243683824 -1.59802948969

File: eTaSL/robots/custom_robots.urdf.xacro (robot description, xacro)
@@ -6,6 +6,6 @@
 <link name="world"/>
 <!-- BODY BEGIN -->
-<xacro:indy7_robot robot_id="0" xyz="-0.448677062988 0.283258587122 0.00913608074188" rpy="-0.000704484632721 0.0154524099057 -1.57827017697" connected_to="world"/>
-<xacro:panda_robot robot_id="1" xyz="0.513780832291 0.201571017504 0.0159308314323" rpy="-8.17645361403e-06 0.0124823842846 -1.59885212731" connected_to="world"/>
+<xacro:indy7_robot robot_id="0" xyz="-0.446637332439 0.281307071447 0.0100173950195" rpy="-0.00174475416079 0.0142583405311 -1.57746320792" connected_to="world"/>
+<xacro:panda_robot robot_id="1" xyz="0.513214468956 0.203078538179 0.0138563513756" rpy="7.93323960496e-05 0.00979243683824 -1.59802948969" connected_to="world"/>
 <!-- BODY END -->
 </robot>

Commit message: no cut dot

File: eTaSL/robots/custom_robots.urdf (robot description, URDF)
Before this commit: robot custom_robots, 21 links, 20 joints
Joints:
- joint indy0_joint_world: origin xyz=-0.446637332439 0.281307071447 0.0100173950195 rpy=-0.00174475416079 0.0142583405311 -1.57746320792 -> xyz=-0.447880357504 0.250642836094 0.00950443744659 rpy=-0.000968054148476 0.0128687964372 -1.58305426787
- joint panda1_joint_world: origin xyz=0.513214468956 0.203078538179 0.0138563513756 rpy=7.93323960496e-05 0.00979243683824 -1.59802948969 -> xyz=0.512257456779 0.167007505894 0.0140748023987 rpy=0.000771270407877 0.00837523026527 -1.60367098473

File: eTaSL/robots/custom_robots.urdf.xacro (robot description, xacro)
@@ -6,6 +6,6 @@
 <link name="world"/>
 <!-- BODY BEGIN -->
-<xacro:indy7_robot robot_id="0" xyz="-0.446637332439 0.281307071447 0.0100173950195" rpy="-0.00174475416079 0.0142583405311 -1.57746320792" connected_to="world"/>
-<xacro:panda_robot robot_id="1" xyz="0.513214468956 0.203078538179 0.0138563513756" rpy="7.93323960496e-05 0.00979243683824 -1.59802948969" connected_to="world"/>
+<xacro:indy7_robot robot_id="0" xyz="-0.447880357504 0.250642836094 0.00950443744659" rpy="-0.000968054148476 0.0128687964372 -1.58305426787" connected_to="world"/>
+<xacro:panda_robot robot_id="1" xyz="0.512257456779 0.167007505894 0.0140748023987" rpy="0.000771270407877 0.00837523026527 -1.60367098473" connected_to="world"/>
 <!-- BODY END -->
 </robot>

Commit message: new env operation checked

File: eTaSL/robots/custom_robots.urdf (robot description, URDF)
Before this commit: robot custom_robots, 21 links, 20 joints
Joints:
- joint indy0_joint_world: origin xyz=-0.447880357504 0.250642836094 0.00950443744659 rpy=-0.000968054148476 0.0128687964372 -1.58305426787 -> xyz=-0.446497768164 0.24981212616 0.0101870894432 rpy=-0.000723567818292 0.0127288557599 -1.582592677
- joint panda1_joint_world: origin xyz=0.512257456779 0.167007505894 0.0140748023987 rpy=0.000771270407877 0.00837523026527 -1.60367098473 -> xyz=0.511958360672 0.168226778507 0.0138182640076 rpy=0.00263808734626 0.00855548671309 -1.60338227502

File: eTaSL/robots/custom_robots.urdf.xacro (robot description, xacro)
@@ -6,6 +6,6 @@
 <link name="world"/>
 <!-- BODY BEGIN -->
-<xacro:indy7_robot robot_id="0" xyz="-0.447880357504 0.250642836094 0.00950443744659" rpy="-0.000968054148476 0.0128687964372 -1.58305426787" connected_to="world"/>
-<xacro:panda_robot robot_id="1" xyz="0.512257456779 0.167007505894 0.0140748023987" rpy="0.000771270407877 0.00837523026527 -1.60367098473" connected_to="world"/>
+<xacro:indy7_robot robot_id="0" xyz="-0.446497768164 0.24981212616 0.0101870894432" rpy="-0.000723567818292 0.0127288557599 -1.582592677" connected_to="world"/>
+<xacro:panda_robot robot_id="1" xyz="0.511958360672 0.168226778507 0.0138182640076" rpy="0.00263808734626 0.00855548671309 -1.60338227502" connected_to="world"/>
 <!-- BODY END -->
 </robot>

Commit message: agent number same as cpu number

File: eTaSL/robots/custom_robots.urdf (robot description, URDF)
Before this commit: robot custom_robots, 21 links, 20 joints
Joints:
- joint indy0_joint_world: origin xyz=-0.446497768164 0.24981212616 0.0101870894432 rpy=-0.000723567818292 0.0127288557599 -1.582592677 -> xyz=-0.447075515985 0.250340640545 0.00948196649551 rpy=-0.000999260999361 0.0112668280549 -1.58245623292
- joint panda1_joint_world: origin xyz=0.511958360672 0.168226778507 0.0138182640076 rpy=0.00263808734626 0.00855548671309 -1.60338227502 -> xyz=0.511685729027 0.168726027012 0.0136389732361 rpy=0.00114617009472 0.00808092808721 -1.60259305356

File: eTaSL/robots/custom_robots.urdf.xacro (robot description, xacro)
@@ -6,6 +6,6 @@
 <link name="world"/>
 <!-- BODY BEGIN -->
-<xacro:indy7_robot robot_id="0" xyz="-0.446497768164 0.24981212616 0.0101870894432" rpy="-0.000723567818292 0.0127288557599 -1.582592677" connected_to="world"/>
-<xacro:panda_robot robot_id="1" xyz="0.511958360672 0.168226778507 0.0138182640076" rpy="0.00263808734626 0.00855548671309 -1.60338227502" connected_to="world"/>
+<xacro:indy7_robot robot_id="0" xyz="-0.447075515985 0.250340640545 0.00948196649551" rpy="-0.000999260999361 0.0112668280549 -1.58245623292" connected_to="world"/>
+<xacro:panda_robot robot_id="1" xyz="0.511685729027 0.168726027012 0.0136389732361" rpy="0.00114617009472 0.00808092808721 -1.60259305356" connected_to="world"/>
 <!-- BODY END -->
 </robot>

Commit message: generalize online item, add joint vel constraint

File: eTaSL/robots/custom_robots.urdf (robot description, URDF)
Before this commit: robot custom_robots, 21 links, 20 joints
Joints:
- joint indy0_joint_world: origin xyz=-0.447075515985 0.250340640545 0.00948196649551 rpy=-0.000999260999361 0.0112668280549 -1.58245623292 -> xyz=-0.446847140789 0.250096917152 0.00919646024704 rpy=-0.000634488292781 0.012427471275 -1.58258260087
- joint panda1_joint_world: origin xyz=0.511685729027 0.168726027012 0.0136389732361 rpy=0.00114617009472 0.00808092808721 -1.60259305356 -> xyz=0.511754155159 0.168157100677 0.0138661265373 rpy=0.00340208155202 0.0120826607184 -1.60351256569

File: eTaSL/robots/custom_robots.urdf.xacro (robot description, xacro)
@@ -6,6 +6,6 @@
 <link name="world"/>
 <!-- BODY BEGIN -->
-<xacro:indy7_robot robot_id="0" xyz="-0.447075515985 0.250340640545 0.00948196649551" rpy="-0.000999260999361 0.0112668280549 -1.58245623292" connected_to="world"/>
-<xacro:panda_robot robot_id="1" xyz="0.511685729027 0.168726027012 0.0136389732361" rpy="0.00114617009472 0.00808092808721 -1.60259305356" connected_to="world"/>
+<xacro:indy7_robot robot_id="0" xyz="-0.446847140789 0.250096917152 0.00919646024704" rpy="-0.000634488292781 0.012427471275 -1.58258260087" connected_to="world"/>
+<xacro:panda_robot robot_id="1" xyz="0.511754155159 0.168157100677 0.0138661265373" rpy="0.00340208155202 0.0120826607184 -1.60351256569" connected_to="world"/>
 <!-- BODY END -->
 </robot>

Commit message: indy gripper applied

File: eTaSL/robots/custom_robots.urdf (robot description, URDF)
Before this commit: robot custom_robots, 21 links, 20 joints
Links:
- link indy0_link6: geometry collision cylinder length=0.25 radius=0.05; visual mesh filename=package://indy7_description/meshes/stl/Indy7_6.stl
Joints:
- joint indy0_joint_world: origin xyz=-0.446847140789 0.250096917152 0.00919646024704 rpy=-0.000634488292781 0.012427471275 -1.58258260087 -> xyz=-0.447144120932 0.252235591412 0.0095442533493 rpy=-0.000328128620623 0.0115290161139 -1.58381785638
- joint panda1_joint_world: origin xyz=0.511754155159 0.168157100677 0.0138661265373 rpy=0.00340208155202 0.0120826607184 -1.60351256569 -> xyz=0.511944293976 0.169146895409 0.0143564343452 rpy=0.00260427106974 0.0105923906964 -1.60387145407

File: eTaSL/robots/custom_robots.urdf.xacro (robot description, xacro)
@@ -6,6 +6,6 @@
 <link name="world"/>
 <!-- BODY BEGIN -->
-<xacro:indy7_robot robot_id="0" xyz="-0.446847140789 0.250096917152 0.00919646024704" rpy="-0.000634488292781 0.012427471275 -1.58258260087" connected_to="world"/>
-<xacro:panda_robot robot_id="1" xyz="0.511754155159 0.168157100677 0.0138661265373" rpy="0.00340208155202 0.0120826607184 -1.60351256569" connected_to="world"/>
+<xacro:indy7_robot robot_id="0" xyz="-0.447144120932 0.252235591412 0.0095442533493" rpy="-0.000328128620623 0.0115290161139 -1.58381785638" connected_to="world"/>
+<xacro:panda_robot robot_id="1" xyz="0.511944293976 0.169146895409 0.0143564343452" rpy="0.00260427106974 0.0105923906964 -1.60387145407" connected_to="world"/>
 <!-- BODY END -->
 </robot>

File: eTaSL/robots/indy7_robot.xacro (robot description, xacro)
@@ -141,7 +141,7 @@
 		</visual>
 		<collision>
-			<origin xyz="0 0 -0.054" rpy="0 0 0"/>
-			<geometry>
-				<cylinder length="0.218" radius="0.050"/>
+			<origin xyz="0 0 -0.038" rpy="0 0 0"/>
+			<geometry>
+				<cylinder length="0.25" radius="0.050"/>
 			</geometry>
 		</collision>

Commit message: add int-trajectory following

File: eTaSL/robots/custom_robots.urdf (robot description, URDF)
Before this commit: robot custom_robots, 21 links, 20 joints
Joints:
- joint indy0_joint_world: origin xyz=-0.447144120932 0.252235591412 0.0095442533493 rpy=-0.000328128620623 0.0115290161139 -1.58381785638 -> xyz=-0.446407794952 0.251397013664 0.0102092623711 rpy=-2.17016113899e-07 0.0128620837997 -1.58386984055
- joint panda1_joint_world: origin xyz=0.511944293976 0.169146895409 0.0143564343452 rpy=0.00260427106974 0.0105923906964 -1.60387145407 -> xyz=0.511913180351 0.169161915779 0.0142871141434 rpy=0.00272143505924 0.0108322837398 -1.60386662363

File: eTaSL/robots/custom_robots.urdf.xacro (robot description, xacro)
@@ -6,6 +6,6 @@
 <link name="world"/>
 <!-- BODY BEGIN -->
-<xacro:indy7_robot robot_id="0" xyz="-0.447144120932 0.252235591412 0.0095442533493" rpy="-0.000328128620623 0.0115290161139 -1.58381785638" connected_to="world"/>
-<xacro:panda_robot robot_id="1" xyz="0.511944293976 0.169146895409 0.0143564343452" rpy="0.00260427106974 0.0105923906964 -1.60387145407" connected_to="world"/>
+<xacro:indy7_robot robot_id="0" xyz="-0.446407794952 0.251397013664 0.0102092623711" rpy="-2.17016113899e-07 0.0128620837997 -1.58386984055" connected_to="world"/>
+<xacro:panda_robot robot_id="1" xyz="0.511913180351 0.169161915779 0.0142871141434" rpy="0.00272143505924 0.0108322837398 -1.60386662363" connected_to="world"/>
 <!-- BODY END -->
 </robot>

Commit message: geometry hierarchy cleaned

File: eTaSL/robots/custom_robots.urdf (robot description, URDF)
Before this commit: robot custom_robots, 21 links, 20 joints
Joints:
- joint indy0_joint_world: origin xyz=-0.446407794952 0.251397013664 0.0102092623711 rpy=-2.17016113899e-07 0.0128620837997 -1.58386984055 -> xyz=-0.446839213371 0.251892447472 0.00962364673615 rpy=-0.000221643092241 0.0127894207085 -1.58349226199
- joint panda1_joint_world: origin xyz=0.511913180351 0.169161915779 0.0142871141434 rpy=0.00272143505924 0.0108322837398 -1.60386662363 -> xyz=0.511829197407 0.169160187244 0.0143783092499 rpy=0.00309285480819 0.0105787110691 -1.60372835817

File: eTaSL/robots/custom_robots.urdf.xacro (robot description, xacro)
@@ -6,6 +6,6 @@
 <link name="world"/>
 <!-- BODY BEGIN -->
-<xacro:indy7_robot robot_id="0" xyz="-0.446407794952 0.251397013664 0.0102092623711" rpy="-2.17016113899e-07 0.0128620837997 -1.58386984055" connected_to="world"/>
-<xacro:panda_robot robot_id="1" xyz="0.511913180351 0.169161915779 0.0142871141434" rpy="0.00272143505924 0.0108322837398 -1.60386662363" connected_to="world"/>
+<xacro:indy7_robot robot_id="0" xyz="-0.446839213371 0.251892447472 0.00962364673615" rpy="-0.000221643092241 0.0127894207085 -1.58349226199" connected_to="world"/>
+<xacro:panda_robot robot_id="1" xyz="0.511829197407 0.169160187244 0.0143783092499" rpy="0.00309285480819 0.0105787110691 -1.60372835817" connected_to="world"/>
 <!-- BODY END -->
 </robot>

Commit message: etasl planning packaged (not online)

File: eTaSL/robots/custom_robots.urdf (robot description, URDF)
Before this commit: robot custom_robots, 21 links, 20 joints
Joints:
- joint indy0_joint_world: origin xyz=-0.446839213371 0.251892447472 0.00962364673615 rpy=-0.000221643092241 0.0127894207085 -1.58349226199 -> xyz=-0.447407871485 0.252505540848 0.00936406850815 rpy=-8.29578625356e-05 0.0128187767105 -1.58374292425
- joint panda1_joint_world: origin xyz=0.511829197407 0.169160187244 0.0143783092499 rpy=0.00309285480819 0.0105787110691 -1.60372835817 -> xyz=0.511892914772 0.16920042038 0.0142872333527 rpy=0.00272208513882 0.0104494805971 -1.60373832782

File: eTaSL/robots/custom_robots.urdf.xacro (robot description, xacro)
@@ -6,6 +6,6 @@
 <link name="world"/>
 <!-- BODY BEGIN -->
-<xacro:indy7_robot robot_id="0" xyz="-0.446839213371 0.251892447472 0.00962364673615" rpy="-0.000221643092241 0.0127894207085 -1.58349226199" connected_to="world"/>
-<xacro:panda_robot robot_id="1" xyz="0.511829197407 0.169160187244 0.0143783092499" rpy="0.00309285480819 0.0105787110691 -1.60372835817" connected_to="world"/>
+<xacro:indy7_robot robot_id="0" xyz="-0.447407871485 0.252505540848 0.00936406850815" rpy="-8.29578625356e-05 0.0128187767105 -1.58374292425" connected_to="world"/>
+<xacro:panda_robot robot_id="1" xyz="0.511892914772 0.16920042038 0.0142872333527" rpy="0.00272208513882 0.0104494805971 -1.60373832782" connected_to="world"/>
 <!-- BODY END -->
 </robot>
