Commit message: online planning separated

File: eTaSL/robots/custom_robots.urdf (robot description, URDF)
Before this commit: robot custom_robots, 21 links, 20 joints
Joints:
- joint indy0_joint_world: origin xyz=-0.447407871485 0.252505540848 0.00936406850815 rpy=-8.29578625356e-05 0.0128187767105 -1.58374292425 -> xyz=-0.447512328625 0.252558410168 0.00948530435562 rpy=-0.000463986218909 0.0127358003948 -1.58367656815
- joint panda1_joint_world: origin xyz=0.511892914772 0.16920042038 0.0142872333527 rpy=0.00272208513882 0.0104494805971 -1.60373832782 -> xyz=0.511829257011 0.169106900692 0.0143933296204 rpy=0.00281619112069 0.010968875249 -1.603940525

File: eTaSL/robots/custom_robots.urdf.xacro (robot description, xacro)
@@ -6,6 +6,6 @@
 <link name="world"/>
 <!-- BODY BEGIN -->
-<xacro:indy7_robot robot_id="0" xyz="-0.447407871485 0.252505540848 0.00936406850815" rpy="-8.29578625356e-05 0.0128187767105 -1.58374292425" connected_to="world"/>
-<xacro:panda_robot robot_id="1" xyz="0.511892914772 0.16920042038 0.0142872333527" rpy="0.00272208513882 0.0104494805971 -1.60373832782" connected_to="world"/>
+<xacro:indy7_robot robot_id="0" xyz="-0.447512328625 0.252558410168 0.00948530435562" rpy="-0.000463986218909 0.0127358003948 -1.58367656815" connected_to="world"/>
+<xacro:panda_robot robot_id="1" xyz="0.511829257011 0.169106900692 0.0143933296204" rpy="0.00281619112069 0.010968875249 -1.603940525" connected_to="world"/>
 <!-- BODY END -->
 </robot>

Commit message: packaged

File: eTaSL/robots/custom_robots.urdf (robot description, URDF)
Before this commit: robot custom_robots, 21 links, 20 joints
Joints:
- joint indy0_joint_world: origin xyz=-0.447512328625 0.252558410168 0.00948530435562 rpy=-0.000463986218909 0.0127358003948 -1.58367656815 -> xyz=-0.446431159973 0.251623213291 0.00984662771225 rpy=-0.000115271915586 0.011570294712 -1.58406070544
- joint panda1_joint_world: origin xyz=0.511829257011 0.169106900692 0.0143933296204 rpy=0.00281619112069 0.010968875249 -1.603940525 -> xyz=0.511838555336 0.16913831234 0.0143668651581 rpy=0.00224158799323 0.00993735963386 -1.60357374038

File: eTaSL/robots/custom_robots.urdf.xacro (robot description, xacro)
@@ -6,6 +6,6 @@
 <link name="world"/>
 <!-- BODY BEGIN -->
-<xacro:indy7_robot robot_id="0" xyz="-0.447512328625 0.252558410168 0.00948530435562" rpy="-0.000463986218909 0.0127358003948 -1.58367656815" connected_to="world"/>
-<xacro:panda_robot robot_id="1" xyz="0.511829257011 0.169106900692 0.0143933296204" rpy="0.00281619112069 0.010968875249 -1.603940525" connected_to="world"/>
+<xacro:indy7_robot robot_id="0" xyz="-0.446431159973 0.251623213291 0.00984662771225" rpy="-0.000115271915586 0.011570294712 -1.58406070544" connected_to="world"/>
+<xacro:panda_robot robot_id="1" xyz="0.511838555336 0.16913831234 0.0143668651581" rpy="0.00224158799323 0.00993735963386 -1.60357374038" connected_to="world"/>
 <!-- BODY END -->
 </robot>

Commit message: sequential waypoint activation

File: eTaSL/robots/custom_robots.urdf (robot description, URDF)
Before this commit: robot custom_robots, 21 links, 20 joints
Links:
- link indy0_link3: geometry collision cylinder length=0.2 radius=0.065; visual mesh filename=package://indy7_description/meshes/stl/Indy7_3.stl
- link indy0_link4: geometry collision cylinder length=0.35 radius=0.06; visual mesh filename=package://indy7_description/meshes/stl/Indy7_4.stl
- link indy0_link6: geometry collision cylinder length=0.25 radius=0.06; visual mesh filename=package://indy7_description/meshes/stl/Indy7_6.stl
Joints:
- joint indy0_joint_world: origin xyz=-0.446431159973 0.251623213291 0.00984662771225 rpy=-0.000115271915586 0.011570294712 -1.58406070544 -> xyz=-0.44688218832 0.251997053623 0.0096560716629 rpy=0.000112986510724 0.0124107802243 -1.58381359361
- joint panda1_joint_world: origin xyz=0.511838555336 0.16913831234 0.0143668651581 rpy=0.00224158799323 0.00993735963386 -1.60357374038 -> xyz=0.511956453323 0.168998122215 0.0146180391312 rpy=0.00301172885219 0.0100915657917 -1.60411686047

File: eTaSL/robots/custom_robots.urdf.xacro (robot description, xacro)
@@ -6,6 +6,6 @@
 <link name="world"/>
 <!-- BODY BEGIN -->
-<xacro:indy7_robot robot_id="0" xyz="-0.446431159973 0.251623213291 0.00984662771225" rpy="-0.000115271915586 0.011570294712 -1.58406070544" connected_to="world"/>
-<xacro:panda_robot robot_id="1" xyz="0.511838555336 0.16913831234 0.0143668651581" rpy="0.00224158799323 0.00993735963386 -1.60357374038" connected_to="world"/>
+<xacro:indy7_robot robot_id="0" xyz="-0.44688218832 0.251997053623 0.0096560716629" rpy="0.000112986510724 0.0124107802243 -1.58381359361" connected_to="world"/>
+<xacro:panda_robot robot_id="1" xyz="0.511956453323 0.168998122215 0.0146180391312" rpy="0.00301172885219 0.0100915657917 -1.60411686047" connected_to="world"/>
 <!-- BODY END -->
 </robot>

File: eTaSL/robots/indy7_robot.xacro (robot description, xacro)
@@ -83,5 +83,5 @@
 			<origin xyz="0 0 0.03" rpy="0 0 0"/>
 			<geometry>
-				<cylinder length="0.2" radius="0.055"/>
+				<cylinder length="0.2" radius="0.065"/>
 			</geometry>
 		</collision>
@@ -103,5 +103,5 @@
 			<origin xyz="0 0 -0.092" rpy="0 0 0"/>
 			<geometry>
-				<cylinder length="0.35" radius="0.055"/>
+				<cylinder length="0.35" radius="0.06"/>
 			</geometry>
 		</collision>
@@ -143,5 +143,5 @@
 			<origin xyz="0 0 -0.038" rpy="0 0 0"/>
 			<geometry>
-				<cylinder length="0.25" radius="0.050"/>
+				<cylinder length="0.25" radius="0.06"/>
 			</geometry>
 		</collision>

Commit message: collision mesh code refined

File: eTaSL/robots/custom_robots.urdf (robot description, URDF)
Before this commit: robot custom_robots, 21 links, 20 joints
Links:
- link indy0_link0: geometry collision cylinder length=0.2 radius=0.05; visual mesh filename=package://indy7_description/meshes/stl/Indy7_0.stl
- link indy0_tcp: geometry collision cylinder length=0.08 radius=0.016; collision cylinder length=0.08 radius=0.016
- link panda1_hand: geometry collision cylinder length=0.14 radius=0.06; visual mesh filename=package://franka_description/meshes/visual/hand.dae
- link panda1_leftfinger: geometry collision cylinder length=0.0325 radius=0.018; visual mesh filename=package://franka_description/meshes/visual/finger.dae
- link panda1_link0: geometry collision cylinder length=0.102 radius=0.1; collision cylinder length=0.3 radius=0.05
- link panda1_link1: geometry collision cylinder length=0.132 radius=0.11; visual mesh filename=package://franka_description/meshes/visual/link1.dae
- link panda1_link2: geometry collision cylinder length=0.175 radius=0.09; visual mesh filename=package://franka_description/meshes/visual/link2.dae
- link panda1_link3: geometry collision cylinder length=0.12 radius=0.09; visual mesh filename=package://franka_description/meshes/visual/link3.dae
- link panda1_link4: geometry collision cylinder length=0.17 radius=0.08; visual mesh filename=package://franka_description/meshes/visual/link4.dae
- link panda1_link5: geometry collision cylinder length=0.238 radius=0.08; visual mesh filename=package://franka_description/meshes/visual/link5.dae
- link panda1_link6: geometry collision cylinder length=0.09 radius=0.09; visual mesh filename=package://franka_description/meshes/visual/link6.dae
- link panda1_link7: geometry visual mesh filename=package://franka_description/meshes/visual/link7.dae
- link panda1_rightfinger: geometry collision cylinder length=0.0325 radius=0.018; visual mesh filename=package://franka_description/meshes/visual/finger.dae
Joints:
- joint indy0_joint_world: origin xyz=-0.44688218832 0.251997053623 0.0096560716629 rpy=0.000112986510724 0.0124107802243 -1.58381359361 -> xyz=-0.446289390326 0.251102805138 0.0102017521858 rpy=-0.000417408398833 0.0117274232265 -1.58323164053
- joint panda1_joint_world: origin xyz=0.511956453323 0.168998122215 0.0146180391312 rpy=0.00301172885219 0.0100915657917 -1.60411686047 -> xyz=0.511917114258 0.169139146805 0.0143296122551 rpy=0.00296737500071 0.00948517817286 -1.60379212552

File: eTaSL/robots/custom_robots.urdf.xacro (robot description, xacro)
@@ -6,6 +6,6 @@
 <link name="world"/>
 <!-- BODY BEGIN -->
-<xacro:indy7_robot robot_id="0" xyz="-0.44688218832 0.251997053623 0.0096560716629" rpy="0.000112986510724 0.0124107802243 -1.58381359361" connected_to="world"/>
-<xacro:panda_robot robot_id="1" xyz="0.511956453323 0.168998122215 0.0146180391312" rpy="0.00301172885219 0.0100915657917 -1.60411686047" connected_to="world"/>
+<xacro:indy7_robot robot_id="0" xyz="-0.446289390326 0.251102805138 0.0102017521858" rpy="-0.000417408398833 0.0117274232265 -1.58323164053" connected_to="world"/>
+<xacro:panda_robot robot_id="1" xyz="0.511917114258 0.169139146805 0.0143296122551" rpy="0.00296737500071 0.00948517817286 -1.60379212552" connected_to="world"/>
 <!-- BODY END -->
 </robot>

File: eTaSL/robots/indy7_robot.xacro (robot description, xacro)
@@ -11,4 +11,5 @@
 	<xacro:property name="PI" value="3.1415926535897931"/>
 	<xacro:property name="indy_material" value="metal_grey"/>
+	<xacro:property name="tool_material" value="red"/>
 	<!-- <material name="grey"> <color rgba="0.5 0.5 0.5 1"/> </material> -->
 	<link name="indy${robot_id}_link0">
@@ -20,4 +21,10 @@
 			<material name="${indy_material}"/>
 		</visual>
+		<collision>
+			<origin xyz="-0.1   0.    0.03" rpy="-0.          1.57079633  0."/>
+			<geometry>
+				<cylinder length="0.2" radius="0.05"/>
+			</geometry>
+		</collision>
 		<inertial>
 			<origin xyz="0 0 0" rpy="0 0 0"/>
@@ -152,5 +159,37 @@
 		</inertial>
 	</link>
-	<link name="indy${robot_id}_tcp"/>
+	<link name="indy${robot_id}_tcp">
+		<visual>
+			<origin xyz="0 0 0" rpy="0 0 1.570796"/>
+			<geometry>
+				<mesh filename="package://my_mesh/meshes/stl/indy_gripper_asm2_ctd.STL" scale="0.001 0.001 0.001"/>
+			</geometry>
+			<material name="${tool_material}"/>
+		</visual>
+		<collision>
+			<origin xyz="0.005 0.044 0.1" rpy="0 0 0"/>
+			<geometry>
+				<cylinder length="0.08" radius="0.016"/>
+			</geometry>
+		</collision>
+		<collision>
+			<origin xyz="-0.005  0.044  0.1" rpy="0 0 0"/>
+			<geometry>
+				<cylinder length="0.08" radius="0.016"/>
+			</geometry>
+		</collision>
+		<collision>
+			<origin xyz="0.005 -0.044  0.1" rpy="0 0 0"/>
+			<geometry>
+				<cylinder length="0.08" radius="0.016"/>
+			</geometry>
+		</collision>
+		<collision>
+			<origin xyz="-0.005 -0.044  0.1" rpy="0 0 0"/>
+			<geometry>
+				<cylinder length="0.08" radius="0.016"/>
+			</geometry>
+		</collision>
+	</link>
 	<joint name="indy${robot_id}_joint0" type="revolute">
 		<parent link="indy${robot_id}_link0"/>

File: eTaSL/robots/panda_robot.xacro (robot description, xacro)
@@ -2,6 +2,6 @@
 <robot xmlns:xacro="http://www.ros.org/wiki/xacro" name="panda">
   <xacro:macro name="panda_robot" params="robot_id:='0' xyz:='0 0 0' rpy:='0 0 0'  connected_to:=''">
-    <xacro:include filename="$(find franka_description)/robots/panda_arm.xacro"/>
-    <xacro:include filename="$(find franka_description)/robots/hand.xacro"/>
+    <xacro:include filename="$(env TAMP_ETASL_DIR)/robots/panda_arm.xacro"/>
+    <xacro:include filename="$(env TAMP_ETASL_DIR)/robots/hand.xacro"/>
     <xacro:panda_arm arm_id="panda${robot_id}" rpy="${rpy}" xyz="${xyz}" connected_to="${connected_to}"/>
     <xacro:hand ns="panda${robot_id}" rpy="0 0 ${-pi/4}" connected_to="panda${robot_id}_link8"/>

Commit message: add/remove geometry

File: eTaSL/robots/custom_robots.urdf (robot description, URDF)
Before this commit: robot custom_robots, 21 links, 20 joints
Joints:
- joint indy0_joint_world: origin xyz=-0.446289390326 0.251102805138 0.0102017521858 rpy=-0.000417408398833 0.0117274232265 -1.58323164053 -> xyz=-0.446444660425 0.251354336739 0.0101016163826 rpy=-0.000398831143589 0.0121609276968 -1.58361334748
- joint panda1_joint_world: origin xyz=0.511917114258 0.169139146805 0.0143296122551 rpy=0.00296737500071 0.00948517817286 -1.60379212552 -> xyz=0.511824667454 0.169109284878 0.014355301857 rpy=0.00285221566738 0.00993357506894 -1.60374202568

File: eTaSL/robots/custom_robots.urdf.xacro (robot description, xacro)
@@ -6,6 +6,6 @@
 <link name="world"/>
 <!-- BODY BEGIN -->
-<xacro:indy7_robot robot_id="0" xyz="-0.446289390326 0.251102805138 0.0102017521858" rpy="-0.000417408398833 0.0117274232265 -1.58323164053" connected_to="world"/>
-<xacro:panda_robot robot_id="1" xyz="0.511917114258 0.169139146805 0.0143296122551" rpy="0.00296737500071 0.00948517817286 -1.60379212552" connected_to="world"/>
+<xacro:indy7_robot robot_id="0" xyz="-0.446444660425 0.251354336739 0.0101016163826" rpy="-0.000398831143589 0.0121609276968 -1.58361334748" connected_to="world"/>
+<xacro:panda_robot robot_id="1" xyz="0.511824667454 0.169109284878 0.014355301857" rpy="0.00285221566738 0.00993357506894 -1.60374202568" connected_to="world"/>
 <!-- BODY END -->
 </robot>

Commit message: add/remove geometry/object

File: eTaSL/robots/custom_robots.urdf (robot description, URDF)
Before this commit: robot custom_robots, 21 links, 20 joints
Joints:
- joint indy0_joint_world: origin xyz=-0.446444660425 0.251354336739 0.0101016163826 rpy=-0.000398831143589 0.0121609276968 -1.58361334748 -> xyz=-0.446714758873 0.251704216003 0.00980758666992 rpy=-0.000296321109737 0.0118551048418 -1.58347059079
- joint panda1_joint_world: origin xyz=0.511824667454 0.169109284878 0.014355301857 rpy=0.00285221566738 0.00993357506894 -1.60374202568 -> xyz=0.511953771114 0.169003307819 0.0144295096397 rpy=0.00316326577134 0.0100679614536 -1.60417851098

File: eTaSL/robots/custom_robots.urdf.xacro (robot description, xacro)
@@ -6,6 +6,6 @@
 <link name="world"/>
 <!-- BODY BEGIN -->
-<xacro:indy7_robot robot_id="0" xyz="-0.446444660425 0.251354336739 0.0101016163826" rpy="-0.000398831143589 0.0121609276968 -1.58361334748" connected_to="world"/>
-<xacro:panda_robot robot_id="1" xyz="0.511824667454 0.169109284878 0.014355301857" rpy="0.00285221566738 0.00993357506894 -1.60374202568" connected_to="world"/>
+<xacro:indy7_robot robot_id="0" xyz="-0.446714758873 0.251704216003 0.00980758666992" rpy="-0.000296321109737 0.0118551048418 -1.58347059079" connected_to="world"/>
+<xacro:panda_robot robot_id="1" xyz="0.511953771114 0.169003307819 0.0144295096397" rpy="0.00316326577134 0.0100679614536 -1.60417851098" connected_to="world"/>
 <!-- BODY END -->
 </robot>

Commit message: binder availability check added

File: eTaSL/robots/custom_robots.urdf (robot description, URDF)
Before this commit: robot custom_robots, 21 links, 20 joints
Joints:
- joint indy0_joint_world: origin xyz=-0.446714758873 0.251704216003 0.00980758666992 rpy=-0.000296321109737 0.0118551048418 -1.58347059079 -> xyz=-0.446644991636 0.251748383045 0.00969982147217 rpy=-0.000271692878386 0.0117162761169 -1.58346710702
- joint panda1_joint_world: origin xyz=0.511953771114 0.169003307819 0.0144295096397 rpy=0.00316326577134 0.0100679614536 -1.60417851098 -> xyz=0.511959433556 0.16899561882 0.0144457221031 rpy=0.002842357247 0.00929103684367 -1.60402505824

File: eTaSL/robots/custom_robots.urdf.xacro (robot description, xacro)
@@ -6,6 +6,6 @@
 <link name="world"/>
 <!-- BODY BEGIN -->
-<xacro:indy7_robot robot_id="0" xyz="-0.446714758873 0.251704216003 0.00980758666992" rpy="-0.000296321109737 0.0118551048418 -1.58347059079" connected_to="world"/>
-<xacro:panda_robot robot_id="1" xyz="0.511953771114 0.169003307819 0.0144295096397" rpy="0.00316326577134 0.0100679614536 -1.60417851098" connected_to="world"/>
+<xacro:indy7_robot robot_id="0" xyz="-0.446644991636 0.251748383045 0.00969982147217" rpy="-0.000271692878386 0.0117162761169 -1.58346710702" connected_to="world"/>
+<xacro:panda_robot robot_id="1" xyz="0.511959433556 0.16899561882 0.0144457221031" rpy="0.002842357247 0.00929103684367 -1.60402505824" connected_to="world"/>
 <!-- BODY END -->
 </robot>

Commit message: binder registering

File: eTaSL/robots/custom_robots.urdf (robot description, URDF)
Before this commit: robot custom_robots, 21 links, 20 joints
Joints:
- joint indy0_joint_world: origin xyz=-0.446644991636 0.251748383045 0.00969982147217 rpy=-0.000271692878386 0.0117162761169 -1.58346710702 -> xyz=-0.44746735692 0.252653777599 0.00912934541702 rpy=-0.000108813423242 0.0120797112477 -1.58356838782
- joint panda1_joint_world: origin xyz=0.511959433556 0.16899561882 0.0144457221031 rpy=0.002842357247 0.00929103684367 -1.60402505824 -> xyz=0.512002706528 0.168995440006 0.014458835125 rpy=0.00305518093518 0.00958716682748 -1.60397746828

File: eTaSL/robots/custom_robots.urdf.xacro (robot description, xacro)
@@ -6,6 +6,6 @@
 <link name="world"/>
 <!-- BODY BEGIN -->
-<xacro:indy7_robot robot_id="0" xyz="-0.446644991636 0.251748383045 0.00969982147217" rpy="-0.000271692878386 0.0117162761169 -1.58346710702" connected_to="world"/>
-<xacro:panda_robot robot_id="1" xyz="0.511959433556 0.16899561882 0.0144457221031" rpy="0.002842357247 0.00929103684367 -1.60402505824" connected_to="world"/>
+<xacro:indy7_robot robot_id="0" xyz="-0.44746735692 0.252653777599 0.00912934541702" rpy="-0.000108813423242 0.0120797112477 -1.58356838782" connected_to="world"/>
+<xacro:panda_robot robot_id="1" xyz="0.512002706528 0.168995440006 0.014458835125" rpy="0.00305518093518 0.00958716682748 -1.60397746828" connected_to="world"/>
 <!-- BODY END -->
 </robot>

Commit message: init search, build graph optimized

File: eTaSL/robots/custom_robots.urdf (robot description, URDF)
Before this commit: robot custom_robots, 21 links, 20 joints
Joints:
- joint indy0_joint_world: origin xyz=-0.44746735692 0.252653777599 0.00912934541702 rpy=-0.000108813423242 0.0120797112477 -1.58356838782 -> xyz=-0.447554945946 0.252621471882 0.00895714759827 rpy=0.000218331973274 0.0113785043803 -1.58362463673
- joint panda1_joint_world: origin xyz=0.512002706528 0.168995440006 0.014458835125 rpy=0.00305518093518 0.00958716682748 -1.60397746828 -> xyz=0.512020647526 0.169103205204 0.0144633054733 rpy=0.00347274780491 0.00851996101077 -1.6038241594

File: eTaSL/robots/custom_robots.urdf.xacro (robot description, xacro)
@@ -6,6 +6,6 @@
 <link name="world"/>
 <!-- BODY BEGIN -->
-<xacro:indy7_robot robot_id="0" xyz="-0.44746735692 0.252653777599 0.00912934541702" rpy="-0.000108813423242 0.0120797112477 -1.58356838782" connected_to="world"/>
-<xacro:panda_robot robot_id="1" xyz="0.512002706528 0.168995440006 0.014458835125" rpy="0.00305518093518 0.00958716682748 -1.60397746828" connected_to="world"/>
+<xacro:indy7_robot robot_id="0" xyz="-0.447554945946 0.252621471882 0.00895714759827" rpy="0.000218331973274 0.0113785043803 -1.58362463673" connected_to="world"/>
+<xacro:panda_robot robot_id="1" xyz="0.512020647526 0.169103205204 0.0144633054733" rpy="0.00347274780491 0.00851996101077 -1.6038241594" connected_to="world"/>
 <!-- BODY END -->
 </robot>

Commit message: add: table view

File: eTaSL/robots/custom_robots.urdf (robot description, URDF)
Before this commit: robot custom_robots, 21 links, 20 joints
Joints:
- joint indy0_joint_world: origin xyz=-0.447554945946 0.252621471882 0.00895714759827 rpy=0.000218331973274 0.0113785043803 -1.58362463673 -> xyz=-0.447089582682 0.251743137836 0.00930815935135 rpy=-0.000777551145325 0.0099242762868 -1.58336192744
- joint panda1_joint_world: origin xyz=0.512020647526 0.169103205204 0.0144633054733 rpy=0.00347274780491 0.00851996101077 -1.6038241594 -> xyz=0.511796474457 0.169063687325 0.0137922167778 rpy=0.00260240796696 0.00891747931083 -1.60378843737

File: eTaSL/robots/custom_robots.urdf.xacro (robot description, xacro)
@@ -6,6 +6,6 @@
 <link name="world"/>
 <!-- BODY BEGIN -->
-<xacro:indy7_robot robot_id="0" xyz="-0.447554945946 0.252621471882 0.00895714759827" rpy="0.000218331973274 0.0113785043803 -1.58362463673" connected_to="world"/>
-<xacro:panda_robot robot_id="1" xyz="0.512020647526 0.169103205204 0.0144633054733" rpy="0.00347274780491 0.00851996101077 -1.6038241594" connected_to="world"/>
+<xacro:indy7_robot robot_id="0" xyz="-0.447089582682 0.251743137836 0.00930815935135" rpy="-0.000777551145325 0.0099242762868 -1.58336192744" connected_to="world"/>
+<xacro:panda_robot robot_id="1" xyz="0.511796474457 0.169063687325 0.0137922167778" rpy="0.00260240796696 0.00891747931083 -1.60378843737" connected_to="world"/>
 <!-- BODY END -->
 </robot>

Commit message: geometry highlight

File: eTaSL/robots/custom_robots.urdf (robot description, URDF)
Before this commit: robot custom_robots, 21 links, 20 joints
Joints:
- joint indy0_joint_world: origin xyz=-0.447089582682 0.251743137836 0.00930815935135 rpy=-0.000777551145325 0.0099242762868 -1.58336192744 -> xyz=-0.446351528168 0.250944495201 0.0100504755974 rpy=-0.000982771636904 0.0102033592034 -1.58339573208
- joint panda1_joint_world: origin xyz=0.511796474457 0.169063687325 0.0137922167778 rpy=0.00260240796696 0.00891747931083 -1.60378843737 -> xyz=0.511830508709 0.169060587883 0.0139080882072 rpy=0.00195979646653 0.010065130463 -1.60364898676

File: eTaSL/robots/custom_robots.urdf.xacro (robot description, xacro)
@@ -6,6 +6,6 @@
 <link name="world"/>
 <!-- BODY BEGIN -->
-<xacro:indy7_robot robot_id="0" xyz="-0.447089582682 0.251743137836 0.00930815935135" rpy="-0.000777551145325 0.0099242762868 -1.58336192744" connected_to="world"/>
-<xacro:panda_robot robot_id="1" xyz="0.511796474457 0.169063687325 0.0137922167778" rpy="0.00260240796696 0.00891747931083 -1.60378843737" connected_to="world"/>
+<xacro:indy7_robot robot_id="0" xyz="-0.446351528168 0.250944495201 0.0100504755974" rpy="-0.000982771636904 0.0102033592034 -1.58339573208" connected_to="world"/>
+<xacro:panda_robot robot_id="1" xyz="0.511830508709 0.169060587883 0.0139080882072" rpy="0.00195979646653 0.010065130463 -1.60364898676" connected_to="world"/>
 <!-- BODY END -->
 </robot>

Commit message: add: edit on ui

File: eTaSL/robots/custom_robots.urdf (robot description, URDF)
Before this commit: robot custom_robots, 21 links, 20 joints
Joints:
- joint indy0_joint_world: origin xyz=-0.446351528168 0.250944495201 0.0100504755974 rpy=-0.000982771636904 0.0102033592034 -1.58339573208 -> xyz=-0.447125524282 0.25188177824 0.00954228639603 rpy=-0.000786073748207 0.0113239621656 -1.58316111891
- joint panda1_joint_world: origin xyz=0.511830508709 0.169060587883 0.0139080882072 rpy=0.00195979646653 0.010065130463 -1.60364898676 -> xyz=0.511731863022 0.169007122517 0.0142500400543 rpy=0.00226339383764 0.0112383342552 -1.60351950715

File: eTaSL/robots/custom_robots.urdf.xacro (robot description, xacro)
@@ -6,6 +6,6 @@
 <link name="world"/>
 <!-- BODY BEGIN -->
-<xacro:indy7_robot robot_id="0" xyz="-0.446351528168 0.250944495201 0.0100504755974" rpy="-0.000982771636904 0.0102033592034 -1.58339573208" connected_to="world"/>
-<xacro:panda_robot robot_id="1" xyz="0.511830508709 0.169060587883 0.0139080882072" rpy="0.00195979646653 0.010065130463 -1.60364898676" connected_to="world"/>
+<xacro:indy7_robot robot_id="0" xyz="-0.447125524282 0.25188177824 0.00954228639603" rpy="-0.000786073748207 0.0113239621656 -1.58316111891" connected_to="world"/>
+<xacro:panda_robot robot_id="1" xyz="0.511731863022 0.169007122517 0.0142500400543" rpy="0.00226339383764 0.0112383342552 -1.60351950715" connected_to="world"/>
 <!-- BODY END -->
 </robot>
