Commit message: adding items on ui

File: eTaSL/robots/custom_robots.urdf (robot description, URDF)
Before this commit: robot custom_robots, 21 links, 20 joints
Joints:
- joint indy0_joint_world: origin xyz=-0.447125524282 0.25188177824 0.00954228639603 rpy=-0.000786073748207 0.0113239621656 -1.58316111891 -> xyz=-0.44669726491 0.251301169395 0.00963199138641 rpy=-0.000266146761863 0.00986735077519 -1.58340901368
- joint panda1_joint_world: origin xyz=0.511731863022 0.169007122517 0.0142500400543 rpy=0.00226339383764 0.0112383342552 -1.60351950715 -> xyz=0.511927962303 0.168936312199 0.0140175819397 rpy=0.00304314049613 0.00752384593206 -1.6042687524

File: eTaSL/robots/custom_robots.urdf.xacro (robot description, xacro)
@@ -6,6 +6,6 @@
 <link name="world"/>
 <!-- BODY BEGIN -->
-<xacro:indy7_robot robot_id="0" xyz="-0.447125524282 0.25188177824 0.00954228639603" rpy="-0.000786073748207 0.0113239621656 -1.58316111891" connected_to="world"/>
-<xacro:panda_robot robot_id="1" xyz="0.511731863022 0.169007122517 0.0142500400543" rpy="0.00226339383764 0.0112383342552 -1.60351950715" connected_to="world"/>
+<xacro:indy7_robot robot_id="0" xyz="-0.44669726491 0.251301169395 0.00963199138641" rpy="-0.000266146761863 0.00986735077519 -1.58340901368" connected_to="world"/>
+<xacro:panda_robot robot_id="1" xyz="0.511927962303 0.168936312199 0.0140175819397" rpy="0.00304314049613 0.00752384593206 -1.6042687524" connected_to="world"/>
 <!-- BODY END -->
 </robot>

Commit message: alert window

File: eTaSL/robots/custom_robots.urdf (robot description, URDF)
Before this commit: robot custom_robots, 21 links, 20 joints
Joints:
- joint indy0_joint_world: origin xyz=-0.44669726491 0.251301169395 0.00963199138641 rpy=-0.000266146761863 0.00986735077519 -1.58340901368 -> xyz=-0.447575032711 0.252288937569 0.00884616374969 rpy=-0.000299019047122 0.0100618512555 -1.5834750926
- joint panda1_joint_world: origin xyz=0.511927962303 0.168936312199 0.0140175819397 rpy=0.00304314049613 0.00752384593206 -1.6042687524 -> xyz=0.511860847473 0.168938755989 0.0141784548759 rpy=0.00353412327475 0.00806033419847 -1.60389642216

File: eTaSL/robots/custom_robots.urdf.xacro (robot description, xacro)
@@ -6,6 +6,6 @@
 <link name="world"/>
 <!-- BODY BEGIN -->
-<xacro:indy7_robot robot_id="0" xyz="-0.44669726491 0.251301169395 0.00963199138641" rpy="-0.000266146761863 0.00986735077519 -1.58340901368" connected_to="world"/>
-<xacro:panda_robot robot_id="1" xyz="0.511927962303 0.168936312199 0.0140175819397" rpy="0.00304314049613 0.00752384593206 -1.6042687524" connected_to="world"/>
+<xacro:indy7_robot robot_id="0" xyz="-0.447575032711 0.252288937569 0.00884616374969" rpy="-0.000299019047122 0.0100618512555 -1.5834750926" connected_to="world"/>
+<xacro:panda_robot robot_id="1" xyz="0.511860847473 0.168938755989 0.0141784548759" rpy="0.00353412327475 0.00806033419847 -1.60389642216" connected_to="world"/>
 <!-- BODY END -->
 </robot>

Commit message: add color column

File: eTaSL/robots/custom_robots.urdf (robot description, URDF)
Before this commit: robot custom_robots, 21 links, 20 joints
Joints:
- joint indy0_joint_world: origin xyz=-0.447575032711 0.252288937569 0.00884616374969 rpy=-0.000299019047122 0.0100618512555 -1.5834750926 -> xyz=-0.446887671947 0.251476824284 0.00942754745483 rpy=-0.000177686551762 0.00997097933108 -1.58349111017
- joint panda1_joint_world: origin xyz=0.511860847473 0.168938755989 0.0141784548759 rpy=0.00353412327475 0.00806033419847 -1.60389642216 -> xyz=0.511890292168 0.168987095356 0.0141258239746 rpy=0.00280295202734 0.00798156443412 -1.60367766159

File: eTaSL/robots/custom_robots.urdf.xacro (robot description, xacro)
@@ -6,6 +6,6 @@
 <link name="world"/>
 <!-- BODY BEGIN -->
-<xacro:indy7_robot robot_id="0" xyz="-0.447575032711 0.252288937569 0.00884616374969" rpy="-0.000299019047122 0.0100618512555 -1.5834750926" connected_to="world"/>
-<xacro:panda_robot robot_id="1" xyz="0.511860847473 0.168938755989 0.0141784548759" rpy="0.00353412327475 0.00806033419847 -1.60389642216" connected_to="world"/>
+<xacro:indy7_robot robot_id="0" xyz="-0.446887671947 0.251476824284 0.00942754745483" rpy="-0.000177686551762 0.00997097933108 -1.58349111017" connected_to="world"/>
+<xacro:panda_robot robot_id="1" xyz="0.511890292168 0.168987095356 0.0141258239746" rpy="0.00280295202734 0.00798156443412 -1.60367766159" connected_to="world"/>
 <!-- BODY END -->
 </robot>

Commit message: apply button - geometry

File: eTaSL/robots/custom_robots.urdf (robot description, URDF)
Before this commit: robot custom_robots, 21 links, 20 joints
Joints:
- joint indy0_joint_world: origin xyz=-0.446887671947 0.251476824284 0.00942754745483 rpy=-0.000177686551762 0.00997097933108 -1.58349111017 -> xyz=-0.446841061115 0.251525461674 0.00928843021393 rpy=-0.000500482817951 0.00848237961543 -1.58320916313
- joint panda1_joint_world: origin xyz=0.511890292168 0.168987095356 0.0141258239746 rpy=0.00280295202734 0.00798156443412 -1.60367766159 -> xyz=0.51185053587 0.1689915061 0.0139050483704 rpy=0.00189289953126 0.00749565300636 -1.60355150794

File: eTaSL/robots/custom_robots.urdf.xacro (robot description, xacro)
@@ -6,6 +6,6 @@
 <link name="world"/>
 <!-- BODY BEGIN -->
-<xacro:indy7_robot robot_id="0" xyz="-0.446887671947 0.251476824284 0.00942754745483" rpy="-0.000177686551762 0.00997097933108 -1.58349111017" connected_to="world"/>
-<xacro:panda_robot robot_id="1" xyz="0.511890292168 0.168987095356 0.0141258239746" rpy="0.00280295202734 0.00798156443412 -1.60367766159" connected_to="world"/>
+<xacro:indy7_robot robot_id="0" xyz="-0.446841061115 0.251525461674 0.00928843021393" rpy="-0.000500482817951 0.00848237961543 -1.58320916313" connected_to="world"/>
+<xacro:panda_robot robot_id="1" xyz="0.51185053587 0.1689915061 0.0139050483704" rpy="0.00189289953126 0.00749565300636 -1.60355150794" connected_to="world"/>
 <!-- BODY END -->
 </robot>

Commit message: apply button - all

File: eTaSL/robots/custom_robots.urdf (robot description, URDF)
Before this commit: robot custom_robots, 21 links, 20 joints
Joints:
- joint indy0_joint_world: origin xyz=-0.446841061115 0.251525461674 0.00928843021393 rpy=-0.000500482817951 0.00848237961543 -1.58320916313 -> xyz=-0.446829646826 0.25150924921 0.00932848453522 rpy=-0.00028751925484 0.00897833830555 -1.58346420697
- joint panda1_joint_world: origin xyz=0.51185053587 0.1689915061 0.0139050483704 rpy=0.00189289953126 0.00749565300636 -1.60355150794 -> xyz=0.511869132519 0.168899774551 0.0140367746353 rpy=0.00255439968358 0.00729224601369 -1.60384236158

File: eTaSL/robots/custom_robots.urdf.xacro (robot description, xacro)
@@ -6,6 +6,6 @@
 <link name="world"/>
 <!-- BODY BEGIN -->
-<xacro:indy7_robot robot_id="0" xyz="-0.446841061115 0.251525461674 0.00928843021393" rpy="-0.000500482817951 0.00848237961543 -1.58320916313" connected_to="world"/>
-<xacro:panda_robot robot_id="1" xyz="0.51185053587 0.1689915061 0.0139050483704" rpy="0.00189289953126 0.00749565300636 -1.60355150794" connected_to="world"/>
+<xacro:indy7_robot robot_id="0" xyz="-0.446829646826 0.25150924921 0.00932848453522" rpy="-0.00028751925484 0.00897833830555 -1.58346420697" connected_to="world"/>
+<xacro:panda_robot robot_id="1" xyz="0.511869132519 0.168899774551 0.0140367746353" rpy="0.00255439968358 0.00729224601369 -1.60384236158" connected_to="world"/>
 <!-- BODY END -->
 </robot>

Commit message: save/load

File: eTaSL/robots/custom_robots.urdf (robot description, URDF)
Before this commit: robot custom_robots, 21 links, 20 joints
Joints:
- joint indy0_joint_world: origin xyz=-0.446829646826 0.25150924921 0.00932848453522 rpy=-0.00028751925484 0.00897833830555 -1.58346420697 -> xyz=-0.446975767612 0.251331269741 0.0091809630394 rpy=-0.000479467040228 0.00876867086048 -1.58309623578
- joint panda1_joint_world: origin xyz=0.511869132519 0.168899774551 0.0140367746353 rpy=0.00255439968358 0.00729224601369 -1.60384236158 -> xyz=0.511975884438 0.16916590929 0.0137903094292 rpy=0.00302905504579 0.00716966608649 -1.60358394961

File: eTaSL/robots/custom_robots.urdf.xacro (robot description, xacro)
@@ -6,6 +6,6 @@
 <link name="world"/>
 <!-- BODY BEGIN -->
-<xacro:indy7_robot robot_id="0" xyz="-0.446829646826 0.25150924921 0.00932848453522" rpy="-0.00028751925484 0.00897833830555 -1.58346420697" connected_to="world"/>
-<xacro:panda_robot robot_id="1" xyz="0.511869132519 0.168899774551 0.0140367746353" rpy="0.00255439968358 0.00729224601369 -1.60384236158" connected_to="world"/>
+<xacro:indy7_robot robot_id="0" xyz="-0.446975767612 0.251331269741 0.0091809630394" rpy="-0.000479467040228 0.00876867086048 -1.58309623578" connected_to="world"/>
+<xacro:panda_robot robot_id="1" xyz="0.511975884438 0.16916590929 0.0137903094292" rpy="0.00302905504579 0.00716966608649 -1.60358394961" connected_to="world"/>
 <!-- BODY END -->
 </robot>

Commit message: table class rearranged

File: eTaSL/robots/custom_robots.urdf (robot description, URDF)
Before this commit: robot custom_robots, 21 links, 20 joints
Joints:
- joint indy0_joint_world: origin xyz=-0.446975767612 0.251331269741 0.0091809630394 rpy=-0.000479467040228 0.00876867086048 -1.58309623578 -> xyz=-0.447489887476 0.252018153667 0.00919073820114 rpy=-0.000773883520826 0.0104158320006 -1.58349013673
- joint panda1_joint_world: origin xyz=0.511975884438 0.16916590929 0.0137903094292 rpy=0.00302905504579 0.00716966608649 -1.60358394961 -> xyz=0.511909782887 0.168973684311 0.0137454867363 rpy=0.00257331026035 0.0090591353786 -1.60378990297

File: eTaSL/robots/custom_robots.urdf.xacro (robot description, xacro)
@@ -6,6 +6,6 @@
 <link name="world"/>
 <!-- BODY BEGIN -->
-<xacro:indy7_robot robot_id="0" xyz="-0.446975767612 0.251331269741 0.0091809630394" rpy="-0.000479467040228 0.00876867086048 -1.58309623578" connected_to="world"/>
-<xacro:panda_robot robot_id="1" xyz="0.511975884438 0.16916590929 0.0137903094292" rpy="0.00302905504579 0.00716966608649 -1.60358394961" connected_to="world"/>
+<xacro:indy7_robot robot_id="0" xyz="-0.447489887476 0.252018153667 0.00919073820114" rpy="-0.000773883520826 0.0104158320006 -1.58349013673" connected_to="world"/>
+<xacro:panda_robot robot_id="1" xyz="0.511909782887 0.168973684311 0.0137454867363" rpy="0.00257331026035 0.0090591353786 -1.60378990297" connected_to="world"/>
 <!-- BODY END -->
 </robot>

Commit message: added marker table

File: eTaSL/robots/custom_robots.urdf (robot description, URDF)
Before this commit: robot custom_robots, 21 links, 20 joints
Joints:
- joint indy0_joint_world: origin xyz=-0.447489887476 0.252018153667 0.00919073820114 rpy=-0.000773883520826 0.0104158320006 -1.58349013673 -> xyz=-0.446726590395 0.251432359219 0.00986218452454 rpy=-0.000369469061368 0.0125775666215 -1.58368285343
- joint panda1_joint_world: origin xyz=0.511909782887 0.168973684311 0.0137454867363 rpy=0.00257331026035 0.0090591353786 -1.60378990297 -> xyz=0.511735975742 0.168907999992 0.0141640901566 rpy=0.00280069150367 0.0109091477839 -1.60412351948

File: eTaSL/robots/custom_robots.urdf.xacro (robot description, xacro)
@@ -6,6 +6,6 @@
 <link name="world"/>
 <!-- BODY BEGIN -->
-<xacro:indy7_robot robot_id="0" xyz="-0.447489887476 0.252018153667 0.00919073820114" rpy="-0.000773883520826 0.0104158320006 -1.58349013673" connected_to="world"/>
-<xacro:panda_robot robot_id="1" xyz="0.511909782887 0.168973684311 0.0137454867363" rpy="0.00257331026035 0.0090591353786 -1.60378990297" connected_to="world"/>
+<xacro:indy7_robot robot_id="0" xyz="-0.446726590395 0.251432359219 0.00986218452454" rpy="-0.000369469061368 0.0125775666215 -1.58368285343" connected_to="world"/>
+<xacro:panda_robot robot_id="1" xyz="0.511735975742 0.168907999992 0.0141640901566" rpy="0.00280069150367 0.0109091477839 -1.60412351948" connected_to="world"/>
 <!-- BODY END -->
 </robot>

Commit message: marker dictionary rearranged

File: eTaSL/robots/custom_robots.urdf (robot description, URDF)
Before this commit: robot custom_robots, 21 links, 20 joints
Joints:
- joint indy0_joint_world: origin xyz=-0.446726590395 0.251432359219 0.00986218452454 rpy=-0.000369469061368 0.0125775666215 -1.58368285343 -> xyz=-0.446890115738 0.251582622528 0.0094285607338 rpy=-0.000148345037642 0.0095512232247 -1.58361760252
- joint panda1_joint_world: origin xyz=0.511735975742 0.168907999992 0.0141640901566 rpy=0.00280069150367 0.0109091477839 -1.60412351948 -> xyz=0.511936485767 0.1687977314 0.0140640735626 rpy=0.00281744671926 0.00706854399847 -1.60383688131

File: eTaSL/robots/custom_robots.urdf.xacro (robot description, xacro)
@@ -6,6 +6,6 @@
 <link name="world"/>
 <!-- BODY BEGIN -->
-<xacro:indy7_robot robot_id="0" xyz="-0.446726590395 0.251432359219 0.00986218452454" rpy="-0.000369469061368 0.0125775666215 -1.58368285343" connected_to="world"/>
-<xacro:panda_robot robot_id="1" xyz="0.511735975742 0.168907999992 0.0141640901566" rpy="0.00280069150367 0.0109091477839 -1.60412351948" connected_to="world"/>
+<xacro:indy7_robot robot_id="0" xyz="-0.446890115738 0.251582622528 0.0094285607338" rpy="-0.000148345037642 0.0095512232247 -1.58361760252" connected_to="world"/>
+<xacro:panda_robot robot_id="1" xyz="0.511936485767 0.1687977314 0.0140640735626" rpy="0.00281744671926 0.00706854399847 -1.60383688131" connected_to="world"/>
 <!-- BODY END -->
 </robot>

Commit message: add marker group table

File: eTaSL/robots/custom_robots.urdf (robot description, URDF)
Before this commit: robot custom_robots, 21 links, 20 joints
Joints:
- joint indy0_joint_world: origin xyz=-0.446890115738 0.251582622528 0.0094285607338 rpy=-0.000148345037642 0.0095512232247 -1.58361760252 -> xyz=-0.446760386229 0.251339614391 0.00939214229584 rpy=2.55546752196e-05 0.0090497179139 -1.58362752967
- joint panda1_joint_world: origin xyz=0.511936485767 0.1687977314 0.0140640735626 rpy=0.00281744671926 0.00706854399847 -1.60383688131 -> xyz=0.511899709702 0.168718695641 0.0142241120338 rpy=0.00291801812264 0.00722125486721 -1.60398812001

File: eTaSL/robots/custom_robots.urdf.xacro (robot description, xacro)
@@ -6,6 +6,6 @@
 <link name="world"/>
 <!-- BODY BEGIN -->
-<xacro:indy7_robot robot_id="0" xyz="-0.446890115738 0.251582622528 0.0094285607338" rpy="-0.000148345037642 0.0095512232247 -1.58361760252" connected_to="world"/>
-<xacro:panda_robot robot_id="1" xyz="0.511936485767 0.1687977314 0.0140640735626" rpy="0.00281744671926 0.00706854399847 -1.60383688131" connected_to="world"/>
+<xacro:indy7_robot robot_id="0" xyz="-0.446760386229 0.251339614391 0.00939214229584" rpy="2.55546752196e-05 0.0090497179139 -1.58362752967" connected_to="world"/>
+<xacro:panda_robot robot_id="1" xyz="0.511899709702 0.168718695641 0.0142241120338" rpy="0.00291801812264 0.00722125486721 -1.60398812001" connected_to="world"/>
 <!-- BODY END -->
 </robot>

Commit message: custom buttons

File: eTaSL/robots/custom_robots.urdf (robot description, URDF)
Before this commit: robot custom_robots, 21 links, 20 joints
Joints:
- joint indy0_joint_world: origin xyz=-0.446760386229 0.251339614391 0.00939214229584 rpy=2.55546752196e-05 0.0090497179139 -1.58362752967 -> xyz=-0.447129100561 0.25176858902 0.00926351547241 rpy=-0.000471391155784 0.00981608902927 -1.58331994107
- joint panda1_joint_world: origin xyz=0.511899709702 0.168718695641 0.0142241120338 rpy=0.00291801812264 0.00722125486721 -1.60398812001 -> xyz=0.511987090111 0.168942570686 0.014035820961 rpy=0.00258412220776 0.00830773103583 -1.60374862654

File: eTaSL/robots/custom_robots.urdf.xacro (robot description, xacro)
@@ -6,6 +6,6 @@
 <link name="world"/>
 <!-- BODY BEGIN -->
-<xacro:indy7_robot robot_id="0" xyz="-0.446760386229 0.251339614391 0.00939214229584" rpy="2.55546752196e-05 0.0090497179139 -1.58362752967" connected_to="world"/>
-<xacro:panda_robot robot_id="1" xyz="0.511899709702 0.168718695641 0.0142241120338" rpy="0.00291801812264 0.00722125486721 -1.60398812001" connected_to="world"/>
+<xacro:indy7_robot robot_id="0" xyz="-0.447129100561 0.25176858902 0.00926351547241" rpy="-0.000471391155784 0.00981608902927 -1.58331994107" connected_to="world"/>
+<xacro:panda_robot robot_id="1" xyz="0.511987090111 0.168942570686 0.014035820961" rpy="0.00258412220776 0.00830773103583 -1.60374862654" connected_to="world"/>
 <!-- BODY END -->
 </robot>

Commit message: mark env, mark obj buttons

File: eTaSL/robots/custom_robots.urdf (robot description, URDF)
Before this commit: robot custom_robots, 21 links, 20 joints
Joints:
- joint indy0_joint_world: origin xyz=-0.447129100561 0.25176858902 0.00926351547241 rpy=-0.000471391155784 0.00981608902927 -1.58331994107 -> xyz=-0.446853458881 0.251941144466 0.00922828912735 rpy=-0.000401127417375 0.00994612273342 -1.58412575687
- joint panda1_joint_world: origin xyz=0.511987090111 0.168942570686 0.014035820961 rpy=0.00258412220776 0.00830773103583 -1.60374862654 -> xyz=0.51176649332 0.168401837349 0.0142036676407 rpy=0.00446882935677 0.00977478182656 -1.60595016666

File: eTaSL/robots/custom_robots.urdf.xacro (robot description, xacro)
@@ -6,6 +6,6 @@
 <link name="world"/>
 <!-- BODY BEGIN -->
-<xacro:indy7_robot robot_id="0" xyz="-0.447129100561 0.25176858902 0.00926351547241" rpy="-0.000471391155784 0.00981608902927 -1.58331994107" connected_to="world"/>
-<xacro:panda_robot robot_id="1" xyz="0.511987090111 0.168942570686 0.014035820961" rpy="0.00258412220776 0.00830773103583 -1.60374862654" connected_to="world"/>
+<xacro:indy7_robot robot_id="0" xyz="-0.446853458881 0.251941144466 0.00922828912735" rpy="-0.000401127417375 0.00994612273342 -1.58412575687" connected_to="world"/>
+<xacro:panda_robot robot_id="1" xyz="0.51176649332 0.168401837349 0.0142036676407" rpy="0.00446882935677 0.00977478182656 -1.60595016666" connected_to="world"/>
 <!-- BODY END -->
 </robot>

Commit message: load with ui from base

File: eTaSL/robots/custom_robots.urdf (robot description, URDF)
Before this commit: robot custom_robots, 21 links, 20 joints
Joints:
- joint indy0_joint_world: origin xyz=-0.446853458881 0.251941144466 0.00922828912735 rpy=-0.000401127417375 0.00994612273342 -1.58412575687 -> xyz=-0.446646004915 0.25178706646 0.00932586193085 rpy=-0.000744570111449 0.00974506666908 -1.58416129344
- joint panda1_joint_world: origin xyz=0.51176649332 0.168401837349 0.0142036676407 rpy=0.00446882935677 0.00977478182656 -1.60595016666 -> xyz=0.511914908886 0.168241202831 0.01401668787 rpy=0.00357848768595 0.00937967387927 -1.60539142562

File: eTaSL/robots/custom_robots.urdf.xacro (robot description, xacro)
@@ -6,6 +6,6 @@
 <link name="world"/>
 <!-- BODY BEGIN -->
-<xacro:indy7_robot robot_id="0" xyz="-0.446853458881 0.251941144466 0.00922828912735" rpy="-0.000401127417375 0.00994612273342 -1.58412575687" connected_to="world"/>
-<xacro:panda_robot robot_id="1" xyz="0.51176649332 0.168401837349 0.0142036676407" rpy="0.00446882935677 0.00977478182656 -1.60595016666" connected_to="world"/>
+<xacro:indy7_robot robot_id="0" xyz="-0.446646004915 0.25178706646 0.00932586193085" rpy="-0.000744570111449 0.00974506666908 -1.58416129344" connected_to="world"/>
+<xacro:panda_robot robot_id="1" xyz="0.511914908886 0.168241202831 0.01401668787" rpy="0.00357848768595 0.00937967387927 -1.60539142562" connected_to="world"/>
 <!-- BODY END -->
 </robot>

Commit message: camera and robot tab

File: eTaSL/robots/custom_robots.urdf (robot description, URDF)
Before this commit: robot custom_robots, 21 links, 20 joints
Joints:
- joint indy0_joint_world: origin xyz=-0.446646004915 0.25178706646 0.00932586193085 rpy=-0.000744570111449 0.00974506666908 -1.58416129344 -> xyz=-0.446480512619 0.251528263092 0.00979518890381 rpy=7.72251143907e-05 0.012837732858 -1.58433052921
- joint panda1_joint_world: origin xyz=0.511914908886 0.168241202831 0.01401668787 rpy=0.00357848768595 0.00937967387927 -1.60539142562 -> xyz=0.511702060699 0.168303191662 0.014661192894 rpy=0.00371903837049 0.0130669918716 -1.60510658312

File: eTaSL/robots/custom_robots.urdf.xacro (robot description, xacro)
@@ -6,6 +6,6 @@
 <link name="world"/>
 <!-- BODY BEGIN -->
-<xacro:indy7_robot robot_id="0" xyz="-0.446646004915 0.25178706646 0.00932586193085" rpy="-0.000744570111449 0.00974506666908 -1.58416129344" connected_to="world"/>
-<xacro:panda_robot robot_id="1" xyz="0.511914908886 0.168241202831 0.01401668787" rpy="0.00357848768595 0.00937967387927 -1.60539142562" connected_to="world"/>
+<xacro:indy7_robot robot_id="0" xyz="-0.446480512619 0.251528263092 0.00979518890381" rpy="7.72251143907e-05 0.012837732858 -1.58433052921" connected_to="world"/>
+<xacro:panda_robot robot_id="1" xyz="0.511702060699 0.168303191662 0.014661192894" rpy="0.00371903837049 0.0130669918716 -1.60510658312" connected_to="world"/>
 <!-- BODY END -->
 </robot>

Commit message: fix online plan

File: eTaSL/robots/custom_robots.urdf (robot description, URDF)
Before this commit: robot custom_robots, 21 links, 20 joints
Links:
- link panda1_hand: geometry collision box size=0.06 0.094 0.22; visual mesh filename=package://franka_description/meshes/visual/hand.dae
- link panda1_link6: geometry collision cylinder length=0.09 radius=0.09; collision sphere radius=0.06

File: eTaSL/robots/hand.xacro (robot description, xacro)
@@ -16,7 +16,7 @@
       </visual>
       <collision>
-        <origin xyz="0 0 0.02" rpy="1.57079633 0 0"/>
+        <origin xyz="0 0 0.025" rpy="1.57079633 0 0"/>
         <geometry>
-          <cylinder length="0.14" radius="0.06"/>
+          <box size="0.06 0.094 0.22"/>
         </geometry>
       </collision>

File: eTaSL/robots/panda_arm.xacro (robot description, xacro)
@@ -145,4 +145,10 @@
         </geometry>
       </collision>
+      <collision>
+        <origin xyz="0.09 -0.07 0" rpy="0 0 0"/>
+        <geometry>
+          <sphere radius="0.06"/>
+        </geometry>
+      </collision>
     </link>
     <joint name="${arm_id}_joint6" type="revolute">

Commit message: Drop tesseract/trajopt

File: eTaSL/robots/custom_robots.urdf (robot description, URDF)
Before this commit: robot custom_robots, 21 links, 20 joints
Links:
- link indy0_tcp: geometry collision cylinder length=0.08 radius=0.016; collision cylinder length=0.08 radius=0.016

File: eTaSL/robots/indy7_robot.xacro (robot description, xacro)
@@ -163,7 +163,7 @@
 			<origin xyz="0 0 0" rpy="0 0 1.570796"/>
 			<geometry>
-				<mesh filename="package://my_mesh/meshes/stl/indy_gripper_asm2_ctd.STL" scale="0.001 0.001 0.001"/>
-			</geometry>
-			<material name="${tool_material}"/>
+				<mesh filename="package://my_mesh/meshes/stl/indy_gripper_asm2_res.STL"/>
+			</geometry>
+			<material name="${indy_material}"/>
 		</visual>
 		<collision>
