Commit message: ompl/etasl hybrid motion plan finished

File: eTaSL/robots/custom_robots.urdf (robot description, URDF)
Before this commit: robot custom_robots, 21 links, 20 joints
Links:
- removed link world
- added link base_link
- link panda1_hand: geometry collision cylinder length=0.05 radius=0.01; collision cylinder length=0.055 radius=0.02
- link panda1_link6: geometry collision cylinder length=0.08 radius=0.04; collision cylinder length=0.09 radius=0.065
Joints:
- removed joint indy0_joint_world
- removed joint panda1_joint_world
- added joint indy0_joint_base_link: type fixed, parent base_link, child indy0_link0, origin xyz=-0.446480512619 0.251528263092 0.00979518890381 rpy=7.72251143907e-05 0.012837732858 -1.58433052921
- added joint panda1_joint_base_link: type fixed, parent base_link, child panda1_link0, origin xyz=0.511702060699 0.168303191662 0.014661192894 rpy=0.00371903837049 0.0130669918716 -1.60510658312

File: eTaSL/robots/custom_robots.urdf.xacro (robot description, xacro)
@@ -4,8 +4,8 @@
 <xacro:include filename="$(env TAMP_ETASL_DIR)/robots/panda_robot.xacro"/>
 <xacro:include filename="$(env TAMP_ETASL_DIR)/robots/indy7_robot.xacro"/>
-<link name="world"/>
+<link name="base_link"/>
 <!-- BODY BEGIN -->
-<xacro:indy7_robot robot_id="0" xyz="-0.446480512619 0.251528263092 0.00979518890381" rpy="7.72251143907e-05 0.012837732858 -1.58433052921" connected_to="world"/>
-<xacro:panda_robot robot_id="1" xyz="0.511702060699 0.168303191662 0.014661192894" rpy="0.00371903837049 0.0130669918716 -1.60510658312" connected_to="world"/>
+<xacro:indy7_robot robot_id="0" xyz="-0.446480512619 0.251528263092 0.00979518890381" rpy="7.72251143907e-05 0.012837732858 -1.58433052921" connected_to="base_link"/>
+<xacro:panda_robot robot_id="1" xyz="0.511702060699 0.168303191662 0.014661192894" rpy="0.00371903837049 0.0130669918716 -1.60510658312" connected_to="base_link"/>
 <!-- BODY END -->
 </robot>

File: eTaSL/robots/hand.xacro (robot description, xacro)
@@ -16,7 +16,19 @@
       </visual>
       <collision>
-        <origin xyz="0 0 0.025" rpy="1.57079633 0 0"/>
+        <origin xyz="0 0 0.03" rpy="1.57079633 0 0"/>
         <geometry>
-          <box size="0.06 0.094 0.22"/>
+          <cylinder length="0.16" radius="0.045"/>
+        </geometry>
+      </collision>
+      <collision>
+        <origin xyz="0 0.07 -0.02" rpy="0 1.57079633 0"/>
+        <geometry>
+          <cylinder length="0.055" radius="0.02"/>
+        </geometry>
+      </collision>
+      <collision>
+        <origin xyz="0 -0.07 -0.02" rpy="1.57079633 0 0"/>
+        <geometry>
+          <cylinder length="0.05" radius="0.01"/>
         </geometry>
       </collision>

File: eTaSL/robots/panda_arm.xacro (robot description, xacro)
@@ -142,11 +142,17 @@
         <origin xyz="0.035 0.    0." rpy="-0.         -1.57079633  0."/>
         <geometry>
-          <cylinder length="0.09" radius="0.09"/>
+          <cylinder length="0.09" radius="0.065"/>
         </geometry>
       </collision>
       <collision>
-        <origin xyz="0.09 -0.07 0" rpy="0 0 0"/>
+        <origin xyz="0.09 -0.01 0." rpy="1.57079633         0.  0."/>
         <geometry>
-          <sphere radius="0.06"/>
+          <cylinder length="0.13" radius="0.05"/>
+        </geometry>
+      </collision>
+      <collision>
+        <origin xyz="0.085 0.05 0." rpy="0.2         1.57079633  0."/>
+        <geometry>
+          <cylinder length="0.08" radius="0.04"/>
         </geometry>
       </collision>

Commit message: data collection initialization up to joints

File: eTaSL/robots/custom_robots.urdf (robot description, URDF)
Before this commit: robot custom_robots, 21 links, 20 joints
Joints:
- joint indy0_joint_base_link: origin xyz=1.48274451419 0.452685329639 0.188611320622 rpy=0.0 0.0 0.340886585646 -> xyz=1.78003959386 1.62701435499 0.0688030359861 rpy=0.0 0.0 4.22082414346
- joint panda1_joint_base_link: origin xyz=0.5035655925 1.68277256243 0.325530553938 rpy=0.0 0.0 1.33622974449 -> xyz=0.809763246433 2.17829170696 0.220872759501 rpy=0.0 0.0 0.572030753901

File: eTaSL/robots/custom_robots.urdf.xacro (robot description, xacro)
@@ -6,6 +6,6 @@
 <link name="base_link"/>
 <!-- BODY BEGIN -->
-<xacro:indy7_robot robot_id="0" xyz="1.48274451419 0.452685329639 0.188611320622" rpy="0 0 0.340886585646" connected_to="base_link"/>
-<xacro:panda_robot robot_id="1" xyz="0.5035655925 1.68277256243 0.325530553938" rpy="0 0 1.33622974449" connected_to="base_link"/>
+<xacro:indy7_robot robot_id="0" xyz="1.78003959386 1.62701435499 0.0688030359861" rpy="0 0 4.22082414346" connected_to="base_link"/>
+<xacro:panda_robot robot_id="1" xyz="0.809763246433 2.17829170696 0.220872759501" rpy="0 0 0.572030753901" connected_to="base_link"/>
 <!-- BODY END -->
 </robot>

Commit message: collision checking

File: eTaSL/robots/custom_robots.urdf (robot description, URDF)
Before this commit: robot custom_robots, 21 links, 20 joints
Joints:
- joint indy0_joint_base_link: origin xyz=1.78003959386 1.62701435499 0.0688030359861 rpy=0.0 0.0 4.22082414346 -> xyz=0.818223732196 1.39940643743 0.20048313416 rpy=0.0 0.0 0.76977434965
- joint panda1_joint_base_link: origin xyz=0.809763246433 2.17829170696 0.220872759501 rpy=0.0 0.0 0.572030753901 -> xyz=2.11001260883 2.11178463597 0.431667235678 rpy=0.0 0.0 6.11172683293

File: eTaSL/robots/custom_robots.urdf.xacro (robot description, xacro)
@@ -6,6 +6,6 @@
 <link name="base_link"/>
 <!-- BODY BEGIN -->
-<xacro:indy7_robot robot_id="0" xyz="1.78003959386 1.62701435499 0.0688030359861" rpy="0 0 4.22082414346" connected_to="base_link"/>
-<xacro:panda_robot robot_id="1" xyz="0.809763246433 2.17829170696 0.220872759501" rpy="0 0 0.572030753901" connected_to="base_link"/>
+<xacro:indy7_robot robot_id="0" xyz="0.818223732196 1.39940643743 0.20048313416" rpy="0 0 0.76977434965" connected_to="base_link"/>
+<xacro:panda_robot robot_id="1" xyz="2.11001260883 2.11178463597 0.431667235678" rpy="0 0 6.11172683293" connected_to="base_link"/>
 <!-- BODY END -->
 </robot>

Commit message: CollectData-scene all prepared

File: eTaSL/robots/custom_robots.urdf (robot description, URDF)
Before this commit: robot custom_robots, 21 links, 20 joints
Joints:
- joint indy0_joint_base_link: origin xyz=0.818223732196 1.39940643743 0.20048313416 rpy=0.0 0.0 0.76977434965 -> xyz=1.75923056352 1.44162550321 0.928389521988 rpy=0.0 0.0 1.70377198488
- joint panda1_joint_base_link: origin xyz=2.11001260883 2.11178463597 0.431667235678 rpy=0.0 0.0 6.11172683293 -> xyz=0.774114225191 1.25002770761 0.667934137264 rpy=0.0 0.0 0.593966399677

File: eTaSL/robots/custom_robots.urdf.xacro (robot description, xacro)
@@ -6,6 +6,6 @@
 <link name="base_link"/>
 <!-- BODY BEGIN -->
-<xacro:indy7_robot robot_id="0" xyz="0.818223732196 1.39940643743 0.20048313416" rpy="0 0 0.76977434965" connected_to="base_link"/>
-<xacro:panda_robot robot_id="1" xyz="2.11001260883 2.11178463597 0.431667235678" rpy="0 0 6.11172683293" connected_to="base_link"/>
+<xacro:indy7_robot robot_id="0" xyz="1.75923056352 1.44162550321 0.928389521988" rpy="0 0 1.70377198488" connected_to="base_link"/>
+<xacro:panda_robot robot_id="1" xyz="0.774114225191 1.25002770761 0.667934137264" rpy="0 0 0.593966399677" connected_to="base_link"/>
 <!-- BODY END -->
 </robot>

Commit message: sample/render/log/log/reset all tested

File: eTaSL/robots/custom_robots.urdf (robot description, URDF)
Before this commit: robot custom_robots, 21 links, 20 joints
Joints:
- joint indy0_joint_base_link: origin xyz=1.75923056352 1.44162550321 0.928389521988 rpy=0.0 0.0 1.70377198488 -> xyz=1.8673293866 1.89028673102 0.713460100451 rpy=0.0 0.0 0.909418703579
- joint panda1_joint_base_link: origin xyz=0.774114225191 1.25002770761 0.667934137264 rpy=0.0 0.0 0.593966399677 -> xyz=0.895389168739 1.10016349925 0.985631874607 rpy=0.0 0.0 0.295217683068

File: eTaSL/robots/custom_robots.urdf.xacro (robot description, xacro)
@@ -6,6 +6,6 @@
 <link name="base_link"/>
 <!-- BODY BEGIN -->
-<xacro:indy7_robot robot_id="0" xyz="1.75923056352 1.44162550321 0.928389521988" rpy="0 0 1.70377198488" connected_to="base_link"/>
-<xacro:panda_robot robot_id="1" xyz="0.774114225191 1.25002770761 0.667934137264" rpy="0 0 0.593966399677" connected_to="base_link"/>
+<xacro:indy7_robot robot_id="0" xyz="1.8673293866 1.89028673102 0.713460100451" rpy="0 0 0.909418703579" connected_to="base_link"/>
+<xacro:panda_robot robot_id="1" xyz="0.895389168739 1.10016349925 0.985631874607" rpy="0 0 0.295217683068" connected_to="base_link"/>
 <!-- BODY END -->
 </robot>

Commit message: planning all tested, only collecting left

File: eTaSL/robots/custom_robots.urdf (robot description, URDF)
Before this commit: robot custom_robots, 21 links, 20 joints
Joints:
- joint indy0_joint_base_link: origin xyz=1.8673293866 1.89028673102 0.713460100451 rpy=0.0 0.0 0.909418703579 -> xyz=1.50934970355 1.05857786809 0.618023227199 rpy=0.0 0.0 0.0877825382904
- joint panda1_joint_base_link: origin xyz=0.895389168739 1.10016349925 0.985631874607 rpy=0.0 0.0 0.295217683068 -> xyz=1.86082969693 2.15357643241 0.516919315114 rpy=0.0 0.0 5.00609329319

File: eTaSL/robots/custom_robots.urdf.xacro (robot description, xacro)
@@ -6,6 +6,6 @@
 <link name="base_link"/>
 <!-- BODY BEGIN -->
-<xacro:indy7_robot robot_id="0" xyz="1.8673293866 1.89028673102 0.713460100451" rpy="0 0 0.909418703579" connected_to="base_link"/>
-<xacro:panda_robot robot_id="1" xyz="0.895389168739 1.10016349925 0.985631874607" rpy="0 0 0.295217683068" connected_to="base_link"/>
+<xacro:indy7_robot robot_id="0" xyz="1.50934970355 1.05857786809 0.618023227199" rpy="0 0 0.0877825382904" connected_to="base_link"/>
+<xacro:panda_robot robot_id="1" xyz="1.86082969693 2.15357643241 0.516919315114" rpy="0 0 5.00609329319" connected_to="base_link"/>
 <!-- BODY END -->
 </robot>

Commit message: kichen scene geometry added

File: eTaSL/robots/custom_robots.urdf (robot description, URDF)
Before this commit: robot custom_robots, 21 links, 20 joints
Joints:
- joint indy0_joint_base_link: origin xyz=1.50934970355 1.05857786809 0.618023227199 rpy=0.0 0.0 0.0877825382904 -> xyz=0.0 0.0 0.0 rpy=0.0 0.0 3.14159265359
- joint panda1_joint_base_link: origin xyz=1.86082969693 2.15357643241 0.516919315114 rpy=0.0 0.0 5.00609329319 -> xyz=-1.4 1.1 -0.1 rpy=0.0 0.0 0.0

File: eTaSL/robots/custom_robots.urdf.xacro (robot description, xacro)
@@ -6,6 +6,6 @@
 <link name="base_link"/>
 <!-- BODY BEGIN -->
-<xacro:indy7_robot robot_id="0" xyz="1.50934970355 1.05857786809 0.618023227199" rpy="0 0 0.0877825382904" connected_to="base_link"/>
-<xacro:panda_robot robot_id="1" xyz="1.86082969693 2.15357643241 0.516919315114" rpy="0 0 5.00609329319" connected_to="base_link"/>
+<xacro:indy7_robot robot_id="0" xyz="0 0 0.0" rpy="0 0 3.14159265359" connected_to="base_link"/>
+<xacro:panda_robot robot_id="1" xyz="-1.4 1.1 -0.1" rpy="0 0 0" connected_to="base_link"/>
 <!-- BODY END -->
 </robot>

Commit message: --

File: eTaSL/robots/custom_robots.urdf (robot description, URDF)
Before this commit: robot custom_robots, 21 links, 20 joints
Joints:
- joint indy0_joint_base_link: origin xyz=0.0 0.0 0.0 rpy=0.0 0.0 3.14159265359 -> xyz=1.23162009238 0.803964211372 0.845043883176 rpy=0.0 0.0 2.24780547472
- joint panda1_joint_base_link: origin xyz=-1.4 1.1 -0.1 rpy=0.0 0.0 0.0 -> xyz=0.834052969431 1.75733693695 0.805944548947 rpy=0.0 0.0 6.07944828478

File: eTaSL/robots/custom_robots.urdf.xacro (robot description, xacro)
@@ -6,6 +6,6 @@
 <link name="base_link"/>
 <!-- BODY BEGIN -->
-<xacro:indy7_robot robot_id="0" xyz="0 0 0.0" rpy="0 0 3.14159265359" connected_to="base_link"/>
-<xacro:panda_robot robot_id="1" xyz="-1.4 1.1 -0.1" rpy="0 0 0" connected_to="base_link"/>
+<xacro:indy7_robot robot_id="0" xyz="1.23162009238 0.803964211372 0.845043883176" rpy="0 0 2.24780547472" connected_to="base_link"/>
+<xacro:panda_robot robot_id="1" xyz="0.834052969431 1.75733693695 0.805944548947" rpy="0 0 6.07944828478" connected_to="base_link"/>
 <!-- BODY END -->
 </robot>

Commit message: dual arm chain urdf, srdf generation

File: eTaSL/robots/custom_robots.urdf (robot description, URDF)
Before this commit: robot custom_robots, 21 links, 20 joints
Joints:
- joint indy0_joint_base_link: origin xyz=1.23162009238 0.803964211372 0.845043883176 rpy=0.0 0.0 2.24780547472 -> xyz=1.90436312731 1.82265572042 0.570589558192 rpy=0.0 0.0 4.50243087359
- joint panda1_joint_base_link: origin xyz=0.834052969431 1.75733693695 0.805944548947 rpy=0.0 0.0 6.07944828478 -> xyz=1.43408856909 0.833387160458 0.818965615746 rpy=0.0 0.0 4.34286812062

File: eTaSL/robots/custom_robots.urdf.xacro (robot description, xacro)
@@ -2,10 +2,10 @@
 <robot xmlns:xacro="http://www.ros.org/wiki/xacro" name="custom_robots">
 <xacro:include filename="$(find indy7_description)/urdf/materials.xacro"/>
-<xacro:include filename="$(env TAMP_ETASL_DIR)/robots/panda_robot.xacro"/>
-<xacro:include filename="$(env TAMP_ETASL_DIR)/robots/indy7_robot.xacro"/>
+<xacro:include filename="$(env TAMP_ETASL_DIR)/robots/panda.xacro"/>
+<xacro:include filename="$(env TAMP_ETASL_DIR)/robots/indy7.xacro"/>
 <link name="base_link"/>
 <!-- BODY BEGIN -->
-<xacro:indy7_robot robot_id="0" xyz="1.23162009238 0.803964211372 0.845043883176" rpy="0 0 2.24780547472" connected_to="base_link"/>
-<xacro:panda_robot robot_id="1" xyz="0.834052969431 1.75733693695 0.805944548947" rpy="0 0 6.07944828478" connected_to="base_link"/>
+<xacro:indy7 robot_id="0" xyz="1.90436312731 1.82265572042 0.570589558192" rpy="0 0 4.50243087359" connected_to="base_link"/>
+<xacro:panda robot_id="1" xyz="1.43408856909 0.833387160458 0.818965615746" rpy="0 0 4.34286812062" connected_to="base_link"/>
 <!-- BODY END -->
 </robot>

File: eTaSL/robots/indy7_robot-bak.xacro (robot description, xacro)
@@ -1,5 +1,5 @@
 <?xml version="1.0" ?>
 <robot name="indy7" xmlns:xacro="http://ros.org/wiki/xacro">
-  <xacro:macro name="indy7_robot" params="robot_id:='indy7' description_pkg:='indy7_description' connected_to:='' xyz:='0 0 0' rpy:='0 0 0'">
+  <xacro:macro name="indy7" params="robot_id:='indy7' description_pkg:='indy7_description' connected_to:='' xyz:='0 0 0' rpy:='0 0 0'">
     <xacro:unless value="${not connected_to}">
       <joint name="indy${robot_id}_joint_${connected_to}" type="fixed">

Commit message: dual arm chain full tested

File: eTaSL/robots/custom_robots.urdf (robot description, URDF)
Before this commit: robot custom_robots, 21 links, 20 joints
Joints:
- joint indy0_joint_base_link: origin xyz=1.90436312731 1.82265572042 0.570589558192 rpy=0.0 0.0 4.50243087359 -> xyz=1.14054548973 1.46580839478 0.582147288053 rpy=0.0 0.0 3.28684256351
- joint panda1_joint_base_link: origin xyz=1.43408856909 0.833387160458 0.818965615746 rpy=0.0 0.0 4.34286812062 -> xyz=2.23049371307 0.936092023629 0.921214813765 rpy=0.0 0.0 0.75277710184

File: eTaSL/robots/custom_robots.urdf.xacro (robot description, xacro)
@@ -6,6 +6,6 @@
 <link name="base_link"/>
 <!-- BODY BEGIN -->
-<xacro:indy7 robot_id="0" xyz="1.90436312731 1.82265572042 0.570589558192" rpy="0 0 4.50243087359" connected_to="base_link"/>
-<xacro:panda robot_id="1" xyz="1.43408856909 0.833387160458 0.818965615746" rpy="0 0 4.34286812062" connected_to="base_link"/>
+<xacro:indy7 robot_id="0" xyz="1.14054548973 1.46580839478 0.582147288053" rpy="0 0 3.28684256351" connected_to="base_link"/>
+<xacro:panda robot_id="1" xyz="2.23049371307 0.936092023629 0.921214813765" rpy="0 0 0.75277710184" connected_to="base_link"/>
 <!-- BODY END -->
 </robot>

File: eTaSL/robots/custom_robots_indy0_panda1.urdf (robot description, URDF)
Before this commit: robot custom_robots, 21 links, 20 joints
Links:
- added link stem
Joints:
- added joint stem_joint_base_link: type fixed, parent stem, child base_link, origin xyz=1.34069597721 1.28529083729 -0.582147300243 rpy=0.0 -0.0 2.99634273926
- joint indy0_joint_base_link: child base_link -> stem
- joint panda1_joint_base_link: origin xyz=1.13134251381 0.991934190815 0.949680852372 rpy=0.0 0.0 2.67668032996 -> xyz=2.23049371307 0.936092023629 0.921214813765 rpy=0.0 0.0 0.75277710184

File: eTaSL/robots/custom_robots_panda1_indy0.urdf (robot description, URDF)
Before this commit: robot custom_robots, 21 links, 20 joints
Links:
- added link stem
Joints:
- added joint stem_joint_base_link: type fixed, parent stem, child base_link, origin xyz=-2.26777505875 0.841763913631 -0.921214818954 rpy=0.0 -0.0 -0.752777081056
- joint indy0_joint_base_link: origin xyz=1.58721767288 1.818021349 0.593100988132 rpy=0.0 0.0 3.62548851476 -> xyz=1.14054548973 1.46580839478 0.582147288053 rpy=0.0 0.0 3.28684256351
- joint panda1_joint1: limit lower=-0.0479965544298 upper=0.0479965544298 effort=3.14159265359 velocity=1.308996939 -> lower=-2.75 upper=2.75 effort=3.14159265359 velocity=1.308996939
- joint panda1_joint2: limit lower=-0.0296705972839 upper=0.0296705972839 effort=3.14159265359 velocity=1.308996939 -> lower=-1.7 upper=1.7 effort=3.14159265359 velocity=1.308996939
- joint panda1_joint3: limit lower=-0.0479965544298 upper=0.0479965544298 effort=3.14159265359 velocity=1.308996939 -> lower=-2.75 upper=2.75 effort=3.14159265359 velocity=1.308996939
- joint panda1_joint4: limit lower=-0.0506145483078 upper=-0.00174532925199 effort=3.14159265359 velocity=1.308996939 -> lower=0.1 upper=2.9 effort=3.14159265359 velocity=1.308996939
- joint panda1_joint5: limit lower=-0.0479965544298 upper=0.0479965544298 effort=3.14159265359 velocity=1.57079632679 -> lower=-2.75 upper=2.75 effort=3.14159265359 velocity=1.57079632679
- joint panda1_joint6: limit lower=0.00174532925199 upper=0.0628318530718 effort=3.14159265359 velocity=1.57079632679 -> lower=-3.6 upper=-0.1 effort=3.14159265359 velocity=1.57079632679
- joint panda1_joint7: limit lower=-0.0479965544298 upper=0.0479965544298 effort=3.14159265359 velocity=1.57079632679 -> lower=-2.75 upper=2.75 effort=3.14159265359 velocity=1.57079632679
- joint panda1_joint_base_link: child base_link -> stem

Commit message: sample data collecting started

File: eTaSL/robots/custom_robots.urdf (robot description, URDF)
Before this commit: robot custom_robots, 21 links, 20 joints
Joints:
- joint indy0_joint_base_link: origin xyz=1.14054548973 1.46580839478 0.582147288053 rpy=0.0 0.0 3.28684256351 -> xyz=2.13872755421 1.7628075055 0.7771689317 rpy=0.0 0.0 0.941098854331
- joint panda1_joint_base_link: origin xyz=2.23049371307 0.936092023629 0.921214813765 rpy=0.0 0.0 0.75277710184 -> xyz=1.43344570825 1.01587451249 0.76331541696 rpy=0.0 0.0 3.86931438791

File: eTaSL/robots/custom_robots.urdf.xacro (robot description, xacro)
@@ -6,6 +6,6 @@
 <link name="base_link"/>
 <!-- BODY BEGIN -->
-<xacro:indy7 robot_id="0" xyz="1.14054548973 1.46580839478 0.582147288053" rpy="0 0 3.28684256351" connected_to="base_link"/>
-<xacro:panda robot_id="1" xyz="2.23049371307 0.936092023629 0.921214813765" rpy="0 0 0.75277710184" connected_to="base_link"/>
+<xacro:indy7 robot_id="0" xyz="2.13872755421 1.7628075055 0.7771689317" rpy="0 0 0.941098854331" connected_to="base_link"/>
+<xacro:panda robot_id="1" xyz="1.43344570825 1.01587451249 0.76331541696" rpy="0 0 3.86931438791" connected_to="base_link"/>
 <!-- BODY END -->
 </robot>

File: eTaSL/robots/custom_robots_indy0_panda1.urdf (robot description, URDF)
Before this commit: robot custom_robots, 22 links, 21 joints
Joints:
- joint panda1_joint_base_link: origin xyz=2.23049371307 0.936092023629 0.921214813765 rpy=0.0 0.0 0.75277710184 -> xyz=1.43344570825 1.01587451249 0.76331541696 rpy=0.0 0.0 3.86931438791
- joint stem_joint_base_link: origin xyz=1.34069597721 1.28529083729 -0.582147300243 rpy=0.0 -0.0 2.99634273926 -> xyz=-2.6842083931 0.690414190292 -0.777168929577 rpy=0.0 -0.0 -0.941098876031

File: eTaSL/robots/custom_robots_panda1_indy0.urdf (robot description, URDF)
Before this commit: robot custom_robots, 22 links, 21 joints
Joints:
- joint indy0_joint_base_link: origin xyz=1.14054548973 1.46580839478 0.582147288053 rpy=0.0 0.0 3.28684256351 -> xyz=2.13872755421 1.7628075055 0.7771689317 rpy=0.0 0.0 0.941098854331
- joint stem_joint_base_link: origin xyz=-2.26777505875 0.841763913631 -0.921214818954 rpy=0.0 -0.0 -0.752777081056 -> xyz=1.74607157707 -0.194940268993 -0.763315439224 rpy=0.0 -0.0 2.41387091849

Commit message: data reenacting implemented

File: eTaSL/robots/custom_robots.urdf (robot description, URDF)
Before this commit: robot custom_robots, 21 links, 20 joints
Joints:
- joint indy0_joint_base_link: origin xyz=2.13872755421 1.7628075055 0.7771689317 rpy=0.0 0.0 0.941098854331 -> xyz=0.948989658221 2.20148041906 0.957612918454 rpy=0.0 0.0 0.528719669396
- joint panda1_joint_base_link: origin xyz=1.43344570825 1.01587451249 0.76331541696 rpy=0.0 0.0 3.86931438791 -> xyz=2.21749448523 2.07076125055 0.870863802837 rpy=0.0 0.0 3.14368247595

File: eTaSL/robots/custom_robots.urdf.xacro (robot description, xacro)
@@ -6,6 +6,6 @@
 <link name="base_link"/>
 <!-- BODY BEGIN -->
-<xacro:indy7 robot_id="0" xyz="2.13872755421 1.7628075055 0.7771689317" rpy="0 0 0.941098854331" connected_to="base_link"/>
-<xacro:panda robot_id="1" xyz="1.43344570825 1.01587451249 0.76331541696" rpy="0 0 3.86931438791" connected_to="base_link"/>
+<xacro:indy7 robot_id="0" xyz="0.948989658221 2.20148041906 0.957612918454" rpy="0 0 0.528719669396" connected_to="base_link"/>
+<xacro:panda robot_id="1" xyz="2.21749448523 2.07076125055 0.870863802837" rpy="0 0 3.14368247595" connected_to="base_link"/>
 <!-- BODY END -->
 </robot>

File: eTaSL/robots/custom_robots_indy0_panda1.urdf (robot description, URDF)
Before this commit: robot custom_robots, 22 links, 21 joints
Joints:
- joint panda1_joint_base_link: origin xyz=1.43344570825 1.01587451249 0.76331541696 rpy=0.0 0.0 3.86931438791 -> xyz=2.21749448523 2.07076125055 0.870863802837 rpy=0.0 0.0 3.14368247595
- joint stem_joint_base_link: origin xyz=-2.6842083931 0.690414190292 -0.777168929577 rpy=0.0 -0.0 -0.941098876031 -> xyz=-1.92989742756 -1.4221791029 -0.957612931728 rpy=0.0 -0.0 -0.528719678579

File: eTaSL/robots/custom_robots_panda1_indy0.urdf (robot description, URDF)
Before this commit: robot custom_robots, 22 links, 21 joints
Joints:
- joint indy0_joint_base_link: origin xyz=2.13872755421 1.7628075055 0.7771689317 rpy=0.0 0.0 0.941098854331 -> xyz=0.948989658221 2.20148041906 0.957612918454 rpy=0.0 0.0 0.528719669396
- joint stem_joint_base_link: origin xyz=1.74607157707 -0.194940268993 -0.763315439224 rpy=0.0 -0.0 2.41387091849 -> xyz=2.2218170166 2.06612253189 -0.87086379528 rpy=0.0 -0.0 3.13950283122
