Commit message: check data rechecked

File: eTaSL/robots/custom_robots.urdf (robot description, URDF)
Before this commit: robot custom_robots, 21 links, 20 joints
Joints:
- joint indy0_joint_base_link: origin xyz=0.948989658221 2.20148041906 0.957612918454 rpy=0.0 0.0 0.528719669396 -> xyz=1.20560620407 1.66640783429 0.621808362521 rpy=0.0 0.0 1.17753509285
- joint panda1_joint_base_link: origin xyz=2.21749448523 2.07076125055 0.870863802837 rpy=0.0 0.0 3.14368247595 -> xyz=2.17124796286 0.872187764433 0.935632393364 rpy=0.0 0.0 3.83301494299

File: eTaSL/robots/custom_robots.urdf.xacro (robot description, xacro)
@@ -6,6 +6,6 @@
 <link name="base_link"/>
 <!-- BODY BEGIN -->
-<xacro:indy7 robot_id="0" xyz="0.948989658221 2.20148041906 0.957612918454" rpy="0 0 0.528719669396" connected_to="base_link"/>
-<xacro:panda robot_id="1" xyz="2.21749448523 2.07076125055 0.870863802837" rpy="0 0 3.14368247595" connected_to="base_link"/>
+<xacro:indy7 robot_id="0" xyz="1.20560620407 1.66640783429 0.621808362521" rpy="0 0 1.17753509285" connected_to="base_link"/>
+<xacro:panda robot_id="1" xyz="2.17124796286 0.872187764433 0.935632393364" rpy="0 0 3.83301494299" connected_to="base_link"/>
 <!-- BODY END -->
 </robot>

File: eTaSL/robots/custom_robots_indy0_panda1.urdf (robot description, URDF)
Before this commit: robot custom_robots, 22 links, 21 joints
Joints:
- joint panda1_joint_base_link: origin xyz=2.21749448523 2.07076125055 0.870863802837 rpy=0.0 0.0 3.14368247595 -> xyz=2.17124796286 0.872187764433 0.935632393364 rpy=0.0 0.0 3.83301494299
- joint stem_joint_base_link: origin xyz=-1.92989742756 -1.4221791029 -0.957612931728 rpy=0.0 -0.0 -0.528719678579 -> xyz=-2.00119304657 0.475003302097 -0.621808350086 rpy=0.0 -0.0 -1.17753509843

File: eTaSL/robots/custom_robots_panda1_indy0.urdf (robot description, URDF)
Before this commit: robot custom_robots, 22 links, 21 joints
Joints:
- joint indy0_joint_base_link: origin xyz=0.948989658221 2.20148041906 0.957612918454 rpy=0.0 0.0 0.528719669396 -> xyz=1.20560620407 1.66640783429 0.621808362521 rpy=0.0 0.0 1.17753509285
- joint stem_joint_base_link: origin xyz=2.2218170166 2.06612253189 -0.87086379528 rpy=0.0 -0.0 3.13950283122 -> xyz=2.22873497009 -0.712579369545 -0.935632407665 rpy=0.0 -0.0 2.45017034859

Commit message: converting data - to cell geometries

File: eTaSL/robots/custom_robots.urdf (robot description, URDF)
Before this commit: robot custom_robots, 21 links, 20 joints
Joints:
- joint indy0_joint_base_link: origin xyz=1.20560620407 1.66640783429 0.621808362521 rpy=0.0 0.0 1.17753509285 -> xyz=2.20429158474 2.04517986435 0.868477234851 rpy=0.0 0.0 0.123801134058
- joint panda1_joint_base_link: origin xyz=2.17124796286 0.872187764433 0.935632393364 rpy=0.0 0.0 3.83301494299 -> xyz=0.780553312561 1.57486136784 0.709225725298 rpy=0.0 0.0 1.59878880455

File: eTaSL/robots/custom_robots.urdf.xacro (robot description, xacro)
@@ -6,6 +6,6 @@
 <link name="base_link"/>
 <!-- BODY BEGIN -->
-<xacro:indy7 robot_id="0" xyz="1.20560620407 1.66640783429 0.621808362521" rpy="0 0 1.17753509285" connected_to="base_link"/>
-<xacro:panda robot_id="1" xyz="2.17124796286 0.872187764433 0.935632393364" rpy="0 0 3.83301494299" connected_to="base_link"/>
+<xacro:indy7 robot_id="0" xyz="2.20429158474 2.04517986435 0.868477234851" rpy="0 0 0.123801134058" connected_to="base_link"/>
+<xacro:panda robot_id="1" xyz="0.780553312561 1.57486136784 0.709225725298" rpy="0 0 1.59878880455" connected_to="base_link"/>
 <!-- BODY END -->
 </robot>

File: eTaSL/robots/custom_robots_indy0_panda1.urdf (robot description, URDF)
Before this commit: robot custom_robots, 22 links, 21 joints
Joints:
- joint panda1_joint_base_link: origin xyz=2.17124796286 0.872187764433 0.935632393364 rpy=0.0 0.0 3.83301494299 -> xyz=0.780553312561 1.57486136784 0.709225725298 rpy=0.0 0.0 1.59878880455
- joint stem_joint_base_link: origin xyz=-2.00119304657 0.475003302097 -0.621808350086 rpy=0.0 -0.0 -1.17753509843 -> xyz=-2.43997001648 -1.75732970238 -0.868477225304 rpy=0.0 -0.0 -0.123801137053

File: eTaSL/robots/custom_robots_panda1_indy0.urdf (robot description, URDF)
Before this commit: robot custom_robots, 22 links, 21 joints
Joints:
- joint indy0_joint_base_link: origin xyz=1.20560620407 1.66640783429 0.621808362521 rpy=0.0 0.0 1.17753509285 -> xyz=2.20429158474 2.04517986435 0.868477234851 rpy=0.0 0.0 0.123801134058
- joint stem_joint_base_link: origin xyz=2.22873497009 -0.712579369545 -0.935632407665 rpy=0.0 -0.0 2.45017034859 -> xyz=-1.55239760876 0.824326038361 -0.709225714207 rpy=0.0 -0.0 -1.59878880413

Commit message: convert data done

File: eTaSL/robots/custom_robots.urdf (robot description, URDF)
Before this commit: robot custom_robots, 21 links, 20 joints
Joints:
- joint indy0_joint_base_link: origin xyz=2.20429158474 2.04517986435 0.868477234851 rpy=0.0 0.0 0.123801134058 -> xyz=1.4265382828 1.99640271031 0.784441997166 rpy=0.0 0.0 6.08376513315
- joint panda1_joint_base_link: origin xyz=0.780553312561 1.57486136784 0.709225725298 rpy=0.0 0.0 1.59878880455 -> xyz=1.78866435412 1.08539320784 0.513434825839 rpy=0.0 0.0 0.203734766538

File: eTaSL/robots/custom_robots.urdf.xacro (robot description, xacro)
@@ -6,6 +6,6 @@
 <link name="base_link"/>
 <!-- BODY BEGIN -->
-<xacro:indy7 robot_id="0" xyz="2.20429158474 2.04517986435 0.868477234851" rpy="0 0 0.123801134058" connected_to="base_link"/>
-<xacro:panda robot_id="1" xyz="0.780553312561 1.57486136784 0.709225725298" rpy="0 0 1.59878880455" connected_to="base_link"/>
+<xacro:indy7 robot_id="0" xyz="1.4265382828 1.99640271031 0.784441997166" rpy="0 0 6.08376513315" connected_to="base_link"/>
+<xacro:panda robot_id="1" xyz="1.78866435412 1.08539320784 0.513434825839" rpy="0 0 0.203734766538" connected_to="base_link"/>
 <!-- BODY END -->
 </robot>

File: eTaSL/robots/custom_robots_indy0_panda1.urdf (robot description, URDF)
Before this commit: robot custom_robots, 22 links, 21 joints
Joints:
- joint panda1_joint_base_link: origin xyz=0.780553312561 1.57486136784 0.709225725298 rpy=0.0 0.0 1.59878880455 -> xyz=1.64384372581 2.22911003969 0.701622466653 rpy=0.0 0.0 2.4712516767
- joint stem_joint_base_link: origin xyz=-2.43997001648 -1.75732970238 -0.868477225304 rpy=0.0 -0.0 -0.123801137053 -> xyz=1.20828998089 -1.20012688637 -0.730634570122 rpy=0.0 -0.0 1.27359020764

File: eTaSL/robots/custom_robots_panda1_indy0.urdf (robot description, URDF)
Before this commit: robot custom_robots, 22 links, 21 joints
Joints:
- joint indy0_joint_base_link: origin xyz=2.20429158474 2.04517986435 0.868477234851 rpy=0.0 0.0 0.123801134058 -> xyz=0.793663700935 1.50677374563 0.730634550362 rpy=0.0 0.0 5.00959510631
- joint stem_joint_base_link: origin xyz=-1.55239760876 0.824326038361 -0.709225714207 rpy=0.0 -0.0 -1.59878880413 -> xyz=-0.0967094898224 2.76799583435 -0.701622486115 rpy=0.0 -0.0 -2.47125168813

Commit message: loading scene

File: eTaSL/robots/custom_robots.urdf (robot description, URDF)
Before this commit: robot custom_robots, 21 links, 20 joints
Joints:
- joint indy0_joint_base_link: origin xyz=1.4265382828 1.99640271031 0.784441997166 rpy=0.0 0.0 6.08376513315 -> xyz=0.793663700935 1.50677374563 0.730634550362 rpy=0.0 0.0 5.00959510631
- joint panda1_joint_base_link: origin xyz=1.78866435412 1.08539320784 0.513434825839 rpy=0.0 0.0 0.203734766538 -> xyz=1.64384372581 2.22911003969 0.701622466653 rpy=0.0 0.0 2.4712516767

File: eTaSL/robots/custom_robots.urdf.xacro (robot description, xacro)
@@ -6,6 +6,6 @@
 <link name="base_link"/>
 <!-- BODY BEGIN -->
-<xacro:indy7 robot_id="0" xyz="1.4265382828 1.99640271031 0.784441997166" rpy="0 0 6.08376513315" connected_to="base_link"/>
-<xacro:panda robot_id="1" xyz="1.78866435412 1.08539320784 0.513434825839" rpy="0 0 0.203734766538" connected_to="base_link"/>
+<xacro:indy7 robot_id="0" xyz="0.793663700935 1.50677374563 0.730634550362" rpy="0 0 5.00959510631" connected_to="base_link"/>
+<xacro:panda robot_id="1" xyz="1.64384372581 2.22911003969 0.701622466653" rpy="0 0 2.4712516767" connected_to="base_link"/>
 <!-- BODY END -->
 </robot>

File: eTaSL/robots/custom_robots_indy0_panda1.urdf (robot description, URDF)
Before this commit: robot custom_robots, 22 links, 21 joints
Joints:
- joint panda1_joint_base_link: origin xyz=1.64384372581 2.22911003969 0.701622466653 rpy=0.0 0.0 2.4712516767 -> xyz=2.09178725976 1.79130520417 0.559874914025 rpy=0.0 0.0 2.33434042526
- joint stem_joint_base_link: origin xyz=1.20828998089 -1.20012688637 -0.730634570122 rpy=0.0 -0.0 1.27359020764 -> xyz=0.419996738434 -2.06658935547 -0.500553131104 rpy=0.0 -0.0 0.737355161022

File: eTaSL/robots/custom_robots_panda1_indy0.urdf (robot description, URDF)
Before this commit: robot custom_robots, 22 links, 21 joints
Joints:
- joint indy0_joint_base_link: origin xyz=0.793663700935 1.50677374563 0.730634550362 rpy=0.0 0.0 5.00959510631 -> xyz=1.07853271998 1.8121689086 0.500553136673 rpy=0.0 0.0 5.5458301331
- joint stem_joint_base_link: origin xyz=-0.0967094898224 2.76799583435 -0.701622486115 rpy=0.0 -0.0 -2.47125168813 -> xyz=0.15242087841 2.7497484684 -0.559874892235 rpy=0.0 -0.0 -2.33434041074

Commit message: structured network training

File: eTaSL/robots/custom_robots.urdf (robot description, URDF)
Before this commit: robot custom_robots, 21 links, 20 joints
Joints:
- joint indy0_joint_base_link: origin xyz=0.793663700935 1.50677374563 0.730634550362 rpy=0.0 0.0 5.00959510631 -> xyz=1.84112781679 0.933416006597 0.64192495556 rpy=0.0 0.0 5.95316536284
- joint panda1_joint_base_link: origin xyz=1.64384372581 2.22911003969 0.701622466653 rpy=0.0 0.0 2.4712516767 -> xyz=0.899744439262 1.42486487413 0.960543345375 rpy=0.0 0.0 1.0299310825

File: eTaSL/robots/custom_robots.urdf.xacro (robot description, xacro)
@@ -6,6 +6,6 @@
 <link name="base_link"/>
 <!-- BODY BEGIN -->
-<xacro:indy7 robot_id="0" xyz="0.793663700935 1.50677374563 0.730634550362" rpy="0 0 5.00959510631" connected_to="base_link"/>
-<xacro:panda robot_id="1" xyz="1.64384372581 2.22911003969 0.701622466653" rpy="0 0 2.4712516767" connected_to="base_link"/>
+<xacro:indy7 robot_id="0" xyz="1.84112781679 0.933416006597 0.64192495556" rpy="0 0 5.95316536284" connected_to="base_link"/>
+<xacro:panda robot_id="1" xyz="0.899744439262 1.42486487413 0.960543345375" rpy="0 0 1.0299310825" connected_to="base_link"/>
 <!-- BODY END -->
 </robot>

File: eTaSL/robots/custom_robots_indy0_panda1.urdf (robot description, URDF)
Before this commit: robot custom_robots, 22 links, 21 joints
Joints:
- joint panda1_joint_base_link: origin xyz=2.09178725976 1.79130520417 0.559874914025 rpy=0.0 0.0 2.33434042526 -> xyz=0.899744439262 1.42486487413 0.960543345375 rpy=0.0 0.0 1.0299310825
- joint stem_joint_base_link: origin xyz=0.419996738434 -2.06658935547 -0.500553131104 rpy=0.0 -0.0 0.737355161022 -> xyz=-1.43928837776 -1.47968435287 -0.641924977303 rpy=0.0 -0.0 0.330019953999

File: eTaSL/robots/custom_robots_panda1_indy0.urdf (robot description, URDF)
Before this commit: robot custom_robots, 22 links, 21 joints
Joints:
- joint indy0_joint_base_link: origin xyz=1.07853271998 1.8121689086 0.500553136673 rpy=0.0 0.0 5.5458301331 -> xyz=1.84112781679 0.933416006597 0.64192495556 rpy=0.0 0.0 5.95316536284
- joint stem_joint_base_link: origin xyz=0.15242087841 2.7497484684 -0.559874892235 rpy=0.0 -0.0 -2.33434041074 -> xyz=-1.68474316597 0.03768658638 -0.960543334484 rpy=0.0 -0.0 -1.0299310913

Commit message: save_tmp

File: eTaSL/robots/custom_robots.urdf (robot description, URDF)
Before this commit: robot custom_robots, 21 links, 20 joints
Joints:
- joint indy0_joint_base_link: origin xyz=1.84112781679 0.933416006597 0.64192495556 rpy=0.0 0.0 5.95316536284 -> xyz=-0.447842508554 0.252281308174 0.00795543193817 rpy=-0.000699172050315 0.00570982817079 -1.59473908718
- joint panda1_joint_base_link: origin xyz=0.899744439262 1.42486487413 0.960543345375 rpy=0.0 0.0 1.0299310825 -> xyz=0.511233150959 0.157657206059 0.012868642807 rpy=0.00131621839311 -3.37064275204e-05 -1.61483536451

File: eTaSL/robots/custom_robots.urdf.xacro (robot description, xacro)
@@ -6,6 +6,6 @@
 <link name="base_link"/>
 <!-- BODY BEGIN -->
-<xacro:indy7 robot_id="0" xyz="1.84112781679 0.933416006597 0.64192495556" rpy="0 0 5.95316536284" connected_to="base_link"/>
-<xacro:panda robot_id="1" xyz="0.899744439262 1.42486487413 0.960543345375" rpy="0 0 1.0299310825" connected_to="base_link"/>
+<xacro:indy7 robot_id="0" xyz="-0.447842508554 0.252281308174 0.00795543193817" rpy="-0.000699172050315 0.00570982817079 -1.59473908718" connected_to="base_link"/>
+<xacro:panda robot_id="1" xyz="0.511233150959 0.157657206059 0.012868642807" rpy="0.00131621839311 -3.37064275204e-05 -1.61483536451" connected_to="base_link"/>
 <!-- BODY END -->
 </robot>

File: eTaSL/robots/custom_robots_indy0_panda1.urdf (robot description, URDF)
Before this commit: robot custom_robots, 22 links, 21 joints
Joints:
- joint panda1_joint_base_link: origin xyz=0.899744439262 1.42486487413 0.960543345375 rpy=0.0 0.0 1.0299310825 -> xyz=0.87606235504 1.13347322658 0.685762418466 rpy=0.0 0.0 4.50983292483
- joint stem_joint_base_link: origin xyz=-1.43928837776 -1.47968435287 -0.641924977303 rpy=0.0 -0.0 0.330019953999 -> xyz=1.09260034561 -2.13035464287 -0.845345258713 rpy=0.0 -0.0 1.66813374687

File: eTaSL/robots/custom_robots_panda1_indy0.urdf (robot description, URDF)
Before this commit: robot custom_robots, 22 links, 21 joints
Joints:
- joint indy0_joint_base_link: origin xyz=1.84112781679 0.933416006597 0.64192495556 rpy=0.0 0.0 5.95316536284 -> xyz=2.22645352325 0.880392530093 0.845345268103 rpy=0.0 0.0 4.61505156013
- joint stem_joint_base_link: origin xyz=-1.68474316597 0.03768658638 -0.960543334484 rpy=0.0 -0.0 -1.0299310913 -> xyz=1.2865408659 -0.630126595497 -0.685762405396 rpy=0.0 -0.0 1.773352385

Commit message: experiment debugged

File: eTaSL/robots/custom_robots.urdf (robot description, URDF)
Before this commit: robot custom_robots, 21 links, 20 joints
Links:
- link indy0_tcp: geometry collision cylinder length=0.083 radius=0.015; collision cylinder length=0.083 radius=0.015
- link panda1_link5: geometry collision cylinder length=0.12 radius=0.06; collision cylinder length=0.2 radius=0.08
Joints:
- joint indy0_joint0: limit lower=-3.05432619099 upper=3.05432619099 effort=3.141592653589793 velocity=1.3089969389957472 -> lower=-3.05432619099 upper=3.05432619099 effort=3.141592653589793 velocity=0.6544984694978736
- joint indy0_joint1: limit lower=-3.05432619099 upper=3.05432619099 effort=3.141592653589793 velocity=1.3089969389957472 -> lower=-3.05432619099 upper=3.05432619099 effort=3.141592653589793 velocity=0.6544984694978736
- joint indy0_joint2: limit lower=-3.05432619099 upper=3.05432619099 effort=3.141592653589793 velocity=1.3089969389957472 -> lower=-3.05432619099 upper=3.05432619099 effort=3.141592653589793 velocity=0.6544984694978736
- joint indy0_joint3: limit lower=-3.05432619099 upper=3.05432619099 effort=3.141592653589793 velocity=1.5707963267948966 -> lower=-3.05432619099 upper=3.05432619099 effort=3.141592653589793 velocity=0.7853981633974483
- joint indy0_joint4: limit lower=-3.05432619099 upper=3.05432619099 effort=3.141592653589793 velocity=1.5707963267948966 -> lower=-3.05432619099 upper=3.05432619099 effort=3.141592653589793 velocity=0.7853981633974483
- joint indy0_joint5: limit lower=-3.75245789179 upper=3.75245789179 effort=3.141592653589793 velocity=1.5707963267948966 -> lower=-3.75245789179 upper=3.75245789179 effort=3.141592653589793 velocity=0.7853981633974483
- joint indy0_joint_base_link: origin xyz=-0.447842508554 0.252281308174 0.00795543193817 rpy=-0.000699172050315 0.00570982817079 -1.59473908718 -> xyz=-0.444375276566 0.24876666069 0.0120660662651 rpy=-0.00347209485447 0.0010262729627 -1.58766529131
- joint panda1_joint1: limit lower=-2.75 upper=2.75 effort=3.141592653589793 velocity=1.3089969389957472 -> lower=-2.75 upper=2.75 effort=3.141592653589793 velocity=0.6544984694978736
- joint panda1_joint2: limit lower=-1.7 upper=1.7 effort=3.141592653589793 velocity=1.3089969389957472 -> lower=-1.7 upper=1.7 effort=3.141592653589793 velocity=0.6544984694978736
- joint panda1_joint3: limit lower=-2.75 upper=2.75 effort=3.141592653589793 velocity=1.3089969389957472 -> lower=-2.75 upper=2.75 effort=3.141592653589793 velocity=0.6544984694978736
- joint panda1_joint4: limit lower=-2.9 upper=-0.1 effort=3.141592653589793 velocity=1.3089969389957472 -> lower=-2.9 upper=-0.1 effort=3.141592653589793 velocity=0.6544984694978736
- joint panda1_joint5: limit lower=-2.75 upper=2.75 effort=3.141592653589793 velocity=1.5707963267948966 -> lower=-2.75 upper=2.75 effort=3.141592653589793 velocity=0.7853981633974483
- joint panda1_joint6: limit lower=0.1 upper=3.6 effort=3.141592653589793 velocity=1.5707963267948966 -> lower=0.1 upper=3.6 effort=3.141592653589793 velocity=0.7853981633974483
- joint panda1_joint7: limit lower=-2.75 upper=2.75 effort=3.141592653589793 velocity=1.5707963267948966 -> lower=-2.75 upper=2.75 effort=3.141592653589793 velocity=0.7853981633974483
- joint panda1_joint_base_link: origin xyz=0.511233150959 0.157657206059 0.012868642807 rpy=0.00131621839311 -3.37064275204e-05 -1.61483536451 -> xyz=0.512558698654 0.165808618069 0.0120181441307 rpy=-0.0016779836511 0.000554054982627 -1.60498128646

File: eTaSL/robots/custom_robots.urdf.xacro (robot description, xacro)
@@ -6,6 +6,6 @@
 <link name="base_link"/>
 <!-- BODY BEGIN -->
-<xacro:indy7 robot_id="0" xyz="-0.447842508554 0.252281308174 0.00795543193817" rpy="-0.000699172050315 0.00570982817079 -1.59473908718" connected_to="base_link"/>
-<xacro:panda robot_id="1" xyz="0.511233150959 0.157657206059 0.012868642807" rpy="0.00131621839311 -3.37064275204e-05 -1.61483536451" connected_to="base_link"/>
+<xacro:indy7 robot_id="0" xyz="-0.444375276566 0.24876666069 0.0120660662651" rpy="-0.00347209485447 0.0010262729627 -1.58766529131" connected_to="base_link"/>
+<xacro:panda robot_id="1" xyz="0.512558698654 0.165808618069 0.0120181441307" rpy="-0.0016779836511 0.000554054982627 -1.60498128646" connected_to="base_link"/>
 <!-- BODY END -->
 </robot>

File: eTaSL/robots/indy7.xacro (robot description, xacro)
@@ -168,25 +168,25 @@
 		</visual>
 		<collision>
-			<origin xyz="0.005 0.044 0.1" rpy="0 0 0"/>
-			<geometry>
-				<cylinder length="0.08" radius="0.016"/>
-			</geometry>
-		</collision>
-		<collision>
-			<origin xyz="-0.005  0.044  0.1" rpy="0 0 0"/>
-			<geometry>
-				<cylinder length="0.08" radius="0.016"/>
-			</geometry>
-		</collision>
-		<collision>
-			<origin xyz="0.005 -0.044  0.1" rpy="0 0 0"/>
-			<geometry>
-				<cylinder length="0.08" radius="0.016"/>
-			</geometry>
-		</collision>
-		<collision>
-			<origin xyz="-0.005 -0.044  0.1" rpy="0 0 0"/>
-			<geometry>
-				<cylinder length="0.08" radius="0.016"/>
+			<origin xyz="0.006 0.045 0.1" rpy="0 0 0"/>
+			<geometry>
+				<cylinder length="0.083" radius="0.015"/>
+			</geometry>
+		</collision>
+		<collision>
+			<origin xyz="-0.006  0.045  0.1" rpy="0 0 0"/>
+			<geometry>
+				<cylinder length="0.083" radius="0.015"/>
+			</geometry>
+		</collision>
+		<collision>
+			<origin xyz="0.006 -0.045  0.1" rpy="0 0 0"/>
+			<geometry>
+				<cylinder length="0.083" radius="0.015"/>
+			</geometry>
+		</collision>
+		<collision>
+			<origin xyz="-0.006 -0.045  0.1" rpy="0 0 0"/>
+			<geometry>
+				<cylinder length="0.083" radius="0.015"/>
 			</geometry>
 		</collision>

File: eTaSL/robots/panda_arm.xacro (robot description, xacro)
@@ -121,5 +121,11 @@
         <origin xyz="0.      0.0315 -0.115" rpy="2.87423726 -0.          0. "/>
         <geometry>
-          <cylinder length="0.238" radius="0.08"/>
+          <cylinder length="0.20" radius="0.08"/>
+        </geometry>
+      </collision>
+      <collision>
+        <origin xyz="0.      0.0315 0" rpy="0 1.57079633 1.57079633"/>
+        <geometry>
+          <cylinder length="0.12" radius="0.06"/>
         </geometry>
       </collision>
