Commit message: data collecting & training first trial final ver.

File: eTaSL/robots/custom_robots.urdf (robot description, URDF)
Before this commit: robot custom_robots, 21 links, 20 joints
Joints:
- joint indy0_joint_base_link: origin xyz=-0.444375276566 0.24876666069 0.0120660662651 rpy=-0.00347209485447 0.0010262729627 -1.58766529131 -> xyz=1.27387225503 2.19506259557 0.964992293848 rpy=0.0 0.0 4.02263637312
- joint panda1_joint_base_link: origin xyz=0.512558698654 0.165808618069 0.0120181441307 rpy=-0.0016779836511 0.000554054982627 -1.60498128646 -> xyz=1.98939921102 1.46129907119 0.525262459101 rpy=0.0 0.0 1.71500830377

File: eTaSL/robots/custom_robots.urdf.xacro (robot description, xacro)
@@ -6,6 +6,6 @@
 <link name="base_link"/>
 <!-- BODY BEGIN -->
-<xacro:indy7 robot_id="0" xyz="-0.444375276566 0.24876666069 0.0120660662651" rpy="-0.00347209485447 0.0010262729627 -1.58766529131" connected_to="base_link"/>
-<xacro:panda robot_id="1" xyz="0.512558698654 0.165808618069 0.0120181441307" rpy="-0.0016779836511 0.000554054982627 -1.60498128646" connected_to="base_link"/>
+<xacro:indy7 robot_id="0" xyz="1.27387225503 2.19506259557 0.964992293848" rpy="0 0 4.02263637312" connected_to="base_link"/>
+<xacro:panda robot_id="1" xyz="1.98939921102 1.46129907119 0.525262459101" rpy="0 0 1.71500830377" connected_to="base_link"/>
 <!-- BODY END -->
 </robot>

File: eTaSL/robots/custom_robots_indy0_panda1.urdf (robot description, URDF)
Before this commit: robot custom_robots, 22 links, 21 joints
Links:
- link indy0_tcp: geometry collision cylinder length=0.083 radius=0.015; collision cylinder length=0.083 radius=0.015
- link panda1_link5: geometry collision cylinder length=0.12 radius=0.06; collision cylinder length=0.2 radius=0.08
Joints:
- joint indy0_joint0: limit lower=-3.05432619099 upper=3.05432619099 effort=3.14159265359 velocity=1.308996939 -> lower=-3.05432619099 upper=3.05432619099 effort=3.14159265359 velocity=0.654498469498
- joint indy0_joint1: limit lower=-3.05432619099 upper=3.05432619099 effort=3.14159265359 velocity=1.308996939 -> lower=-3.05432619099 upper=3.05432619099 effort=3.14159265359 velocity=0.654498469498
- joint indy0_joint2: limit lower=-3.05432619099 upper=3.05432619099 effort=3.14159265359 velocity=1.308996939 -> lower=-3.05432619099 upper=3.05432619099 effort=3.14159265359 velocity=0.654498469498
- joint indy0_joint3: limit lower=-3.05432619099 upper=3.05432619099 effort=3.14159265359 velocity=1.57079632679 -> lower=-3.05432619099 upper=3.05432619099 effort=3.14159265359 velocity=0.785398163397
- joint indy0_joint4: limit lower=-3.05432619099 upper=3.05432619099 effort=3.14159265359 velocity=1.57079632679 -> lower=-3.05432619099 upper=3.05432619099 effort=3.14159265359 velocity=0.785398163397
- joint indy0_joint5: limit lower=-3.75245789179 upper=3.75245789179 effort=3.14159265359 velocity=1.57079632679 -> lower=-3.75245789179 upper=3.75245789179 effort=3.14159265359 velocity=0.785398163397
- joint panda1_joint1: limit lower=-2.75 upper=2.75 effort=3.14159265359 velocity=1.308996939 -> lower=-2.75 upper=2.75 effort=3.14159265359 velocity=0.654498469498
- joint panda1_joint2: limit lower=-1.7 upper=1.7 effort=3.14159265359 velocity=1.308996939 -> lower=-1.7 upper=1.7 effort=3.14159265359 velocity=0.654498469498
- joint panda1_joint3: limit lower=-2.75 upper=2.75 effort=3.14159265359 velocity=1.308996939 -> lower=-2.75 upper=2.75 effort=3.14159265359 velocity=0.654498469498
- joint panda1_joint4: limit lower=-2.9 upper=-0.1 effort=3.14159265359 velocity=1.308996939 -> lower=-2.9 upper=-0.1 effort=3.14159265359 velocity=0.654498469498
- joint panda1_joint5: limit lower=-2.75 upper=2.75 effort=3.14159265359 velocity=1.57079632679 -> lower=-2.75 upper=2.75 effort=3.14159265359 velocity=0.785398163397
- joint panda1_joint6: limit lower=0.1 upper=3.6 effort=3.14159265359 velocity=1.57079632679 -> lower=0.1 upper=3.6 effort=3.14159265359 velocity=0.785398163397
- joint panda1_joint7: limit lower=-2.75 upper=2.75 effort=3.14159265359 velocity=1.57079632679 -> lower=-2.75 upper=2.75 effort=3.14159265359 velocity=0.785398163397
- joint panda1_joint_base_link: origin xyz=0.87606235504 1.13347322658 0.685762418466 rpy=0.0 0.0 4.50983292483 -> xyz=1.98939921102 1.46129907119 0.525262459101 rpy=0.0 0.0 1.71500830377
- joint stem_joint_base_link: origin xyz=1.09260034561 -2.13035464287 -0.845345258713 rpy=0.0 -0.0 1.66813374687 -> xyz=2.50390291214 0.41415053606 -0.964992284775 rpy=0.0 -0.0 2.26054890098

File: eTaSL/robots/custom_robots_panda1_indy0.urdf (robot description, URDF)
Before this commit: robot custom_robots, 22 links, 21 joints
Links:
- link indy0_tcp: geometry collision cylinder length=0.083 radius=0.015; collision cylinder length=0.083 radius=0.015
- link panda1_link5: geometry collision cylinder length=0.12 radius=0.06; collision cylinder length=0.2 radius=0.08
Joints:
- joint indy0_joint0: limit lower=-3.05432619099 upper=3.05432619099 effort=3.14159265359 velocity=1.308996939 -> lower=-3.05432619099 upper=3.05432619099 effort=3.14159265359 velocity=0.654498469498
- joint indy0_joint1: limit lower=-3.05432619099 upper=3.05432619099 effort=3.14159265359 velocity=1.308996939 -> lower=-3.05432619099 upper=3.05432619099 effort=3.14159265359 velocity=0.654498469498
- joint indy0_joint2: limit lower=-3.05432619099 upper=3.05432619099 effort=3.14159265359 velocity=1.308996939 -> lower=-3.05432619099 upper=3.05432619099 effort=3.14159265359 velocity=0.654498469498
- joint indy0_joint3: limit lower=-3.05432619099 upper=3.05432619099 effort=3.14159265359 velocity=1.57079632679 -> lower=-3.05432619099 upper=3.05432619099 effort=3.14159265359 velocity=0.785398163397
- joint indy0_joint4: limit lower=-3.05432619099 upper=3.05432619099 effort=3.14159265359 velocity=1.57079632679 -> lower=-3.05432619099 upper=3.05432619099 effort=3.14159265359 velocity=0.785398163397
- joint indy0_joint5: limit lower=-3.75245789179 upper=3.75245789179 effort=3.14159265359 velocity=1.57079632679 -> lower=-3.75245789179 upper=3.75245789179 effort=3.14159265359 velocity=0.785398163397
- joint indy0_joint_base_link: origin xyz=2.22645352325 0.880392530093 0.845345268103 rpy=0.0 0.0 4.61505156013 -> xyz=1.27387225503 2.19506259557 0.964992293848 rpy=0.0 0.0 4.02263637312
- joint panda1_joint1: limit lower=-2.75 upper=2.75 effort=3.14159265359 velocity=1.308996939 -> lower=-2.75 upper=2.75 effort=3.14159265359 velocity=0.654498469498
- joint panda1_joint2: limit lower=-1.7 upper=1.7 effort=3.14159265359 velocity=1.308996939 -> lower=-1.7 upper=1.7 effort=3.14159265359 velocity=0.654498469498
- joint panda1_joint3: limit lower=-2.75 upper=2.75 effort=3.14159265359 velocity=1.308996939 -> lower=-2.75 upper=2.75 effort=3.14159265359 velocity=0.654498469498
- joint panda1_joint4: limit lower=0.1 upper=2.9 effort=3.14159265359 velocity=1.308996939 -> lower=0.1 upper=2.9 effort=3.14159265359 velocity=0.654498469498
- joint panda1_joint5: limit lower=-2.75 upper=2.75 effort=3.14159265359 velocity=1.57079632679 -> lower=-2.75 upper=2.75 effort=3.14159265359 velocity=0.785398163397
- joint panda1_joint6: limit lower=-3.6 upper=-0.1 effort=3.14159265359 velocity=1.57079632679 -> lower=-3.6 upper=-0.1 effort=3.14159265359 velocity=0.785398163397
- joint panda1_joint7: limit lower=-2.75 upper=2.75 effort=3.14159265359 velocity=1.57079632679 -> lower=-2.75 upper=2.75 effort=3.14159265359 velocity=0.785398163397
- joint stem_joint_base_link: origin xyz=1.2865408659 -0.630126595497 -0.685762405396 rpy=0.0 -0.0 1.773352385 -> xyz=-1.1602281332 2.17875528336 -0.525262475014 rpy=0.0 -0.0 -1.7150083013

Commit message: each constraint basic operation tested
combined constraint needed

File: eTaSL/robots/custom_robots.urdf (robot description, URDF)
Before this commit: robot custom_robots, 21 links, 20 joints
Joints:
- joint indy0_joint_base_link: origin xyz=1.27387225503 2.19506259557 0.964992293848 rpy=0.0 0.0 4.02263637312 -> xyz=-0.446480512619 0.251528263092 0.00979518890381 rpy=7.72251143907e-05 0.012837732858 -1.58433052921
- joint panda1_joint_base_link: origin xyz=1.98939921102 1.46129907119 0.525262459101 rpy=0.0 0.0 1.71500830377 -> xyz=0.511702060699 0.168303191662 0.014661192894 rpy=0.00371903837049 0.0130669918716 -1.60510658312

File: eTaSL/robots/custom_robots.urdf.xacro (robot description, xacro)
@@ -6,6 +6,6 @@
 <link name="base_link"/>
 <!-- BODY BEGIN -->
-<xacro:indy7 robot_id="0" xyz="1.27387225503 2.19506259557 0.964992293848" rpy="0 0 4.02263637312" connected_to="base_link"/>
-<xacro:panda robot_id="1" xyz="1.98939921102 1.46129907119 0.525262459101" rpy="0 0 1.71500830377" connected_to="base_link"/>
+<xacro:indy7 robot_id="0" xyz="-0.446480512619 0.251528263092 0.00979518890381" rpy="7.72251143907e-05 0.012837732858 -1.58433052921" connected_to="base_link"/>
+<xacro:panda robot_id="1" xyz="0.511702060699 0.168303191662 0.014661192894" rpy="0.00371903837049 0.0130669918716 -1.60510658312" connected_to="base_link"/>
 <!-- BODY END -->
 </robot>

Commit message: wrong robot/world status after second world in data conversion

File: eTaSL/robots/custom_robots.urdf (robot description, URDF)
Before this commit: robot custom_robots, 21 links, 20 joints
Links:
- link indy0_tcp: geometry collision cylinder length=0.08 radius=0.016; collision cylinder length=0.08 radius=0.016
- link panda1_link5: geometry collision cylinder length=0.238 radius=0.08; visual mesh filename=package://franka_description/meshes/visual/link5.dae
Joints:
- joint indy0_joint_base_link: origin xyz=-0.446480512619 0.251528263092 0.00979518890381 rpy=7.72251143907e-05 0.012837732858 -1.58433052921 -> xyz=1.82072648936 1.51551848904 0.873609761456 rpy=0.0 0.0 5.28894471658
- joint panda1_joint_base_link: origin xyz=0.511702060699 0.168303191662 0.014661192894 rpy=0.00371903837049 0.0130669918716 -1.60510658312 -> xyz=1.00627999764 2.09123877292 0.560297783674 rpy=0.0 0.0 4.99165830934

File: eTaSL/robots/custom_robots.urdf.xacro (robot description, xacro)
@@ -6,6 +6,6 @@
 <link name="base_link"/>
 <!-- BODY BEGIN -->
-<xacro:indy7 robot_id="0" xyz="-0.446480512619 0.251528263092 0.00979518890381" rpy="7.72251143907e-05 0.012837732858 -1.58433052921" connected_to="base_link"/>
-<xacro:panda robot_id="1" xyz="0.511702060699 0.168303191662 0.014661192894" rpy="0.00371903837049 0.0130669918716 -1.60510658312" connected_to="base_link"/>
+<xacro:indy7 robot_id="0" xyz="1.27976929132 2.14692452087 0.561689415888" rpy="0 0 3.17708870359" connected_to="base_link"/>
+<xacro:panda robot_id="1" xyz="1.66966774413 1.13748904165 0.670640162967" rpy="0 0 2.9839192782" connected_to="base_link"/>
 <!-- BODY END -->
 </robot>

File: eTaSL/robots/custom_robots_indy0_panda1.urdf (robot description, URDF)
Before this commit: robot custom_robots, 22 links, 21 joints
Joints:
- joint panda1_joint_base_link: origin xyz=1.98939921102 1.46129907119 0.525262459101 rpy=0.0 0.0 1.71500830377 -> xyz=1.28816160756 2.0506651768 0.97209888263 rpy=0.0 0.0 3.1933930461
- joint stem_joint_base_link: origin xyz=2.50390291214 0.41415053606 -0.964992284775 rpy=0.0 -0.0 2.26054890098 -> xyz=-1.4616369009 2.22227668762 -0.789807379246 rpy=0.0 -0.0 -1.58418530859

File: eTaSL/robots/custom_robots_panda1_indy0.urdf (robot description, URDF)
Before this commit: robot custom_robots, 22 links, 21 joints
Joints:
- joint indy0_joint_base_link: origin xyz=1.27387225503 2.19506259557 0.964992293848 rpy=0.0 0.0 4.02263637312 -> xyz=2.2025081522 1.49125902079 0.789807388848 rpy=0.0 0.0 1.58418530838
- joint stem_joint_base_link: origin xyz=-1.1602281332 2.17875528336 -0.525262475014 rpy=0.0 -0.0 -1.7150083013 -> xyz=1.39261162281 1.98121702671 -0.972098886967 rpy=0.0 -0.0 3.08979226202

Commit message: ADD: strict single-thread sampled data checking

File: eTaSL/robots/custom_robots.urdf (robot description, URDF)
Before this commit: robot custom_robots, 21 links, 20 joints
Links:
- link indy0_tcp: geometry collision cylinder length=0.083 radius=0.015; collision cylinder length=0.083 radius=0.015
- link panda1_link5: geometry collision cylinder length=0.12 radius=0.06; collision cylinder length=0.2 radius=0.08
Joints:
- joint indy0_joint_base_link: origin xyz=1.82072648936 1.51551848904 0.873609761456 rpy=0.0 0.0 5.28894471658 -> xyz=2.24761724206 2.0649086405 0.665983084466 rpy=0.0 0.0 2.24402606555
- joint panda1_joint_base_link: origin xyz=1.00627999764 2.09123877292 0.560297783674 rpy=0.0 0.0 4.99165830934 -> xyz=1.13709471236 0.915261168584 0.553192716943 rpy=0.0 0.0 4.61960153851

File: eTaSL/robots/custom_robots.urdf.xacro (robot description, xacro)
@@ -6,6 +6,6 @@
 <link name="base_link"/>
 <!-- BODY BEGIN -->
-<xacro:indy7 robot_id="0" xyz="1.27976929132 2.14692452087 0.561689415888" rpy="0 0 3.17708870359" connected_to="base_link"/>
-<xacro:panda robot_id="1" xyz="1.66966774413 1.13748904165 0.670640162967" rpy="0 0 2.9839192782" connected_to="base_link"/>
+<xacro:indy7 robot_id="0" xyz="2.24761724206 2.0649086405 0.665983084466" rpy="0 0 2.24402606555" connected_to="base_link"/>
+<xacro:panda robot_id="1" xyz="1.13709471236 0.915261168584 0.553192716943" rpy="0 0 4.61960153851" connected_to="base_link"/>
 <!-- BODY END -->
 </robot>

File: eTaSL/robots/custom_robots_indy0_panda1.urdf (robot description, URDF)
Before this commit: robot custom_robots, 22 links, 21 joints
Joints:
- joint panda1_joint_base_link: origin xyz=1.28816160756 2.0506651768 0.97209888263 rpy=0.0 0.0 3.1933930461 -> xyz=1.13709471236 0.915261168584 0.553192716943 rpy=0.0 0.0 4.61960153851
- joint stem_joint_base_link: origin xyz=-1.4616369009 2.22227668762 -0.789807379246 rpy=0.0 -0.0 -1.58418530859 -> xyz=-0.212948918343 3.04471421242 -0.665983080864 rpy=0.0 -0.0 -2.24402607846

File: eTaSL/robots/custom_robots_panda1_indy0.urdf (robot description, URDF)
Before this commit: robot custom_robots, 22 links, 21 joints
Joints:
- joint indy0_joint_base_link: origin xyz=2.2025081522 1.49125902079 0.789807388848 rpy=0.0 0.0 1.58418530838 -> xyz=2.24761724206 2.0649086405 0.665983084466 rpy=0.0 0.0 2.24402606555
- joint stem_joint_base_link: origin xyz=1.39261162281 1.98121702671 -0.972098886967 rpy=0.0 -0.0 3.08979226202 -> xyz=1.01668083668 -1.04740035534 -0.553192734718 rpy=0.0 -0.0 1.66358376677

File: eTaSL/robots/dataset_2012/custom_robots.urdf.xacro (robot description, xacro)
@@ -6,6 +6,6 @@
 <link name="base_link"/>
 <!-- BODY BEGIN -->
-<xacro:indy7 robot_id="0" xyz="1.82072648936 1.51551848904 0.873609761456" rpy="0 0 5.28894471658" connected_to="base_link"/>
-<xacro:panda robot_id="1" xyz="1.00627999764 2.09123877292 0.560297783674" rpy="0 0 4.99165830934" connected_to="base_link"/>
+<xacro:indy7 robot_id="0" xyz="1.47117765439 2.13880621159 0.98596579283" rpy="0 0 6.2121586701" connected_to="base_link"/>
+<xacro:panda robot_id="1" xyz="1.73587238191 0.928318228419 0.841717989793" rpy="0 0 3.4993983017" connected_to="base_link"/>
 <!-- BODY END -->
 </robot>

Commit message: strict data checking debugged

File: eTaSL/robots/custom_robots.urdf (robot description, URDF)
Before this commit: robot custom_robots, 21 links, 20 joints
Joints:
- joint indy0_joint_base_link: origin xyz=2.24761724206 2.0649086405 0.665983084466 rpy=0.0 0.0 2.24402606555 -> xyz=1.80015940705 1.58284533704 0.508719728282 rpy=0.0 0.0 5.042406849
- joint panda1_joint_base_link: origin xyz=1.13709471236 0.915261168584 0.553192716943 rpy=0.0 0.0 4.61960153851 -> xyz=1.11183883425 2.15045839652 0.977799260428 rpy=0.0 0.0 2.21693082774

File: eTaSL/robots/custom_robots.urdf.xacro (robot description, xacro)
@@ -6,6 +6,6 @@
 <link name="base_link"/>
 <!-- BODY BEGIN -->
-<xacro:indy7 robot_id="0" xyz="2.24761724206 2.0649086405 0.665983084466" rpy="0 0 2.24402606555" connected_to="base_link"/>
-<xacro:panda robot_id="1" xyz="1.13709471236 0.915261168584 0.553192716943" rpy="0 0 4.61960153851" connected_to="base_link"/>
+<xacro:indy7 robot_id="0" xyz="1.80015940705 1.58284533704 0.508719728282" rpy="0 0 5.042406849" connected_to="base_link"/>
+<xacro:panda robot_id="1" xyz="1.11183883425 2.15045839652 0.977799260428" rpy="0 0 2.21693082774" connected_to="base_link"/>
 <!-- BODY END -->
 </robot>

File: eTaSL/robots/custom_robots_indy0_panda1.urdf (robot description, URDF)
Before this commit: robot custom_robots, 22 links, 21 joints
Joints:
- joint panda1_joint_base_link: origin xyz=1.13709471236 0.915261168584 0.553192716943 rpy=0.0 0.0 4.61960153851 -> xyz=1.11183883425 2.15045839652 0.977799260428 rpy=0.0 0.0 2.21693082774
- joint stem_joint_base_link: origin xyz=-0.212948918343 3.04471421242 -0.665983080864 rpy=0.0 -0.0 -2.24402607846 -> xyz=0.91407006979 -2.21595335007 -0.508719742298 rpy=0.0 -0.0 1.24077846539

File: eTaSL/robots/custom_robots_panda1_indy0.urdf (robot description, URDF)
Before this commit: robot custom_robots, 22 links, 21 joints
Joints:
- joint indy0_joint_base_link: origin xyz=2.24761724206 2.0649086405 0.665983084466 rpy=0.0 0.0 2.24402606555 -> xyz=1.80015940705 1.58284533704 0.508719728282 rpy=0.0 0.0 5.042406849
- joint stem_joint_base_link: origin xyz=1.01668083668 -1.04740035534 -0.553192734718 rpy=0.0 -0.0 1.66358376677 -> xyz=-1.04751968384 2.18251204491 -0.977799236774 rpy=0.0 -0.0 -2.21693079568

Commit message: new training start

File: eTaSL/robots/custom_robots.urdf (robot description, URDF)
Before this commit: robot custom_robots, 21 links, 20 joints
Links:
- link indy0_tcp: geometry collision cylinder length=0.08 radius=0.016; collision cylinder length=0.08 radius=0.016
- link panda1_link5: geometry collision cylinder length=0.238 radius=0.08; visual mesh filename=package://franka_description/meshes/visual/link5.dae
Joints:
- joint indy0_joint_base_link: origin xyz=1.80015940705 1.58284533704 0.508719728282 rpy=0.0 0.0 5.042406849 -> xyz=0.80598935365 1.47113019577 0.978842064893 rpy=0.0 0.0 5.20390317753
- joint panda1_joint_base_link: origin xyz=1.11183883425 2.15045839652 0.977799260428 rpy=0.0 0.0 2.21693082774 -> xyz=1.98023147441 1.40590763162 0.582734742052 rpy=0.0 0.0 2.67630991295

File: eTaSL/robots/custom_robots.urdf.xacro (robot description, xacro)
@@ -6,6 +6,6 @@
 <link name="base_link"/>
 <!-- BODY BEGIN -->
-<xacro:indy7 robot_id="0" xyz="1.80015940705 1.58284533704 0.508719728282" rpy="0 0 5.042406849" connected_to="base_link"/>
-<xacro:panda robot_id="1" xyz="1.11183883425 2.15045839652 0.977799260428" rpy="0 0 2.21693082774" connected_to="base_link"/>
+<xacro:indy7 robot_id="0" xyz="2.03693081625 1.68234259492 0.579642101225" rpy="0 0 4.35473770107" connected_to="base_link"/>
+<xacro:panda robot_id="1" xyz="1.49639015337 0.85088123284 0.933964702173" rpy="0 0 1.5842200288" connected_to="base_link"/>
 <!-- BODY END -->
 </robot>

File: eTaSL/robots/custom_robots_indy0_panda1.urdf (robot description, URDF)
Before this commit: robot custom_robots, 22 links, 21 joints
Joints:
- joint panda1_joint_base_link: origin xyz=1.11183883425 2.15045839652 0.977799260428 rpy=0.0 0.0 2.21693082774 -> xyz=2.19302557652 1.25793652746 0.611802279564 rpy=0.0 0.0 5.93932705103
- joint stem_joint_base_link: origin xyz=0.91407006979 -2.21595335007 -0.508719742298 rpy=0.0 -0.0 1.24077846539 -> xyz=2.36514997482 0.0308573842049 -0.757959842682 rpy=0.0 -0.0 1.9929919162

File: eTaSL/robots/custom_robots_panda1_indy0.urdf (robot description, URDF)
Before this commit: robot custom_robots, 22 links, 21 joints
Joints:
- joint indy0_joint_base_link: origin xyz=1.80015940705 1.58284533704 0.508719728282 rpy=0.0 0.0 5.042406849 -> xyz=0.941006019462 2.17011383128 0.757959850252 rpy=0.0 0.0 4.29019341093
- joint stem_joint_base_link: origin xyz=-1.04751968384 2.18251204491 -0.977799236774 rpy=0.0 -0.0 -2.21693079568 -> xyz=-1.64056992531 -1.92361521721 -0.611802279949 rpy=0.0 -0.0 0.343858261359

File: eTaSL/robots/dataset_2012/custom_robots.urdf.xacro (robot description, xacro)
@@ -6,6 +6,6 @@
 <link name="base_link"/>
 <!-- BODY BEGIN -->
-<xacro:indy7 robot_id="0" xyz="1.47117765439 2.13880621159 0.98596579283" rpy="0 0 6.2121586701" connected_to="base_link"/>
-<xacro:panda robot_id="1" xyz="1.73587238191 0.928318228419 0.841717989793" rpy="0 0 3.4993983017" connected_to="base_link"/>
+<xacro:indy7 robot_id="0" xyz="0.80598935365 1.47113019577 0.978842064893" rpy="0 0 5.20390317753" connected_to="base_link"/>
+<xacro:panda robot_id="1" xyz="1.98023147441 1.40590763162 0.582734742052" rpy="0 0 2.67630991295" connected_to="base_link"/>
 <!-- BODY END -->
 </robot>

Commit message: converting scene done

File: eTaSL/robots/custom_robots.urdf (robot description, URDF)
Before this commit: robot custom_robots, 21 links, 20 joints
Links:
- link indy0_tcp: geometry collision cylinder length=0.083 radius=0.015; collision cylinder length=0.083 radius=0.015
- link panda1_link5: geometry collision cylinder length=0.12 radius=0.06; collision cylinder length=0.2 radius=0.08
Joints:
- joint indy0_joint_base_link: origin xyz=0.80598935365 1.47113019577 0.978842064893 rpy=0.0 0.0 5.20390317753 -> xyz=-0.446480512619 0.251528263092 0.00979518890381 rpy=7.72251143907e-05 0.012837732858 -1.58433052921
- joint panda1_joint_base_link: origin xyz=1.98023147441 1.40590763162 0.582734742052 rpy=0.0 0.0 2.67630991295 -> xyz=0.511702060699 0.168303191662 0.014661192894 rpy=0.00371903837049 0.0130669918716 -1.60510658312

File: eTaSL/robots/custom_robots.urdf.xacro (robot description, xacro)
@@ -6,6 +6,6 @@
 <link name="base_link"/>
 <!-- BODY BEGIN -->
-<xacro:indy7 robot_id="0" xyz="2.03693081625 1.68234259492 0.579642101225" rpy="0 0 4.35473770107" connected_to="base_link"/>
-<xacro:panda robot_id="1" xyz="1.49639015337 0.85088123284 0.933964702173" rpy="0 0 1.5842200288" connected_to="base_link"/>
+<xacro:indy7 robot_id="0" xyz="-0.446480512619 0.251528263092 0.00979518890381" rpy="7.72251143907e-05 0.012837732858 -1.58433052921" connected_to="base_link"/>
+<xacro:panda robot_id="1" xyz="0.511702060699 0.168303191662 0.014661192894" rpy="0.00371903837049 0.0130669918716 -1.60510658312" connected_to="base_link"/>
 <!-- BODY END -->
 </robot>
