Commit message: generalized training failure final ver.

File: eTaSL/robots/custom_robots.urdf (robot description, URDF)
Before this commit: robot custom_robots, 21 links, 20 joints
Joints:
- joint indy0_joint_base_link: origin xyz=-0.446480512619 0.251528263092 0.00979518890381 rpy=7.72251143907e-05 0.012837732858 -1.58433052921 -> xyz=0.343297365217 0.23133351223 -0.0517830795546 rpy=0.0 0.0 0.945738522619
- joint panda1_joint_base_link: origin xyz=0.511702060699 0.168303191662 0.014661192894 rpy=0.00371903837049 0.0130669918716 -1.60510658312 -> xyz=-0.706039166437 0.203311060274 0.0903344474137 rpy=0.0 0.0 3.88253014034

File: eTaSL/robots/custom_robots.urdf.xacro (robot description, xacro)
@@ -6,6 +6,6 @@
 <link name="base_link"/>
 <!-- BODY BEGIN -->
-<xacro:indy7 robot_id="0" xyz="-0.446480512619 0.251528263092 0.00979518890381" rpy="7.72251143907e-05 0.012837732858 -1.58433052921" connected_to="base_link"/>
-<xacro:panda robot_id="1" xyz="0.511702060699 0.168303191662 0.014661192894" rpy="0.00371903837049 0.0130669918716 -1.60510658312" connected_to="base_link"/>
+<xacro:indy7 robot_id="0" xyz="0.343297365217 0.23133351223 -0.0517830795546" rpy="0 0 0.945738522619" connected_to="base_link"/>
+<xacro:panda robot_id="1" xyz="-0.706039166437 0.203311060274 0.0903344474137" rpy="0 0 3.88253014034" connected_to="base_link"/>
 <!-- BODY END -->
 </robot>

Commit message: constrained motion testing done

File: eTaSL/robots/custom_robots.urdf (robot description, URDF)
Before this commit: robot custom_robots, 21 links, 20 joints
Joints:
- joint indy0_joint_base_link: origin xyz=0.343297365217 0.23133351223 -0.0517830795546 rpy=0.0 0.0 0.945738522619 -> xyz=-0.446480512619 0.251528263092 0.00979518890381 rpy=7.72251143907e-05 0.012837732858 -1.58433052921
- joint panda1_joint_base_link: origin xyz=-0.706039166437 0.203311060274 0.0903344474137 rpy=0.0 0.0 3.88253014034 -> xyz=0.511702060699 0.168303191662 0.014661192894 rpy=0.00371903837049 0.0130669918716 -1.60510658312

File: eTaSL/robots/custom_robots.urdf.xacro (robot description, xacro)
@@ -6,6 +6,6 @@
 <link name="base_link"/>
 <!-- BODY BEGIN -->
-<xacro:indy7 robot_id="0" xyz="0.343297365217 0.23133351223 -0.0517830795546" rpy="0 0 0.945738522619" connected_to="base_link"/>
-<xacro:panda robot_id="1" xyz="-0.706039166437 0.203311060274 0.0903344474137" rpy="0 0 3.88253014034" connected_to="base_link"/>
+<xacro:indy7 robot_id="0" xyz="-0.446480512619 0.251528263092 0.00979518890381" rpy="7.72251143907e-05 0.012837732858 -1.58433052921" connected_to="base_link"/>
+<xacro:panda robot_id="1" xyz="0.511702060699 0.168303191662 0.014661192894" rpy="0.00371903837049 0.0130669918716 -1.60510658312" connected_to="base_link"/>
 <!-- BODY END -->
 </robot>
