Commit message: rviz tested

File: src/robots/custom_robots.urdf (robot description, URDF)
Before this commit: robot custom_robots, 21 links, 20 joints
Joints:
- joint indy0_joint_base_link: origin xyz=-0.446480512619 0.251528263092 0.00979518890381 rpy=7.72251143907e-05 0.012837732858 -1.58433052921 -> xyz=-0.487274616957 0.264187186956 0.0159955620766 rpy=-0.0026469464508 0.00914991724636 -1.57092377058
- joint panda1_joint_base_link: origin xyz=0.511702060699 0.168303191662 0.014661192894 rpy=0.00371903837049 0.0130669918716 -1.60510658312 -> xyz=0.473329782486 0.19310387969 0.0185957551003 rpy=0.000191128456776 0.00652094311388 -1.59126089616

File: src/robots/custom_robots.urdf.xacro (robot description, xacro)
@@ -6,6 +6,6 @@
 <link name="base_link"/>
 <!-- BODY BEGIN -->
-<xacro:indy7 robot_id="0" xyz="-0.446480512619 0.251528263092 0.00979518890381" rpy="7.72251143907e-05 0.012837732858 -1.58433052921" connected_to="base_link"/>
-<xacro:panda robot_id="1" xyz="0.511702060699 0.168303191662 0.014661192894" rpy="0.00371903837049 0.0130669918716 -1.60510658312" connected_to="base_link"/>
+<xacro:indy7 robot_id="0" xyz="-0.487274616957 0.264187186956 0.0159955620766" rpy="-0.0026469464508 0.00914991724636 -1.57092377058" connected_to="base_link"/>
+<xacro:panda robot_id="1" xyz="0.473329782486 0.19310387969 0.0185957551003" rpy="0.000191128456776 0.00652094311388 -1.59126089616" connected_to="base_link"/>
 <!-- BODY END -->
 </robot>

Commit message: xacro_customizer tested

File: src/robots/custom_robots.urdf (robot description, URDF)
Before this commit: robot custom_robots, 21 links, 20 joints
Joints:
- joint indy0_joint_base_link: origin xyz=-0.487274616957 0.264187186956 0.0159955620766 rpy=-0.0026469464508 0.00914991724636 -1.57092377058 -> xyz=-0.486727714539 0.263820081949 0.0160670280457 rpy=-0.00308669584165 0.00781093992537 -1.57082280324
- joint panda1_joint_base_link: origin xyz=0.473329782486 0.19310387969 0.0185957551003 rpy=0.000191128456776 0.00652094311388 -1.59126089616 -> xyz=0.473153322935 0.193206578493 0.0185115933418 rpy=8.92397463516e-05 0.00680347551784 -1.59112972609

File: src/robots/custom_robots.urdf.xacro (robot description, xacro)
@@ -6,6 +6,6 @@
 <link name="base_link"/>
 <!-- BODY BEGIN -->
-<xacro:indy7 robot_id="0" xyz="-0.487274616957 0.264187186956 0.0159955620766" rpy="-0.0026469464508 0.00914991724636 -1.57092377058" connected_to="base_link"/>
-<xacro:panda robot_id="1" xyz="0.473329782486 0.19310387969 0.0185957551003" rpy="0.000191128456776 0.00652094311388 -1.59126089616" connected_to="base_link"/>
+<xacro:indy7 robot_id="0" xyz="-0.486727714539 0.263820081949 0.0160670280457" rpy="-0.00308669584165 0.00781093992537 -1.57082280324" connected_to="base_link"/>
+<xacro:panda robot_id="1" xyz="0.473153322935 0.193206578493 0.0185115933418" rpy="8.92397463516e-05 0.00680347551784 -1.59112972609" connected_to="base_link"/>
 <!-- BODY END -->
 </robot>

Commit message: geometry.builder tested

File: src/robots/custom_robots.urdf (robot description, URDF)
Before this commit: robot custom_robots, 21 links, 20 joints
Joints:
- joint indy0_joint_base_link: origin xyz=-0.486727714539 0.263820081949 0.0160670280457 rpy=-0.00308669584165 0.00781093992537 -1.57082280324 -> xyz=-0.487554013729 0.264571011066 0.0158407092094 rpy=-0.00288702970446 0.00926925062681 -1.57075154968
- joint panda1_joint_base_link: origin xyz=0.473153322935 0.193206578493 0.0185115933418 rpy=8.92397463516e-05 0.00680347551784 -1.59112972609 -> xyz=0.473406910896 0.193002581596 0.0188117027283 rpy=6.62986996645e-05 0.00712266650345 -1.59124614593

File: src/robots/custom_robots.urdf.xacro (robot description, xacro)
@@ -6,6 +6,6 @@
 <link name="base_link"/>
 <!-- BODY BEGIN -->
-<xacro:indy7 robot_id="0" xyz="-0.486727714539 0.263820081949 0.0160670280457" rpy="-0.00308669584165 0.00781093992537 -1.57082280324" connected_to="base_link"/>
-<xacro:panda robot_id="1" xyz="0.473153322935 0.193206578493 0.0185115933418" rpy="8.92397463516e-05 0.00680347551784 -1.59112972609" connected_to="base_link"/>
+<xacro:indy7 robot_id="0" xyz="-0.487554013729 0.264571011066 0.0158407092094" rpy="-0.00288702970446 0.00926925062681 -1.57075154968" connected_to="base_link"/>
+<xacro:panda robot_id="1" xyz="0.473406910896 0.193002581596 0.0188117027283" rpy="6.62986996645e-05 0.00712266650345 -1.59124614593" connected_to="base_link"/>
 <!-- BODY END -->
 </robot>

Commit message: planning scene all tested

File: src/robots/custom_robots.urdf (robot description, URDF)
Before this commit: robot custom_robots, 21 links, 20 joints
Joints:
- joint indy0_joint_base_link: origin xyz=-0.487554013729 0.264571011066 0.0158407092094 rpy=-0.00288702970446 0.00926925062681 -1.57075154968 -> xyz=-0.487381994724 0.264186501503 0.0159141421318 rpy=-0.00264487634469 0.00953402629287 -1.57078364719
- joint panda1_joint_base_link: origin xyz=0.473406910896 0.193002581596 0.0188117027283 rpy=6.62986996645e-05 0.00712266650345 -1.59124614593 -> xyz=0.473399341106 0.192869663239 0.018578350544 rpy=-0.000374430259411 0.00358412421389 -1.59089641456

File: src/robots/custom_robots.urdf.xacro (robot description, xacro)
@@ -6,6 +6,6 @@
 <link name="base_link"/>
 <!-- BODY BEGIN -->
-<xacro:indy7 robot_id="0" xyz="-0.487554013729 0.264571011066 0.0158407092094" rpy="-0.00288702970446 0.00926925062681 -1.57075154968" connected_to="base_link"/>
-<xacro:panda robot_id="1" xyz="0.473406910896 0.193002581596 0.0188117027283" rpy="6.62986996645e-05 0.00712266650345 -1.59124614593" connected_to="base_link"/>
+<xacro:indy7 robot_id="0" xyz="-0.487381994724 0.264186501503 0.0159141421318" rpy="-0.00264487634469 0.00953402629287 -1.57078364719" connected_to="base_link"/>
+<xacro:panda robot_id="1" xyz="0.473399341106 0.192869663239 0.018578350544" rpy="-0.000374430259411 0.00358412421389 -1.59089641456" connected_to="base_link"/>
 <!-- BODY END -->
 </robot>

Commit message: planning scene updated with handle-releated functions

File: src/robots/custom_robots.urdf (robot description, URDF)
Before this commit: robot custom_robots, 21 links, 20 joints
Joints:
- joint indy0_joint_base_link: origin xyz=-0.487381994724 0.264186501503 0.0159141421318 rpy=-0.00264487634469 0.00953402629287 -1.57078364719 -> xyz=-0.487072825432 0.26375412941 0.016174197197 rpy=-0.00279357536993 0.00890654193816 -1.57098664825
- joint panda1_joint_base_link: origin xyz=0.473399341106 0.192869663239 0.018578350544 rpy=-0.000374430259411 0.00358412421389 -1.59089641456 -> xyz=0.473319411278 0.193055033684 0.0183472633362 rpy=-0.000866180148766 0.00422341913319 -1.59064682222

File: src/robots/custom_robots.urdf.xacro (robot description, xacro)
@@ -6,6 +6,6 @@
 <link name="base_link"/>
 <!-- BODY BEGIN -->
-<xacro:indy7 robot_id="0" xyz="-0.487381994724 0.264186501503 0.0159141421318" rpy="-0.00264487634469 0.00953402629287 -1.57078364719" connected_to="base_link"/>
-<xacro:panda robot_id="1" xyz="0.473399341106 0.192869663239 0.018578350544" rpy="-0.000374430259411 0.00358412421389 -1.59089641456" connected_to="base_link"/>
+<xacro:indy7 robot_id="0" xyz="-0.487072825432 0.26375412941 0.016174197197" rpy="-0.00279357536993 0.00890654193816 -1.57098664825" connected_to="base_link"/>
+<xacro:panda robot_id="1" xyz="0.473319411278 0.193055033684 0.0183472633362" rpy="-0.000866180148766 0.00422341913319 -1.59064682222" connected_to="base_link"/>
 <!-- BODY END -->
 </robot>

Commit message: moveit planning run-tested

File: src/robots/custom_robots.urdf (robot description, URDF)
Before this commit: robot custom_robots, 21 links, 20 joints
Joints:
- joint indy0_joint_base_link: origin xyz=-0.487072825432 0.26375412941 0.016174197197 rpy=-0.00279357536993 0.00890654193816 -1.57098664825 -> xyz=-0.487790256739 0.265209257603 0.0148949027061 rpy=-0.0031989610126 0.00663049911201 -1.57043366273
- joint panda1_joint_base_link: origin xyz=0.473319411278 0.193055033684 0.0183472633362 rpy=-0.000866180148766 0.00422341913319 -1.59064682222 -> xyz=0.473460495472 0.192622900009 0.0184848308563 rpy=-0.000500397768373 0.00289756451477 -1.59143596187

File: src/robots/custom_robots.urdf.xacro (robot description, xacro)
@@ -6,6 +6,6 @@
 <link name="base_link"/>
 <!-- BODY BEGIN -->
-<xacro:indy7 robot_id="0" xyz="-0.487072825432 0.26375412941 0.016174197197" rpy="-0.00279357536993 0.00890654193816 -1.57098664825" connected_to="base_link"/>
-<xacro:panda robot_id="1" xyz="0.473319411278 0.193055033684 0.0183472633362" rpy="-0.000866180148766 0.00422341913319 -1.59064682222" connected_to="base_link"/>
+<xacro:indy7 robot_id="0" xyz="-0.487790256739 0.265209257603 0.0148949027061" rpy="-0.0031989610126 0.00663049911201 -1.57043366273" connected_to="base_link"/>
+<xacro:panda robot_id="1" xyz="0.473460495472 0.192622900009 0.0184848308563" rpy="-0.000500397768373 0.00289756451477 -1.59143596187" connected_to="base_link"/>
 <!-- BODY END -->
 </robot>

Commit message: moveit planning test done

File: src/robots/custom_robots.urdf (robot description, URDF)
Before this commit: robot custom_robots, 21 links, 20 joints
Joints:
- joint indy0_joint_base_link: origin xyz=-0.487790256739 0.265209257603 0.0148949027061 rpy=-0.0031989610126 0.00663049911201 -1.57043366273 -> xyz=-0.487524271011 0.264843404293 0.0154437422752 rpy=-0.00314533691826 0.00758479375283 -1.57074989065
- joint panda1_joint_base_link: origin xyz=0.473460495472 0.192622900009 0.0184848308563 rpy=-0.000500397768373 0.00289756451477 -1.59143596187 -> xyz=0.473399251699 0.192876219749 0.0178402662277 rpy=-0.00125492709797 0.00126576460748 -1.5910533579

File: src/robots/custom_robots.urdf.xacro (robot description, xacro)
@@ -6,6 +6,6 @@
 <link name="base_link"/>
 <!-- BODY BEGIN -->
-<xacro:indy7 robot_id="0" xyz="-0.487790256739 0.265209257603 0.0148949027061" rpy="-0.0031989610126 0.00663049911201 -1.57043366273" connected_to="base_link"/>
-<xacro:panda robot_id="1" xyz="0.473460495472 0.192622900009 0.0184848308563" rpy="-0.000500397768373 0.00289756451477 -1.59143596187" connected_to="base_link"/>
+<xacro:indy7 robot_id="0" xyz="-0.487524271011 0.264843404293 0.0154437422752" rpy="-0.00314533691826 0.00758479375283 -1.57074989065" connected_to="base_link"/>
+<xacro:panda robot_id="1" xyz="0.473399251699 0.192876219749 0.0178402662277" rpy="-0.00125492709797 0.00126576460748 -1.5910533579" connected_to="base_link"/>
 <!-- BODY END -->
 </robot>

Commit message: etasl planning test done

File: src/robots/custom_robots.urdf (robot description, URDF)
Before this commit: robot custom_robots, 21 links, 20 joints
Joints:
- joint indy0_joint_base_link: origin xyz=-0.487524271011 0.264843404293 0.0154437422752 rpy=-0.00314533691826 0.00758479375283 -1.57074989065 -> xyz=-0.487214565277 0.264153718948 0.0159312486649 rpy=-0.00326889998706 0.0073027963031 -1.57100398561
- joint panda1_joint_base_link: origin xyz=0.473399251699 0.192876219749 0.0178402662277 rpy=-0.00125492709797 0.00126576460748 -1.5910533579 -> xyz=0.473313033581 0.192986249924 0.0180513858795 rpy=-0.000651149065145 0.00248345970283 -1.59097476361

File: src/robots/custom_robots.urdf.xacro (robot description, xacro)
@@ -6,6 +6,6 @@
 <link name="base_link"/>
 <!-- BODY BEGIN -->
-<xacro:indy7 robot_id="0" xyz="-0.487524271011 0.264843404293 0.0154437422752" rpy="-0.00314533691826 0.00758479375283 -1.57074989065" connected_to="base_link"/>
-<xacro:panda robot_id="1" xyz="0.473399251699 0.192876219749 0.0178402662277" rpy="-0.00125492709797 0.00126576460748 -1.5910533579" connected_to="base_link"/>
+<xacro:indy7 robot_id="0" xyz="-0.487214565277 0.264153718948 0.0159312486649" rpy="-0.00326889998706 0.0073027963031 -1.57100398561" connected_to="base_link"/>
+<xacro:panda robot_id="1" xyz="0.473313033581 0.192986249924 0.0180513858795" rpy="-0.000651149065145 0.00248345970283 -1.59097476361" connected_to="base_link"/>
 <!-- BODY END -->
 </robot>

Commit message: TMP pipeline - ObjectAstar tested

File: src/robots/custom_robots.urdf (robot description, URDF)
Before this commit: robot custom_robots, 21 links, 20 joints
Joints:
- joint indy0_joint_base_link: origin xyz=-0.487214565277 0.264153718948 0.0159312486649 rpy=-0.00326889998706 0.0073027963031 -1.57100398561 -> xyz=-0.486579537392 0.263651669025 0.0163976550102 rpy=-0.00320856492163 0.00748790328272 -1.57129538441
- joint panda1_joint_base_link: origin xyz=0.473313033581 0.192986249924 0.0180513858795 rpy=-0.000651149065145 0.00248345970283 -1.59097476361 -> xyz=0.473220765591 0.192988872528 0.0179921388626 rpy=-0.000648226279876 0.00175002294357 -1.59079679863

File: src/robots/custom_robots.urdf.xacro (robot description, xacro)
@@ -6,6 +6,6 @@
 <link name="base_link"/>
 <!-- BODY BEGIN -->
-<xacro:indy7 robot_id="0" xyz="-0.487214565277 0.264153718948 0.0159312486649" rpy="-0.00326889998706 0.0073027963031 -1.57100398561" connected_to="base_link"/>
-<xacro:panda robot_id="1" xyz="0.473313033581 0.192986249924 0.0180513858795" rpy="-0.000651149065145 0.00248345970283 -1.59097476361" connected_to="base_link"/>
+<xacro:indy7 robot_id="0" xyz="-0.486579537392 0.263651669025 0.0163976550102" rpy="-0.00320856492163 0.00748790328272 -1.57129538441" connected_to="base_link"/>
+<xacro:panda robot_id="1" xyz="0.473220765591 0.192988872528 0.0179921388626" rpy="-0.000648226279876 0.00175002294357 -1.59079679863" connected_to="base_link"/>
 <!-- BODY END -->
 </robot>

Commit message: TMP multiprocess tested

File: src/robots/custom_robots.urdf (robot description, URDF)
Before this commit: robot custom_robots, 21 links, 20 joints
Joints:
- joint indy0_joint_base_link: origin xyz=-0.486579537392 0.263651669025 0.0163976550102 rpy=-0.00320856492163 0.00748790328272 -1.57129538441 -> xyz=-0.486864924431 0.263942539692 0.0160436630249 rpy=-0.00305673280132 0.00735572670333 -1.57125071836
- joint panda1_joint_base_link: origin xyz=0.473220765591 0.192988872528 0.0179921388626 rpy=-0.000648226279876 0.00175002294357 -1.59079679863 -> xyz=0.473213374615 0.192947745323 0.0181459188461 rpy=-0.000542537016707 0.0024738931964 -1.59092726017

File: src/robots/custom_robots.urdf.xacro (robot description, xacro)
@@ -6,6 +6,6 @@
 <link name="base_link"/>
 <!-- BODY BEGIN -->
-<xacro:indy7 robot_id="0" xyz="-0.486579537392 0.263651669025 0.0163976550102" rpy="-0.00320856492163 0.00748790328272 -1.57129538441" connected_to="base_link"/>
-<xacro:panda robot_id="1" xyz="0.473220765591 0.192988872528 0.0179921388626" rpy="-0.000648226279876 0.00175002294357 -1.59079679863" connected_to="base_link"/>
+<xacro:indy7 robot_id="0" xyz="-0.486864924431 0.263942539692 0.0160436630249" rpy="-0.00305673280132 0.00735572670333 -1.57125071836" connected_to="base_link"/>
+<xacro:panda robot_id="1" xyz="0.473213374615 0.192947745323 0.0181459188461" rpy="-0.000542537016707 0.0024738931964 -1.59092726017" connected_to="base_link"/>
 <!-- BODY END -->
 </robot>

Commit message: implemented moveit dual arm

File: src/robots/custom_robots.urdf (robot description, URDF)
Before this commit: robot custom_robots, 21 links, 20 joints
Joints:
- joint indy0_joint_base_link: origin xyz=-0.486864924431 0.263942539692 0.0160436630249 rpy=-0.00305673280132 0.00735572670333 -1.57125071836 -> xyz=-0.486797600985 0.26384139061 0.0161607861519 rpy=-0.00325296848485 0.00713929622346 -1.57110748028
- joint panda1_joint_base_link: origin xyz=0.473213374615 0.192947745323 0.0181459188461 rpy=-0.000542537016707 0.0024738931964 -1.59092726017 -> xyz=0.473222404718 0.193011403084 0.0180019140244 rpy=-0.000844875227355 0.00209182646282 -1.5907203001

File: src/robots/custom_robots.urdf.xacro (robot description, xacro)
@@ -6,6 +6,6 @@
 <link name="base_link"/>
 <!-- BODY BEGIN -->
-<xacro:indy7 robot_id="0" xyz="-0.486864924431 0.263942539692 0.0160436630249" rpy="-0.00305673280132 0.00735572670333 -1.57125071836" connected_to="base_link"/>
-<xacro:panda robot_id="1" xyz="0.473213374615 0.192947745323 0.0181459188461" rpy="-0.000542537016707 0.0024738931964 -1.59092726017" connected_to="base_link"/>
+<xacro:indy7 robot_id="0" xyz="-0.486797600985 0.26384139061 0.0161607861519" rpy="-0.00325296848485 0.00713929622346 -1.57110748028" connected_to="base_link"/>
+<xacro:panda robot_id="1" xyz="0.473222404718 0.193011403084 0.0180019140244" rpy="-0.000844875227355 0.00209182646282 -1.5907203001" connected_to="base_link"/>
 <!-- BODY END -->
 </robot>

File: src/robots/custom_robots_indy0_panda1.urdf (robot description, URDF)
Before this commit: robot custom_robots, 22 links, 21 joints
Joints:
- joint panda1_joint_base_link: origin xyz=2.19302557652 1.25793652746 0.611802279564 rpy=0.0 0.0 5.93932705103 -> xyz=0.473222404718 0.193011403084 0.0180019140244 rpy=-0.000844875227355 0.00209182646282 -1.5907203001
- joint stem_joint_base_link: origin xyz=2.36514997482 0.0308573842049 -0.757959842682 rpy=0.0 -0.0 1.9929919162 -> xyz=0.263798564672 0.486923545599 -0.012693952769 rpy=-0.00714030769409 -0.00325074680366 1.57110747399

File: src/robots/custom_robots_panda1_indy0.urdf (robot description, URDF)
Before this commit: robot custom_robots, 22 links, 21 joints
Joints:
- joint indy0_joint_base_link: origin xyz=0.941006019462 2.17011383128 0.757959850252 rpy=0.0 0.0 4.29019341093 -> xyz=-0.486797600985 0.26384139061 0.0161607861519 rpy=-0.00325296848485 0.00713929622346 -1.57110748028
- joint stem_joint_base_link: origin xyz=-1.64056992531 -1.92361521721 -0.611802279949 rpy=0.0 -0.0 0.343858261359 -> xyz=0.202438160777 -0.469268202782 -0.0179749652743 rpy=-0.00210824347852 -0.000803032847057 1.59072026329

Commit message: initial ui fix

File: src/robots/custom_robots.urdf (robot description, URDF)
Before this commit: robot custom_robots, 21 links, 20 joints
Joints:
- joint indy0_joint_base_link: origin xyz=-0.486797600985 0.26384139061 0.0161607861519 rpy=-0.00325296848485 0.00713929622346 -1.57110748028 -> xyz=-0.487280011177 0.264443635941 0.0157945752144 rpy=-0.00313377464597 0.00761310704768 -1.57110754938
- joint panda1_joint_base_link: origin xyz=0.473222404718 0.193011403084 0.0180019140244 rpy=-0.000844875227355 0.00209182646282 -1.5907203001 -> xyz=0.47326874733 0.192965149879 0.0181476473808 rpy=-0.00103220634817 0.0028170982324 -1.59090047908

File: src/robots/custom_robots.urdf.xacro (robot description, xacro)
@@ -6,6 +6,6 @@
 <link name="base_link"/>
 <!-- BODY BEGIN -->
-<xacro:indy7 robot_id="0" xyz="-0.486797600985 0.26384139061 0.0161607861519" rpy="-0.00325296848485 0.00713929622346 -1.57110748028" connected_to="base_link"/>
-<xacro:panda robot_id="1" xyz="0.473222404718 0.193011403084 0.0180019140244" rpy="-0.000844875227355 0.00209182646282 -1.5907203001" connected_to="base_link"/>
+<xacro:indy7 robot_id="0" xyz="-0.487280011177 0.264443635941 0.0157945752144" rpy="-0.00313377464597 0.00761310704768 -1.57110754938" connected_to="base_link"/>
+<xacro:panda robot_id="1" xyz="0.47326874733 0.192965149879 0.0181476473808" rpy="-0.00103220634817 0.0028170982324 -1.59090047908" connected_to="base_link"/>
 <!-- BODY END -->
 </robot>

File: src/robots/custom_robots_indy0_panda1.urdf (robot description, URDF)
Before this commit: robot custom_robots, 22 links, 21 joints
Joints:
- joint panda1_joint_base_link: origin xyz=0.473222404718 0.193011403084 0.0180019140244 rpy=-0.000844875227355 0.00209182646282 -1.5907203001 -> xyz=0.47326874733 0.192965149879 0.0181476473808 rpy=-0.00103220634817 0.0028170982324 -1.59090047908
- joint stem_joint_base_link: origin xyz=0.263798564672 0.486923545599 -0.012693952769 rpy=-0.00714030769409 -0.00325074680366 1.57110747399 -> xyz=0.264404565096 0.487403094769 -0.0122547037899 rpy=-0.00761408199137 -0.0031314052001 1.5711075419

File: src/robots/custom_robots_panda1_indy0.urdf (robot description, URDF)
Before this commit: robot custom_robots, 22 links, 21 joints
Joints:
- joint indy0_joint_base_link: origin xyz=-0.486797600985 0.26384139061 0.0161607861519 rpy=-0.00325296848485 0.00713929622346 -1.57110748028 -> xyz=-0.487280011177 0.264443635941 0.0157945752144 rpy=-0.00313377464597 0.00761310704768 -1.57110754938
- joint stem_joint_base_link: origin xyz=0.202438160777 -0.469268202782 -0.0179749652743 rpy=-0.00210824347852 -0.000803032847057 1.59072026329 -> xyz=0.202490508556 -0.469275593758 -0.0180616807193 rpy=-0.00283727922998 -0.000975366235613 1.59090040905

Commit message: basic ui functions checked

File: src/robots/custom_robots.urdf (robot description, URDF)
Before this commit: robot custom_robots, 21 links, 20 joints
Joints:
- joint indy0_joint_base_link: origin xyz=-0.487280011177 0.264443635941 0.0157945752144 rpy=-0.00313377464597 0.00761310704768 -1.57110754938 -> xyz=-0.487239867449 0.264511883259 0.0157464146614 rpy=-0.0032244007077 0.00715094916312 -1.57122883195
- joint panda1_joint_base_link: origin xyz=0.47326874733 0.192965149879 0.0181476473808 rpy=-0.00103220634817 0.0028170982324 -1.59090047908 -> xyz=0.473158180714 0.192921757698 0.0181045532227 rpy=-0.000695425424269 0.00240603340554 -1.59131646607

File: src/robots/custom_robots.urdf.xacro (robot description, xacro)
@@ -6,6 +6,6 @@
 <link name="base_link"/>
 <!-- BODY BEGIN -->
-<xacro:indy7 robot_id="0" xyz="-0.487280011177 0.264443635941 0.0157945752144" rpy="-0.00313377464597 0.00761310704768 -1.57110754938" connected_to="base_link"/>
-<xacro:panda robot_id="1" xyz="0.47326874733 0.192965149879 0.0181476473808" rpy="-0.00103220634817 0.0028170982324 -1.59090047908" connected_to="base_link"/>
+<xacro:indy7 robot_id="0" xyz="-0.487239867449 0.264511883259 0.0157464146614" rpy="-0.0032244007077 0.00715094916312 -1.57122883195" connected_to="base_link"/>
+<xacro:panda robot_id="1" xyz="0.473158180714 0.192921757698 0.0181045532227" rpy="-0.000695425424269 0.00240603340554 -1.59131646607" connected_to="base_link"/>
 <!-- BODY END -->
 </robot>

File: src/robots/custom_robots_indy0_panda1.urdf (robot description, URDF)
Before this commit: robot custom_robots, 22 links, 21 joints
Joints:
- joint panda1_joint_base_link: origin xyz=0.47326874733 0.192965149879 0.0181476473808 rpy=-0.00103220634817 0.0028170982324 -1.59090047908 -> xyz=0.473158180714 0.192921757698 0.0181045532227 rpy=-0.000695425424269 0.00240603340554 -1.59131646607
- joint stem_joint_base_link: origin xyz=0.264404565096 0.487403094769 -0.0122547037899 rpy=-0.00761408199137 -0.0031314052001 1.5711075419 -> xyz=0.264406949282 0.487396359444 -0.0122845303267 rpy=-0.00715234293124 -0.00322130770527 1.57122882316

File: src/robots/custom_robots_panda1_indy0.urdf (robot description, URDF)
Before this commit: robot custom_robots, 22 links, 21 joints
Joints:
- joint indy0_joint_base_link: origin xyz=-0.487280011177 0.264443635941 0.0157945752144 rpy=-0.00313377464597 0.00761310704768 -1.57110754938 -> xyz=-0.487239867449 0.264511883259 0.0157464146614 rpy=-0.0032244007077 0.00715094916312 -1.57122883195
- joint stem_joint_base_link: origin xyz=0.202490508556 -0.469275593758 -0.0180616807193 rpy=-0.00283727922998 -0.000975366235613 1.59090040905 -> xyz=0.202632710338 -0.469087719917 -0.0179432816803 rpy=-0.00241979620112 -0.000645910391875 1.59131641167
