Commit message: added: geometry hierarchy

File: src/robots/custom_robots.urdf (robot description, URDF)
Before this commit: robot custom_robots, 21 links, 20 joints
Joints:
- joint indy0_joint_base_link: origin xyz=-0.487239867449 0.264511883259 0.0157464146614 rpy=-0.0032244007077 0.00715094916312 -1.57122883195 -> xyz=-0.487280130386 0.264434039593 0.0159286260605 rpy=-0.00391547901269 0.00688150026222 -1.57084273849
- joint panda1_joint_base_link: origin xyz=0.473158180714 0.192921757698 0.0181045532227 rpy=-0.000695425424269 0.00240603340554 -1.59131646607 -> xyz=0.473311543465 0.192847371101 0.0179858207703 rpy=-0.000611609590822 0.00249272852417 -1.5915967317

File: src/robots/custom_robots.urdf.xacro (robot description, xacro)
@@ -6,6 +6,6 @@
 <link name="base_link"/>
 <!-- BODY BEGIN -->
-<xacro:indy7 robot_id="0" xyz="-0.487239867449 0.264511883259 0.0157464146614" rpy="-0.0032244007077 0.00715094916312 -1.57122883195" connected_to="base_link"/>
-<xacro:panda robot_id="1" xyz="0.473158180714 0.192921757698 0.0181045532227" rpy="-0.000695425424269 0.00240603340554 -1.59131646607" connected_to="base_link"/>
+<xacro:indy7 robot_id="0" xyz="-0.487280130386 0.264434039593 0.0159286260605" rpy="-0.00391547901269 0.00688150026222 -1.57084273849" connected_to="base_link"/>
+<xacro:panda robot_id="1" xyz="0.473311543465 0.192847371101 0.0179858207703" rpy="-0.000611609590822 0.00249272852417 -1.5915967317" connected_to="base_link"/>
 <!-- BODY END -->
 </robot>

File: src/robots/custom_robots_indy0_panda1.urdf (robot description, URDF)
Before this commit: robot custom_robots, 22 links, 21 joints
Joints:
- joint panda1_joint_base_link: origin xyz=0.473158180714 0.192921757698 0.0181045532227 rpy=-0.000695425424269 0.00240603340554 -1.59131646607 -> xyz=0.473311543465 0.192847371101 0.0179858207703 rpy=-0.000611609590822 0.00249272852417 -1.5915967317
- joint stem_joint_base_link: origin xyz=0.264406949282 0.487396359444 -0.0122845303267 rpy=-0.00715234293124 -0.00322130770527 1.57122882316 -> xyz=0.264514774084 0.487343907356 -0.0122006293386 rpy=-0.00688168222307 -0.00391515981352 1.57084273775

File: src/robots/custom_robots_panda1_indy0.urdf (robot description, URDF)
Before this commit: robot custom_robots, 22 links, 21 joints
Joints:
- joint indy0_joint_base_link: origin xyz=-0.487239867449 0.264511883259 0.0157464146614 rpy=-0.0032244007077 0.00715094916312 -1.57122883195 -> xyz=-0.487280130386 0.264434039593 0.0159286260605 rpy=-0.00391547901269 0.00688150026222 -1.57084273849
- joint stem_joint_base_link: origin xyz=0.202632710338 -0.469087719917 -0.0179432816803 rpy=-0.00241979620112 -0.000645910391875 1.59131641167 -> xyz=0.202694237232 -0.469187378883 -0.0177675765008 rpy=-0.00250491005542 -0.000559631303214 1.59159666971
