Commit message: update panda collision

File: src/robots/hand.xacro (robot description, xacro)
@@ -16,7 +16,13 @@
       </visual>
       <collision>
-        <origin xyz="0 0 0.03" rpy="1.57079633 0 0"/>
+        <origin xyz="0.0 0.0 -0.01" rpy="0.  0.  0."/>
         <geometry>
-          <cylinder length="0.16" radius="0.045"/>
+          <cylinder length="0.04" radius="0.05"/>
+        </geometry>
+      </collision>
+      <collision>
+        <origin xyz="0 0 0.03" rpy="0 0 1.57079633"/>
+        <geometry>
+          <box size="0.22 0.06 0.075"/>
         </geometry>
       </collision>
@@ -24,14 +30,41 @@
         <origin xyz="0 0.07 -0.02" rpy="0 1.57079633 0"/>
         <geometry>
-          <cylinder length="0.055" radius="0.02"/>
+          <cylinder length="0.07" radius="0.02"/>
         </geometry>
       </collision>
       <collision>
-        <origin xyz="0 -0.07 -0.02" rpy="1.57079633 0 0"/>
+        <origin xyz="0 -0.08 -0.02" rpy="1.57079633 0 0"/>
         <geometry>
-          <cylinder length="0.05" radius="0.01"/>
+          <cylinder length="0.03" radius="0.01"/>
+        </geometry>
+      </collision>
+    <!-- left finger -->
+      <visual>
+        <origin xyz="0 0.04 0.0584" rpy="0 0 0"/>
+        <geometry>
+          <mesh filename="package://franka_description/meshes/visual/finger.dae"/>
+        </geometry>
+      </visual>
+      <collision>
+        <origin xyz="0 0.0535 0.0934" rpy="0 0 0"/>
+        <geometry>
+          <cylinder length="0.045" radius="0.018"/>
+        </geometry>
+      </collision>
+    <!-- right finger -->
+      <visual>
+        <origin xyz="0 -0.04 0.0584" rpy="0 0 ${pi}"/>
+        <geometry>
+          <mesh filename="package://franka_description/meshes/visual/finger.dae"/>
+        </geometry>
+      </visual>
+      <collision>
+        <origin xyz="0 -0.0535 0.0934" rpy="0 0 -3.14159265"/>
+        <geometry>
+          <cylinder length="0.045" radius="0.018"/>
         </geometry>
       </collision>
     </link>
+    <!--
     <link name="${ns}_leftfinger">
       <visual>
@@ -76,4 +109,5 @@
       <mimic joint="${ns}_finger_joint1" />
     </joint>
+    -->
   </xacro:macro>
 </robot>

File: src/robots/panda_arm.xacro (robot description, xacro)
@@ -16,7 +16,13 @@
       </visual>
       <collision>
-        <origin xyz="-0.03  0.    0.03" rpy="3.14159265 -1.37340077  3.14159265"/>
+        <origin xyz="-0.02  0.    0.1" rpy="0 0 0"/>
         <geometry>
-          <cylinder length="0.102" radius="0.1"/>
+          <cylinder length="0.035" radius="0.085"/>
+        </geometry>
+      </collision>
+      <collision>
+        <origin xyz="-0.04  0.    0.03" rpy="0 0 0"/>
+        <geometry>
+          <cylinder length="0.102" radius="0.12"/>
         </geometry>
       </collision>
@@ -35,7 +41,7 @@
       </visual>
       <collision>
-        <origin xyz=" 0.     -0.0275 -0.075" rpy=" -2.71183037 0 0"/>
+        <origin xyz=" 0   0 -0.13" rpy="0 0 0"/>
         <geometry>
-          <cylinder length="0.132" radius="0.11"/>
+          <cylinder length="0.17" radius="0.075"/>
         </geometry>
       </collision>
@@ -56,7 +62,7 @@
       </visual>
       <collision>
-        <origin xyz="  0.    -0.08   0.035" rpy="  1.98320677 -0.          0."/>
+        <origin xyz="  0.    0   0" rpy="  0 -0.          0."/>
         <geometry>
-          <cylinder length="0.175" radius="0.09"/>
+          <cylinder length="0.26" radius="0.075"/>
         </geometry>
       </collision>
@@ -77,7 +83,7 @@
       </visual>
       <collision>
-        <origin xyz="  0.04   0.027 -0.035" rpy=" 2.48451772 -0.7355124  -1.69290814"/>
+        <origin xyz=" 0   0 -0.13" rpy=" 0 0 0"/>
         <geometry>
-          <cylinder length="0.12" radius="0.09"/>
+          <cylinder length="0.25" radius="0.075"/>
         </geometry>
       </collision>
@@ -98,7 +104,7 @@
       </visual>
       <collision>
-        <origin xyz="-0.0555  0.058   0.027" rpy="-2.0064792  -0.71456939  1.05945848"/>
+        <origin xyz="0.0  0.0   0.0" rpy="0 0 0"/>
         <geometry>
-          <cylinder length="0.17" radius="0.08"/>
+          <cylinder length="0.23" radius="0.07"/>
         </geometry>
       </collision>
@@ -119,13 +125,19 @@
       </visual>
       <collision>
-        <origin xyz="0.      0.0315 -0.115" rpy="2.87423726 -0.          0. "/>
+        <origin xyz="0.0 0.0 -0.27" rpy="0 -0.          0. "/>
         <geometry>
-          <cylinder length="0.20" radius="0.08"/>
+          <cylinder length="0.22" radius="0.07"/>
         </geometry>
       </collision>
       <collision>
-        <origin xyz="0.      0.0315 0" rpy="0 1.57079633 1.57079633"/>
+        <origin xyz="0.      0.08 -0.13" rpy="0 0 0"/>
         <geometry>
-          <cylinder length="0.12" radius="0.06"/>
+          <cylinder length="0.18" radius="0.05"/>
+        </geometry>
+      </collision>
+      <collision>
+        <origin xyz="0.      0.037 0" rpy="0 1.57079633 1.57079633"/>
+        <geometry>
+          <cylinder length="0.20" radius="0.06"/>
         </geometry>
       </collision>
@@ -146,19 +158,7 @@
       </visual>
       <collision>
-        <origin xyz="0.035 0.    0." rpy="-0.         -1.57079633  0."/>
+        <origin xyz="0.09 0.005 0." rpy="1.57079633         0.  0."/>
         <geometry>
-          <cylinder length="0.09" radius="0.065"/>
-        </geometry>
-      </collision>
-      <collision>
-        <origin xyz="0.09 -0.01 0." rpy="1.57079633         0.  0."/>
-        <geometry>
-          <cylinder length="0.13" radius="0.05"/>
-        </geometry>
-      </collision>
-      <collision>
-        <origin xyz="0.085 0.05 0." rpy="0.2         1.57079633  0."/>
-        <geometry>
-          <cylinder length="0.08" radius="0.04"/>
+          <cylinder length="0.16" radius="0.05"/>
         </geometry>
       </collision>

Commit message: in progress - pipeline, GraspChecker

File: src/robots/hand.xacro (robot description, xacro)
@@ -16,7 +16,7 @@
       </visual>
       <collision>
-        <origin xyz="0.0 0.0 -0.01" rpy="0.  0.  0."/>
+        <origin xyz="0.0 0.0 -0.09" rpy="0.  0.  0."/>
         <geometry>
-          <cylinder length="0.04" radius="0.05"/>
+          <cylinder length="0.20" radius="0.05"/>
         </geometry>
       </collision>

File: src/robots/panda_arm.xacro (robot description, xacro)
@@ -136,10 +136,4 @@
         </geometry>
       </collision>
-      <collision>
-        <origin xyz="0.      0.037 0" rpy="0 1.57079633 1.57079633"/>
-        <geometry>
-          <cylinder length="0.20" radius="0.06"/>
-        </geometry>
-      </collision>
     </link>
     <joint name="${arm_id}_joint5" type="revolute">
@@ -158,7 +152,7 @@
       </visual>
       <collision>
-        <origin xyz="0.09 0.005 0." rpy="1.57079633         0.  0."/>
+        <origin xyz="0.   0 -0.037" rpy="0 0 0"/>
         <geometry>
-          <cylinder length="0.16" radius="0.05"/>
+          <cylinder length="0.20" radius="0.06"/>
         </geometry>
       </collision>

Commit message: RRT* tend to move through edge-collision. remove, use RRT & TangentBundle in planning instead.

File: src/robots/hand.xacro (robot description, xacro)
@@ -22,19 +22,19 @@
       </collision>
       <collision>
-        <origin xyz="0 0 0.03" rpy="0 0 1.57079633"/>
+        <origin xyz="0 0 0.03" rpy="0 0 0"/>
         <geometry>
-          <box size="0.22 0.06 0.075"/>
+          <box size="0.06 0.22 0.085"/>
         </geometry>
       </collision>
       <collision>
-        <origin xyz="0 0.07 -0.02" rpy="0 1.57079633 0"/>
+        <origin xyz="0 0.06 -0.03" rpy="0 0 0"/>
         <geometry>
-          <cylinder length="0.07" radius="0.02"/>
+          <box size="0.08 0.07 0.04"/>
         </geometry>
       </collision>
       <collision>
-        <origin xyz="0 -0.08 -0.02" rpy="1.57079633 0 0"/>
+        <origin xyz="0 -0.075 -0.022" rpy="0 0 0"/>
         <geometry>
-          <cylinder length="0.03" radius="0.01"/>
+          <box size="0.02 0.06 0.02"/>
         </geometry>
       </collision>
@@ -47,7 +47,7 @@
       </visual>
       <collision>
-        <origin xyz="0 0.0535 0.0934" rpy="0 0 0"/>
+        <origin xyz="0 0.0535 0.095" rpy="0 0 0"/>
         <geometry>
-          <cylinder length="0.045" radius="0.018"/>
+          <box size="0.04 0.04 0.05"/>
         </geometry>
       </collision>
@@ -60,7 +60,7 @@
       </visual>
       <collision>
-        <origin xyz="0 -0.0535 0.0934" rpy="0 0 -3.14159265"/>
+        <origin xyz="0 -0.0535 0.095" rpy="0 0 0"/>
         <geometry>
-          <cylinder length="0.045" radius="0.018"/>
+          <box size="0.04 0.04 0.05"/>
         </geometry>
       </collision>

Commit message: better colision checking

File: src/robots/hand.xacro (robot description, xacro)
@@ -47,7 +47,7 @@
       </visual>
       <collision>
-        <origin xyz="0 0.0535 0.095" rpy="0 0 0"/>
+        <origin xyz="0 0.05 0.095" rpy="0 0 0"/>
         <geometry>
-          <box size="0.04 0.04 0.05"/>
+          <box size="0.04 0.04 0.055"/>
         </geometry>
       </collision>
@@ -60,7 +60,7 @@
       </visual>
       <collision>
-        <origin xyz="0 -0.0535 0.095" rpy="0 0 0"/>
+        <origin xyz="0 -0.05 0.095" rpy="0 0 0"/>
         <geometry>
-          <box size="0.04 0.04 0.05"/>
+          <box size="0.04 0.04 0.055"/>
         </geometry>
       </collision>

Commit message: more finger collision margin, auto_stop disablable on plan execution

File: src/robots/hand.xacro (robot description, xacro)
@@ -47,7 +47,7 @@
       </visual>
       <collision>
-        <origin xyz="0 0.05 0.095" rpy="0 0 0"/>
+        <origin xyz="0 0.05 0.10" rpy="0 0 0"/>
         <geometry>
-          <box size="0.04 0.04 0.055"/>
+          <box size="0.06 0.04 0.055"/>
         </geometry>
       </collision>
@@ -60,7 +60,7 @@
       </visual>
       <collision>
-        <origin xyz="0 -0.05 0.095" rpy="0 0 0"/>
+        <origin xyz="0 -0.05 0.10" rpy="0 0 0"/>
         <geometry>
-          <box size="0.04 0.04 0.055"/>
+          <box size="0.06 0.04 0.055"/>
         </geometry>
       </collision>

Commit message: box object handle update / display action points when playing / finger size change

File: src/robots/hand.xacro (robot description, xacro)
@@ -47,7 +47,7 @@
       </visual>
       <collision>
-        <origin xyz="0 0.05 0.10" rpy="0 0 0"/>
+        <origin xyz="0 0.05 0.099" rpy="0 0 0"/>
         <geometry>
-          <box size="0.06 0.04 0.055"/>
+          <box size="0.048 0.04 0.052"/>
         </geometry>
       </collision>
@@ -60,7 +60,7 @@
       </visual>
       <collision>
-        <origin xyz="0 -0.05 0.10" rpy="0 0 0"/>
+        <origin xyz="0 -0.05 0.099" rpy="0 0 0"/>
         <geometry>
-          <box size="0.06 0.04 0.055"/>
+          <box size="0.048 0.04 0.052"/>
         </geometry>
       </collision>

Commit message: Demo finished, Panda boundary fix, floor marker added,

File: src/robots/hand.xacro (robot description, xacro)
@@ -47,7 +47,7 @@
       </visual>
       <collision>
-        <origin xyz="0 0.05 0.099" rpy="0 0 0"/>
+        <origin xyz="0 0.05 0.098" rpy="0 0 0"/>
         <geometry>
-          <box size="0.048 0.04 0.052"/>
+          <box size="0.045 0.04 0.052"/>
         </geometry>
       </collision>
@@ -60,7 +60,7 @@
       </visual>
       <collision>
-        <origin xyz="0 -0.05 0.099" rpy="0 0 0"/>
+        <origin xyz="0 -0.05 0.098" rpy="0 0 0"/>
         <geometry>
-          <box size="0.048 0.04 0.052"/>
+          <box size="0.045 0.04 0.052"/>
         </geometry>
       </collision>

File: src/robots/panda_arm.xacro (robot description, xacro)
@@ -24,5 +24,5 @@
         <origin xyz="-0.04  0.    0.03" rpy="0 0 0"/>
         <geometry>
-          <cylinder length="0.102" radius="0.12"/>
+          <cylinder length="0.102" radius="0.15"/>
         </geometry>
       </collision>
@@ -64,5 +64,5 @@
         <origin xyz="  0.    0   0" rpy="  0 -0.          0."/>
         <geometry>
-          <cylinder length="0.26" radius="0.075"/>
+          <cylinder length="0.3" radius="0.075"/>
         </geometry>
       </collision>
@@ -106,5 +106,5 @@
         <origin xyz="0.0  0.0   0.0" rpy="0 0 0"/>
         <geometry>
-          <cylinder length="0.23" radius="0.07"/>
+          <cylinder length="0.26" radius="0.07"/>
         </geometry>
       </collision>
@@ -125,13 +125,13 @@
       </visual>
       <collision>
-        <origin xyz="0.0 0.0 -0.27" rpy="0 -0.          0. "/>
+        <origin xyz="0.0 0.0 -0.26" rpy="0 -0.          0. "/>
         <geometry>
-          <cylinder length="0.22" radius="0.07"/>
+          <cylinder length="0.25" radius="0.07"/>
         </geometry>
       </collision>
       <collision>
-        <origin xyz="0.      0.08 -0.13" rpy="0 0 0"/>
+        <origin xyz="0.      0.09 -0.13" rpy="0 0 0"/>
         <geometry>
-          <cylinder length="0.18" radius="0.05"/>
+          <cylinder length="0.18" radius="0.07"/>
         </geometry>
       </collision>
@@ -154,5 +154,5 @@
         <origin xyz="0.   0 -0.037" rpy="0 0 0"/>
         <geometry>
-          <cylinder length="0.20" radius="0.06"/>
+          <cylinder length="0.22" radius="0.06"/>
         </geometry>
       </collision>
