Commit message: added: grasp-collision-filtering

File: src/robots/indy7.xacro (robot description, xacro)
@@ -148,7 +148,7 @@
 		</visual>
 		<collision>
-			<origin xyz="0 0 -0.038" rpy="0 0 0"/>
-			<geometry>
-				<cylinder length="0.25" radius="0.06"/>
+			<origin xyz="0 0 -0.048" rpy="0 0 0"/>
+			<geometry>
+				<cylinder length="0.24" radius="0.06"/>
 			</geometry>
 		</collision>
@@ -167,4 +167,10 @@
 			<material name="${indy_material}"/>
 		</visual>
+		<collision>
+			<origin xyz="0 0 0.04" rpy="0 0 0"/>
+			<geometry>
+				<box size="0.06 0.08 0.06"/>
+			</geometry>
+		</collision>
 		<collision>
 			<origin xyz="0.006 0.045 0.1" rpy="0 0 0"/>

Commit message: fix indy boundary

File: src/robots/indy7.xacro (robot description, xacro)
@@ -64,5 +64,5 @@
 			<origin xyz="-0.225 0 0.09" rpy="${PI/2} 0 -${PI/2}"/>
 			<geometry>
-				<cylinder length="0.450" radius="0.073"/>
+				<cylinder length="0.50" radius="0.073"/>
 			</geometry>
 		</collision>
@@ -70,5 +70,5 @@
 			<origin xyz="0 0 -0.01" rpy="0 0 0"/>
 			<geometry>
-				<cylinder length="0.2" radius="0.085"/>
+				<cylinder length="0.3" radius="0.085"/>
 			</geometry>
 		</collision>
@@ -90,5 +90,5 @@
 			<origin xyz="0 0 0.03" rpy="0 0 0"/>
 			<geometry>
-				<cylinder length="0.2" radius="0.065"/>
+				<cylinder length="0.25" radius="0.065"/>
 			</geometry>
 		</collision>
@@ -110,5 +110,5 @@
 			<origin xyz="0 0 -0.092" rpy="0 0 0"/>
 			<geometry>
-				<cylinder length="0.35" radius="0.06"/>
+				<cylinder length="0.4" radius="0.06"/>
 			</geometry>
 		</collision>
@@ -130,5 +130,5 @@
 			<origin xyz="-0 0 -0.0225" rpy="0 0 0"/>
 			<geometry>
-				<cylinder length="0.183" radius="0.055"/>
+				<cylinder length="0.23" radius="0.055"/>
 			</geometry>
 		</collision>
@@ -148,7 +148,7 @@
 		</visual>
 		<collision>
-			<origin xyz="0 0 -0.048" rpy="0 0 0"/>
-			<geometry>
-				<cylinder length="0.24" radius="0.06"/>
+			<origin xyz="0 0 -0.058" rpy="0 0 0"/>
+			<geometry>
+				<cylinder length="0.26" radius="0.06"/>
 			</geometry>
 		</collision>
@@ -176,5 +176,5 @@
 			<origin xyz="0.006 0.045 0.1" rpy="0 0 0"/>
 			<geometry>
-				<cylinder length="0.083" radius="0.015"/>
+				<cylinder length="0.113" radius="0.015"/>
 			</geometry>
 		</collision>
@@ -182,5 +182,5 @@
 			<origin xyz="-0.006  0.045  0.1" rpy="0 0 0"/>
 			<geometry>
-				<cylinder length="0.083" radius="0.015"/>
+				<cylinder length="0.113" radius="0.015"/>
 			</geometry>
 		</collision>
@@ -188,5 +188,5 @@
 			<origin xyz="0.006 -0.045  0.1" rpy="0 0 0"/>
 			<geometry>
-				<cylinder length="0.083" radius="0.015"/>
+				<cylinder length="0.113" radius="0.015"/>
 			</geometry>
 		</collision>
@@ -194,5 +194,5 @@
 			<origin xyz="-0.006 -0.045  0.1" rpy="0 0 0"/>
 			<geometry>
-				<cylinder length="0.083" radius="0.015"/>
+				<cylinder length="0.113" radius="0.015"/>
 			</geometry>
 		</collision>

Commit message: fix indy boundary

File: src/robots/indy7.xacro (robot description, xacro)
@@ -64,5 +64,5 @@
 			<origin xyz="-0.225 0 0.09" rpy="${PI/2} 0 -${PI/2}"/>
 			<geometry>
-				<cylinder length="0.450" radius="0.073"/>
+				<cylinder length="0.50" radius="0.073"/>
 			</geometry>
 		</collision>
@@ -70,5 +70,5 @@
 			<origin xyz="0 0 -0.01" rpy="0 0 0"/>
 			<geometry>
-				<cylinder length="0.2" radius="0.085"/>
+				<cylinder length="0.3" radius="0.085"/>
 			</geometry>
 		</collision>
@@ -90,5 +90,5 @@
 			<origin xyz="0 0 0.03" rpy="0 0 0"/>
 			<geometry>
-				<cylinder length="0.2" radius="0.065"/>
+				<cylinder length="0.25" radius="0.065"/>
 			</geometry>
 		</collision>
@@ -110,5 +110,5 @@
 			<origin xyz="0 0 -0.092" rpy="0 0 0"/>
 			<geometry>
-				<cylinder length="0.35" radius="0.06"/>
+				<cylinder length="0.4" radius="0.06"/>
 			</geometry>
 		</collision>
@@ -130,5 +130,5 @@
 			<origin xyz="-0 0 -0.0225" rpy="0 0 0"/>
 			<geometry>
-				<cylinder length="0.183" radius="0.055"/>
+				<cylinder length="0.23" radius="0.055"/>
 			</geometry>
 		</collision>
@@ -148,7 +148,7 @@
 		</visual>
 		<collision>
-			<origin xyz="0 0 -0.048" rpy="0 0 0"/>
-			<geometry>
-				<cylinder length="0.24" radius="0.06"/>
+			<origin xyz="0 0 -0.058" rpy="0 0 0"/>
+			<geometry>
+				<cylinder length="0.26" radius="0.06"/>
 			</geometry>
 		</collision>
@@ -176,5 +176,5 @@
 			<origin xyz="0.006 0.045 0.1" rpy="0 0 0"/>
 			<geometry>
-				<cylinder length="0.083" radius="0.015"/>
+				<cylinder length="0.095" radius="0.015"/>
 			</geometry>
 		</collision>
@@ -182,5 +182,5 @@
 			<origin xyz="-0.006  0.045  0.1" rpy="0 0 0"/>
 			<geometry>
-				<cylinder length="0.083" radius="0.015"/>
+				<cylinder length="0.095" radius="0.015"/>
 			</geometry>
 		</collision>
@@ -188,5 +188,5 @@
 			<origin xyz="0.006 -0.045  0.1" rpy="0 0 0"/>
 			<geometry>
-				<cylinder length="0.083" radius="0.015"/>
+				<cylinder length="0.095" radius="0.015"/>
 			</geometry>
 		</collision>
@@ -194,5 +194,5 @@
 			<origin xyz="-0.006 -0.045  0.1" rpy="0 0 0"/>
 			<geometry>
-				<cylinder length="0.083" radius="0.015"/>
+				<cylinder length="0.095" radius="0.015"/>
 			</geometry>
 		</collision>

Commit message: Demo prepared

File: src/robots/indy7.xacro (robot description, xacro)
@@ -160,41 +160,4 @@
 	</link>
 	<link name="indy${robot_id}_tcp">
-		<visual>
-			<origin xyz="0 0 0" rpy="0 0 1.570796"/>
-			<geometry>
-				<mesh filename="package://my_mesh/meshes/stl/indy_gripper_asm2_res.STL"/>
-			</geometry>
-			<material name="${indy_material}"/>
-		</visual>
-		<collision>
-			<origin xyz="0 0 0.04" rpy="0 0 0"/>
-			<geometry>
-				<box size="0.06 0.08 0.06"/>
-			</geometry>
-		</collision>
-		<collision>
-			<origin xyz="0.006 0.045 0.1" rpy="0 0 0"/>
-			<geometry>
-				<cylinder length="0.095" radius="0.015"/>
-			</geometry>
-		</collision>
-		<collision>
-			<origin xyz="-0.006  0.045  0.1" rpy="0 0 0"/>
-			<geometry>
-				<cylinder length="0.095" radius="0.015"/>
-			</geometry>
-		</collision>
-		<collision>
-			<origin xyz="0.006 -0.045  0.1" rpy="0 0 0"/>
-			<geometry>
-				<cylinder length="0.095" radius="0.015"/>
-			</geometry>
-		</collision>
-		<collision>
-			<origin xyz="-0.006 -0.045  0.1" rpy="0 0 0"/>
-			<geometry>
-				<cylinder length="0.095" radius="0.015"/>
-			</geometry>
-		</collision>
 	</link>
 	<joint name="indy${robot_id}_joint0" type="revolute">

Commit message: done-execution

File: src/robots/indy7.xacro (robot description, xacro)
@@ -160,4 +160,41 @@
 	</link>
 	<link name="indy${robot_id}_tcp">
+<!--		<visual>-->
+<!--			<origin xyz="0 0 0" rpy="0 0 1.570796"/>-->
+<!--			<geometry>-->
+<!--				<mesh filename="package://my_mesh/meshes/stl/indy_gripper_asm2_res.STL"/>-->
+<!--			</geometry>-->
+<!--			<material name="${indy_material}"/>-->
+<!--		</visual>-->
+<!--		<collision>-->
+<!--			<origin xyz="0 0 0.04" rpy="0 0 0"/>-->
+<!--			<geometry>-->
+<!--				<box size="0.06 0.08 0.06"/>-->
+<!--			</geometry>-->
+<!--		</collision>-->
+<!--		<collision>-->
+<!--			<origin xyz="0.006 0.045 0.1" rpy="0 0 0"/>-->
+<!--			<geometry>-->
+<!--				<cylinder length="0.095" radius="0.015"/>-->
+<!--			</geometry>-->
+<!--		</collision>-->
+<!--		<collision>-->
+<!--			<origin xyz="-0.006  0.045  0.1" rpy="0 0 0"/>-->
+<!--			<geometry>-->
+<!--				<cylinder length="0.095" radius="0.015"/>-->
+<!--			</geometry>-->
+<!--		</collision>-->
+<!--		<collision>-->
+<!--			<origin xyz="0.006 -0.045  0.1" rpy="0 0 0"/>-->
+<!--			<geometry>-->
+<!--				<cylinder length="0.095" radius="0.015"/>-->
+<!--			</geometry>-->
+<!--		</collision>-->
+<!--		<collision>-->
+<!--			<origin xyz="-0.006 -0.045  0.1" rpy="0 0 0"/>-->
+<!--			<geometry>-->
+<!--				<cylinder length="0.095" radius="0.015"/>-->
+<!--			</geometry>-->
+<!--		</collision>-->
 	</link>
 	<joint name="indy${robot_id}_joint0" type="revolute">

Commit message: converted pddl plan initially done - binder not translated

File: src/robots/indy7.xacro (robot description, xacro)
@@ -22,7 +22,7 @@
 		</visual>
 		<collision>
-			<origin xyz="-0.1   0.    0.03" rpy="-0.          1.57079633  0."/>
-			<geometry>
-				<cylinder length="0.2" radius="0.05"/>
+			<origin xyz="-0.1   0.  0.05" rpy="0.  0.  0."/>
+			<geometry>
+				<box size="0.14 0.1 0.1"/>
 			</geometry>
 		</collision>
@@ -42,5 +42,5 @@
 		</visual>
 		<collision>
-			<origin xyz="0 0 0.072" rpy="0 0 0"/>
+			<origin xyz="0 0 0.0725" rpy="0 0 0"/>
 			<geometry>
 				<cylinder length="0.3" radius="0.1"/>

File: src/robots/indy7gripper.xacro (robot description, xacro)
@@ -22,7 +22,7 @@
 		</visual>
 		<collision>
-			<origin xyz="-0.1   0.    0.03" rpy="-0.          1.57079633  0."/>
-			<geometry>
-				<cylinder length="0.2" radius="0.05"/>
+			<origin xyz="-0.1   0.  0.05" rpy="0.  0.  0."/>
+			<geometry>
+				<box size="0.14 0.1 0.1"/>
 			</geometry>
 		</collision>
@@ -42,5 +42,5 @@
 		</visual>
 		<collision>
-			<origin xyz="0 0 0.072" rpy="0 0 0"/>
+			<origin xyz="0 0 0.0725" rpy="0 0 0"/>
 			<geometry>
 				<cylinder length="0.3" radius="0.1"/>

Commit message: pair-wise all done

File: src/robots/indy7.xacro (robot description, xacro)
@@ -24,5 +24,5 @@
 			<origin xyz="-0.1   0.  0.05" rpy="0.  0.  0."/>
 			<geometry>
-				<box size="0.14 0.1 0.1"/>
+				<box size="0.14 0.1 0.08"/>
 			</geometry>
 		</collision>
@@ -42,5 +42,5 @@
 		</visual>
 		<collision>
-			<origin xyz="0 0 0.0725" rpy="0 0 0"/>
+			<origin xyz="0 0 0.0825" rpy="0 0 0"/>
 			<geometry>
 				<cylinder length="0.3" radius="0.1"/>

File: src/robots/indy7gripper.xacro (robot description, xacro)
@@ -24,5 +24,5 @@
 			<origin xyz="-0.1   0.  0.05" rpy="0.  0.  0."/>
 			<geometry>
-				<box size="0.14 0.1 0.1"/>
+				<box size="0.14 0.1 0.08"/>
 			</geometry>
 		</collision>
@@ -42,5 +42,5 @@
 		</visual>
 		<collision>
-			<origin xyz="0 0 0.0725" rpy="0 0 0"/>
+			<origin xyz="0 0 0.0825" rpy="0 0 0"/>
 			<geometry>
 				<cylinder length="0.3" radius="0.1"/>

File: src/robots/panda_arm.xacro (robot description, xacro)
@@ -22,13 +22,7 @@
       </collision>
       <collision>
-        <origin xyz="-0.04  0.    0.03" rpy="0 0 0"/>
+        <origin xyz="-0.04  0.    0.045" rpy="0 0 0"/>
         <geometry>
-          <cylinder length="0.102" radius="0.15"/>
-        </geometry>
-      </collision>
-      <collision>
-        <origin xyz="-0.05  0.    0.03" rpy=" 1.57079633 0 0"/>
-        <geometry>
-          <cylinder length="0.3" radius="0.05"/>
+          <cylinder length="0.07" radius="0.15"/>
         </geometry>
       </collision>

Commit message: panda data samplled

File: src/robots/indy7.xacro (robot description, xacro)
@@ -22,7 +22,7 @@
 		</visual>
 		<collision>
-			<origin xyz="-0.1   0.  0.05" rpy="0.  0.  0."/>
-			<geometry>
-				<box size="0.14 0.1 0.08"/>
+			<origin xyz="-0.1   0.    0.03" rpy="-0.          1.57079633  0."/>
+			<geometry>
+				<cylinder length="0.2" radius="0.05"/>
 			</geometry>
 		</collision>
@@ -42,5 +42,5 @@
 		</visual>
 		<collision>
-			<origin xyz="0 0 0.0825" rpy="0 0 0"/>
+			<origin xyz="0 0 0.072" rpy="0 0 0"/>
 			<geometry>
 				<cylinder length="0.3" radius="0.1"/>
@@ -160,41 +160,41 @@
 	</link>
 	<link name="indy${robot_id}_tcp">
-<!--		<visual>-->
-<!--			<origin xyz="0 0 0" rpy="0 0 1.570796"/>-->
-<!--			<geometry>-->
-<!--				<mesh filename="package://my_mesh/meshes/stl/indy_gripper_asm2_res.STL"/>-->
-<!--			</geometry>-->
-<!--			<material name="${indy_material}"/>-->
-<!--		</visual>-->
-<!--		<collision>-->
-<!--			<origin xyz="0 0 0.04" rpy="0 0 0"/>-->
-<!--			<geometry>-->
-<!--				<box size="0.06 0.08 0.06"/>-->
-<!--			</geometry>-->
-<!--		</collision>-->
-<!--		<collision>-->
-<!--			<origin xyz="0.006 0.045 0.1" rpy="0 0 0"/>-->
-<!--			<geometry>-->
-<!--				<cylinder length="0.095" radius="0.015"/>-->
-<!--			</geometry>-->
-<!--		</collision>-->
-<!--		<collision>-->
-<!--			<origin xyz="-0.006  0.045  0.1" rpy="0 0 0"/>-->
-<!--			<geometry>-->
-<!--				<cylinder length="0.095" radius="0.015"/>-->
-<!--			</geometry>-->
-<!--		</collision>-->
-<!--		<collision>-->
-<!--			<origin xyz="0.006 -0.045  0.1" rpy="0 0 0"/>-->
-<!--			<geometry>-->
-<!--				<cylinder length="0.095" radius="0.015"/>-->
-<!--			</geometry>-->
-<!--		</collision>-->
-<!--		<collision>-->
-<!--			<origin xyz="-0.006 -0.045  0.1" rpy="0 0 0"/>-->
-<!--			<geometry>-->
-<!--				<cylinder length="0.095" radius="0.015"/>-->
-<!--			</geometry>-->
-<!--		</collision>-->
+		<visual>
+			<origin xyz="0 0 0" rpy="0 0 1.570796"/>
+			<geometry>
+				<mesh filename="package://my_mesh/meshes/stl/indy_gripper_asm2_res.STL"/>
+			</geometry>
+			<material name="${indy_material}"/>
+		</visual>
+		<collision>
+			<origin xyz="0 0 0.04" rpy="0 0 0"/>
+			<geometry>
+				<box size="0.06 0.08 0.06"/>
+			</geometry>
+		</collision>
+		<collision>
+			<origin xyz="0.006 0.045 0.1" rpy="0 0 0"/>
+			<geometry>
+				<cylinder length="0.095" radius="0.015"/>
+			</geometry>
+		</collision>
+		<collision>
+			<origin xyz="-0.006  0.045  0.1" rpy="0 0 0"/>
+			<geometry>
+				<cylinder length="0.095" radius="0.015"/>
+			</geometry>
+		</collision>
+		<collision>
+			<origin xyz="0.006 -0.045  0.1" rpy="0 0 0"/>
+			<geometry>
+				<cylinder length="0.095" radius="0.015"/>
+			</geometry>
+		</collision>
+		<collision>
+			<origin xyz="-0.006 -0.045  0.1" rpy="0 0 0"/>
+			<geometry>
+				<cylinder length="0.095" radius="0.015"/>
+			</geometry>
+		</collision>
 	</link>
 	<joint name="indy${robot_id}_joint0" type="revolute">

File: src/robots/panda_arm.xacro (robot description, xacro)
@@ -22,7 +22,13 @@
       </collision>
       <collision>
-        <origin xyz="-0.04  0.    0.045" rpy="0 0 0"/>
+        <origin xyz="-0.04  0.    0.03" rpy="0 0 0"/>
         <geometry>
-          <cylinder length="0.07" radius="0.15"/>
+          <cylinder length="0.102" radius="0.12"/>
+        </geometry>
+      </collision>
+      <collision>
+        <origin xyz="-0.05  0.    0.03" rpy=" 1.57079633 0 0"/>
+        <geometry>
+          <cylinder length="0.3" radius="0.05"/>
         </geometry>
       </collision>
@@ -58,5 +64,5 @@
         <origin xyz="  0.    0   0" rpy="  0 -0.          0."/>
         <geometry>
-          <cylinder length="0.3" radius="0.075"/>
+          <cylinder length="0.26" radius="0.075"/>
         </geometry>
       </collision>
@@ -100,5 +106,5 @@
         <origin xyz="0.0  0.0   0.0" rpy="0 0 0"/>
         <geometry>
-          <cylinder length="0.26" radius="0.07"/>
+          <cylinder length="0.23" radius="0.07"/>
         </geometry>
       </collision>
@@ -119,13 +125,19 @@
       </visual>
       <collision>
-        <origin xyz="0.0 0.0 -0.26" rpy="0 -0.          0. "/>
+        <origin xyz="0.0 0.0 -0.27" rpy="0 -0.          0. "/>
         <geometry>
-          <cylinder length="0.25" radius="0.07"/>
+          <cylinder length="0.22" radius="0.07"/>
         </geometry>
       </collision>
       <collision>
-        <origin xyz="0.      0.09 -0.13" rpy="0 0 0"/>
+        <origin xyz="0.      0.08 -0.13" rpy="0 0 0"/>
         <geometry>
-          <cylinder length="0.18" radius="0.07"/>
+          <cylinder length="0.18" radius="0.05"/>
+        </geometry>
+      </collision>
+      <collision>
+        <origin xyz="0.      0.037 0" rpy="0 1.57079633 1.57079633"/>
+        <geometry>
+          <cylinder length="0.20" radius="0.06"/>
         </geometry>
       </collision>
@@ -146,7 +158,7 @@
       </visual>
       <collision>
-        <origin xyz="0.   0 -0.037" rpy="0 0 0"/>
+        <origin xyz="0.09 0.005 0." rpy="1.57079633         0.  0."/>
         <geometry>
-          <cylinder length="0.22" radius="0.06"/>
+          <cylinder length="0.16" radius="0.05"/>
         </geometry>
       </collision>

File: src/robots/panda_hand.xacro (robot description, xacro)
@@ -16,25 +16,25 @@
       </visual>
       <collision>
-        <origin xyz="0.0 0.0 -0.09" rpy="0.  0.  0."/>
+        <origin xyz="0.0 0.0 -0.01" rpy="0.  0.  0."/>
         <geometry>
-          <cylinder length="0.20" radius="0.05"/>
+          <cylinder length="0.04" radius="0.05"/>
         </geometry>
       </collision>
       <collision>
-        <origin xyz="0 0 0.03" rpy="0 0 0"/>
+        <origin xyz="0 0 0.03" rpy="0 0 1.57079633"/>
         <geometry>
-          <box size="0.06 0.22 0.085"/>
+          <box size="0.22 0.06 0.075"/>
         </geometry>
       </collision>
       <collision>
-        <origin xyz="0 0.06 -0.03" rpy="0 0 0"/>
+        <origin xyz="0 0.07 -0.02" rpy="0 1.57079633 0"/>
         <geometry>
-          <box size="0.08 0.07 0.04"/>
+          <cylinder length="0.07" radius="0.02"/>
         </geometry>
       </collision>
       <collision>
-        <origin xyz="0 -0.075 -0.022" rpy="0 0 0"/>
+        <origin xyz="0 -0.08 -0.02" rpy="1.57079633 0 0"/>
         <geometry>
-          <box size="0.02 0.06 0.02"/>
+          <cylinder length="0.03" radius="0.01"/>
         </geometry>
       </collision>
@@ -47,7 +47,7 @@
       </visual>
       <collision>
-        <origin xyz="0 0.05 0.098" rpy="0 0 0"/>
+        <origin xyz="0 0.0535 0.0934" rpy="0 0 0"/>
         <geometry>
-          <box size="0.045 0.04 0.052"/>
+          <cylinder length="0.045" radius="0.018"/>
         </geometry>
       </collision>
@@ -60,7 +60,7 @@
       </visual>
       <collision>
-        <origin xyz="0 -0.05 0.098" rpy="0 0 0"/>
+        <origin xyz="0 -0.0535 0.0934" rpy="0 0 -3.14159265"/>
         <geometry>
-          <box size="0.045 0.04 0.052"/>
+          <cylinder length="0.045" radius="0.018"/>
         </geometry>
       </collision>

Commit message: mesh adjusted

File: src/robots/indy7.xacro (robot description, xacro)
@@ -22,7 +22,7 @@
 		</visual>
 		<collision>
-			<origin xyz="-0.1   0.    0.03" rpy="-0.          1.57079633  0."/>
-			<geometry>
-				<cylinder length="0.2" radius="0.05"/>
+			<origin xyz="-0.1   0.  0.05" rpy="0.  0.  0."/>
+			<geometry>
+				<box size="0.14 0.1 0.08"/>
 			</geometry>
 		</collision>
@@ -42,5 +42,5 @@
 		</visual>
 		<collision>
-			<origin xyz="0 0 0.072" rpy="0 0 0"/>
+			<origin xyz="0 0 0.0825" rpy="0 0 0"/>
 			<geometry>
 				<cylinder length="0.3" radius="0.1"/>

File: src/robots/panda_arm.xacro (robot description, xacro)
@@ -22,13 +22,13 @@
       </collision>
       <collision>
-        <origin xyz="-0.04  0.    0.03" rpy="0 0 0"/>
+        <origin xyz="-0.04  0.    0.05" rpy="0 0 0"/>
         <geometry>
-          <cylinder length="0.102" radius="0.12"/>
+          <cylinder length="0.08" radius="0.12"/>
         </geometry>
       </collision>
       <collision>
-        <origin xyz="-0.05  0.    0.03" rpy=" 1.57079633 0 0"/>
+        <origin xyz="-0.05  0.    0.05" rpy="0 0 0"/>
         <geometry>
-          <cylinder length="0.3" radius="0.05"/>
+          <box size="0.1 0.3 0.08"/>
         </geometry>
       </collision>
