Commit message: restore latest stable robot model

File: src/robots/indy7.xacro (robot description, xacro)
@@ -160,41 +160,41 @@
 	</link>
 	<link name="indy${robot_id}_tcp">
-		<visual>
-			<origin xyz="0 0 0" rpy="0 0 1.570796"/>
-			<geometry>
-				<mesh filename="package://my_mesh/meshes/stl/indy_gripper_asm2_res.STL"/>
-			</geometry>
-			<material name="${indy_material}"/>
-		</visual>
-		<collision>
-			<origin xyz="0 0 0.04" rpy="0 0 0"/>
-			<geometry>
-				<box size="0.06 0.08 0.06"/>
-			</geometry>
-		</collision>
-		<collision>
-			<origin xyz="0.006 0.045 0.1" rpy="0 0 0"/>
-			<geometry>
-				<cylinder length="0.095" radius="0.015"/>
-			</geometry>
-		</collision>
-		<collision>
-			<origin xyz="-0.006  0.045  0.1" rpy="0 0 0"/>
-			<geometry>
-				<cylinder length="0.095" radius="0.015"/>
-			</geometry>
-		</collision>
-		<collision>
-			<origin xyz="0.006 -0.045  0.1" rpy="0 0 0"/>
-			<geometry>
-				<cylinder length="0.095" radius="0.015"/>
-			</geometry>
-		</collision>
-		<collision>
-			<origin xyz="-0.006 -0.045  0.1" rpy="0 0 0"/>
-			<geometry>
-				<cylinder length="0.095" radius="0.015"/>
-			</geometry>
-		</collision>
+<!--		<visual>-->
+<!--			<origin xyz="0 0 0" rpy="0 0 1.570796"/>-->
+<!--			<geometry>-->
+<!--				<mesh filename="package://my_mesh/meshes/stl/indy_gripper_asm2_res.STL"/>-->
+<!--			</geometry>-->
+<!--			<material name="${indy_material}"/>-->
+<!--		</visual>-->
+<!--		<collision>-->
+<!--			<origin xyz="0 0 0.04" rpy="0 0 0"/>-->
+<!--			<geometry>-->
+<!--				<box size="0.06 0.08 0.06"/>-->
+<!--			</geometry>-->
+<!--		</collision>-->
+<!--		<collision>-->
+<!--			<origin xyz="0.006 0.045 0.1" rpy="0 0 0"/>-->
+<!--			<geometry>-->
+<!--				<cylinder length="0.095" radius="0.015"/>-->
+<!--			</geometry>-->
+<!--		</collision>-->
+<!--		<collision>-->
+<!--			<origin xyz="-0.006  0.045  0.1" rpy="0 0 0"/>-->
+<!--			<geometry>-->
+<!--				<cylinder length="0.095" radius="0.015"/>-->
+<!--			</geometry>-->
+<!--		</collision>-->
+<!--		<collision>-->
+<!--			<origin xyz="0.006 -0.045  0.1" rpy="0 0 0"/>-->
+<!--			<geometry>-->
+<!--				<cylinder length="0.095" radius="0.015"/>-->
+<!--			</geometry>-->
+<!--		</collision>-->
+<!--		<collision>-->
+<!--			<origin xyz="-0.006 -0.045  0.1" rpy="0 0 0"/>-->
+<!--			<geometry>-->
+<!--				<cylinder length="0.095" radius="0.015"/>-->
+<!--			</geometry>-->
+<!--		</collision>-->
 	</link>
 	<joint name="indy${robot_id}_joint0" type="revolute">

File: src/robots/panda_arm.xacro (robot description, xacro)
@@ -22,13 +22,7 @@
       </collision>
       <collision>
-        <origin xyz="-0.04  0.    0.05" rpy="0 0 0"/>
+        <origin xyz="-0.04  0.    0.045" rpy="0 0 0"/>
         <geometry>
-          <cylinder length="0.08" radius="0.12"/>
-        </geometry>
-      </collision>
-      <collision>
-        <origin xyz="-0.05  0.    0.05" rpy="0 0 0"/>
-        <geometry>
-          <box size="0.1 0.3 0.08"/>
+          <cylinder length="0.07" radius="0.15"/>
         </geometry>
       </collision>
@@ -64,5 +58,5 @@
         <origin xyz="  0.    0   0" rpy="  0 -0.          0."/>
         <geometry>
-          <cylinder length="0.26" radius="0.075"/>
+          <cylinder length="0.3" radius="0.075"/>
         </geometry>
       </collision>
@@ -106,5 +100,5 @@
         <origin xyz="0.0  0.0   0.0" rpy="0 0 0"/>
         <geometry>
-          <cylinder length="0.23" radius="0.07"/>
+          <cylinder length="0.26" radius="0.07"/>
         </geometry>
       </collision>
@@ -125,19 +119,13 @@
       </visual>
       <collision>
-        <origin xyz="0.0 0.0 -0.27" rpy="0 -0.          0. "/>
+        <origin xyz="0.0 0.0 -0.26" rpy="0 -0.          0. "/>
         <geometry>
-          <cylinder length="0.22" radius="0.07"/>
+          <cylinder length="0.25" radius="0.07"/>
         </geometry>
       </collision>
       <collision>
-        <origin xyz="0.      0.08 -0.13" rpy="0 0 0"/>
+        <origin xyz="0.      0.09 -0.13" rpy="0 0 0"/>
         <geometry>
-          <cylinder length="0.18" radius="0.05"/>
-        </geometry>
-      </collision>
-      <collision>
-        <origin xyz="0.      0.037 0" rpy="0 1.57079633 1.57079633"/>
-        <geometry>
-          <cylinder length="0.20" radius="0.06"/>
+          <cylinder length="0.18" radius="0.07"/>
         </geometry>
       </collision>
@@ -158,7 +146,7 @@
       </visual>
       <collision>
-        <origin xyz="0.09 0.005 0." rpy="1.57079633         0.  0."/>
+        <origin xyz="0.   0 -0.037" rpy="0 0 0"/>
         <geometry>
-          <cylinder length="0.16" radius="0.05"/>
+          <cylinder length="0.22" radius="0.06"/>
         </geometry>
       </collision>

File: src/robots/panda_hand.xacro (robot description, xacro)
@@ -16,25 +16,25 @@
       </visual>
       <collision>
-        <origin xyz="0.0 0.0 -0.01" rpy="0.  0.  0."/>
+        <origin xyz="0.0 0.0 -0.09" rpy="0.  0.  0."/>
         <geometry>
-          <cylinder length="0.04" radius="0.05"/>
+          <cylinder length="0.20" radius="0.05"/>
         </geometry>
       </collision>
       <collision>
-        <origin xyz="0 0 0.03" rpy="0 0 1.57079633"/>
+        <origin xyz="0 0 0.03" rpy="0 0 0"/>
         <geometry>
-          <box size="0.22 0.06 0.075"/>
+          <box size="0.06 0.22 0.085"/>
         </geometry>
       </collision>
       <collision>
-        <origin xyz="0 0.07 -0.02" rpy="0 1.57079633 0"/>
+        <origin xyz="0 0.06 -0.03" rpy="0 0 0"/>
         <geometry>
-          <cylinder length="0.07" radius="0.02"/>
+          <box size="0.08 0.07 0.04"/>
         </geometry>
       </collision>
       <collision>
-        <origin xyz="0 -0.08 -0.02" rpy="1.57079633 0 0"/>
+        <origin xyz="0 -0.075 -0.022" rpy="0 0 0"/>
         <geometry>
-          <cylinder length="0.03" radius="0.01"/>
+          <box size="0.02 0.06 0.02"/>
         </geometry>
       </collision>
@@ -47,7 +47,7 @@
       </visual>
       <collision>
-        <origin xyz="0 0.0535 0.0934" rpy="0 0 0"/>
+        <origin xyz="0 0.05 0.098" rpy="0 0 0"/>
         <geometry>
-          <cylinder length="0.045" radius="0.018"/>
+          <box size="0.045 0.04 0.052"/>
         </geometry>
       </collision>
@@ -60,7 +60,7 @@
       </visual>
       <collision>
-        <origin xyz="0 -0.0535 0.0934" rpy="0 0 -3.14159265"/>
+        <origin xyz="0 -0.05 0.098" rpy="0 0 0"/>
         <geometry>
-          <cylinder length="0.045" radius="0.018"/>
+          <box size="0.045 0.04 0.052"/>
         </geometry>
       </collision>

Commit message: px150 initial commit

File: src/robots/indy7.xacro (robot description, xacro)
@@ -1,5 +1,5 @@
 <?xml version="1.0" ?>
 <robot name="indy7" xmlns:xacro="http://ros.org/wiki/xacro">
-  <xacro:macro name="indy7" params="robot_id:='indy7' description_pkg:='indy7_description' connected_to:='' xyz:='0 0 0' rpy:='0 0 0'">
+  <xacro:macro name="indy7" params="robot_id:='0' description_pkg:='indy7_description' connected_to:='' xyz:='0 0 0' rpy:='0 0 0'">
     <xacro:unless value="${not connected_to}">
       <joint name="indy${robot_id}_joint_${connected_to}" type="fixed">
