Commit message: round panda fingertip, narrower tool width

File: src/robots/panda_hand.xacro (robot description, xacro)
@@ -47,7 +47,13 @@
       </visual>
       <collision>
-        <origin xyz="0 0.05 0.098" rpy="0 0 0"/>
+        <origin xyz="0 0.05 0.082" rpy="0 0 0"/>
         <geometry>
-          <box size="0.045 0.04 0.052"/>
+          <box size="0.045 0.04 0.02"/>
+        </geometry>
+      </collision>
+      <collision>
+        <origin xyz="0 0.05 0.102" rpy="1.5707 0 0"/>
+        <geometry>
+          <cylinder length="0.04" radius="0.022"/>
         </geometry>
       </collision>
@@ -60,7 +66,13 @@
       </visual>
       <collision>
-        <origin xyz="0 -0.05 0.098" rpy="0 0 0"/>
+        <origin xyz="0 -0.05 0.082" rpy="0 0 0"/>
         <geometry>
-          <box size="0.045 0.04 0.052"/>
+          <box size="0.045 0.04 0.02"/>
+        </geometry>
+      </collision>
+      <collision>
+        <origin xyz="0 -0.05 0.102" rpy="1.5707 0 0"/>
+        <geometry>
+          <cylinder length="0.04" radius="0.022"/>
         </geometry>
       </collision>

Commit message: add IK_NUM, plot grouped bar, panda test scripts

File: src/robots/panda_hand.xacro (robot description, xacro)
@@ -22,7 +22,7 @@
       </collision>
       <collision>
-        <origin xyz="0 0 0.03" rpy="0 0 0"/>
+        <origin xyz="0 0 0.028" rpy="0 0 0"/>
         <geometry>
-          <box size="0.06 0.22 0.085"/>
+          <box size="0.05 0.22 0.08"/>
         </geometry>
       </collision>
