Commit message: tool adjusted

File: src/robots/indy7kiro.xacro (robot description, xacro)
@@ -10,4 +10,5 @@
     </xacro:unless>
 	<xacro:property name="PI" value="3.1415926535897931"/>
+	<xacro:property name="Z_OFF" value="0.032"/>
 	<xacro:property name="indy_material" value="metal_white"/>
 	<xacro:property name="tool_material" value="red"/>
@@ -148,5 +149,5 @@
 		</visual>
 		<visual>
-			<origin xyz="0 0 0.06" rpy="0 0 0"/>
+			<origin xyz="0 0 ${0.06+Z_OFF}" rpy="0 0 0"/>
 			<geometry>
 				<mesh filename="package://my_mesh/meshes/stl/kiro_indytool_link_res.stl"/>
@@ -154,12 +155,19 @@
 			<material name="${indy_material}"/>
 		</visual>
-		<collision>
-			<origin xyz="0 0 -0.058" rpy="0 0 0"/>
-			<geometry>
-				<cylinder length="0.26" radius="0.06"/>
-			</geometry>
-		</collision>
-		<collision>
-			<origin xyz="0.09 0 0.17" rpy="0 ${PI/4} 0"/>
+		<visual>
+			<origin xyz="0 0 ${0.06+Z_OFF/2+0.0005}" rpy="0 0 0"/>
+			<geometry>
+				<cylinder length="${Z_OFF-0.0015}" radius="0.045"/>
+			</geometry>
+			<material name="${indy_material}"/>
+		</visual>
+		<collision>
+			<origin xyz="0 0 ${-0.058+Z_OFF/2}" rpy="0 0 0"/>
+			<geometry>
+				<cylinder length="${0.26+Z_OFF}" radius="0.06"/>
+			</geometry>
+		</collision>
+		<collision>
+			<origin xyz="0.09 0 ${0.17+Z_OFF}" rpy="0 ${PI/4} 0"/>
 			<geometry>
 				<cylinder length="0.3" radius="0.05"/>
@@ -183,5 +191,5 @@
 			<origin xyz="-0.025 -0.0167 0.0" rpy="0 ${PI/2} 0"/>
 			<geometry>
-				<cylinder length="0.05" radius="0.05"/>
+				<cylinder length="0.05" radius="0.045"/>
 			</geometry>
 		</collision>
@@ -234,5 +242,5 @@
 		<parent link="indy${robot_id}_link6"/>
 		<child link="indy${robot_id}_link7"/>
-		<origin xyz="+0.19605 +0.00000000 +0.27855" rpy="-${PI/2} ${PI/4} -${PI}"/>
+		<origin xyz="+0.19605 +0.00000000 ${+0.27855+Z_OFF}" rpy="-${PI/2} ${PI/4} -${PI}"/>
 		<axis xyz="0 0 1"/>
 		<limit effort="10" velocity="1" lower="-${215*PI/180}" upper="${215*PI/180}"/>

Commit message: sweep setting done

File: src/robots/indy7kiro.xacro (robot description, xacro)
@@ -249,5 +249,5 @@
 		<parent link="indy${robot_id}_link7"/>
 		<child link="indy${robot_id}_tcp"/>
-		<origin xyz="-0.04975 -0.0167 0" rpy="0 0 0"/>
+		<origin xyz="-0.04975 -0.0167 0" rpy="-${PI/2} 0 -${PI/2}"/>
 	</joint>
   </xacro:macro>

File: src/robots/kmb.xacro (robot description, xacro)
@@ -31,7 +31,7 @@
 		</collision>
 		<collision>
-			<origin xyz="0.5   0  0.55" rpy="0.  0.  0."/>
+			<origin xyz="0.5   0  0.47" rpy="0.  0.  0."/>
 			<geometry>
-				<box size="0.10 0.7 0.23"/>
+				<box size="0.10 0.7 0.07"/>
 			</geometry>
 		</collision>
