Commit message: mobile mesh update

File: src/robots/kmb.xacro (robot description, xacro)
@@ -15,42 +15,20 @@
 	<link name="kmb${robot_id}_link_r">
 		<visual>
-			<origin xyz="0 0 0.220" rpy="0 0 0"/>
+			<origin xyz="0 0 0" rpy="0 0 0"/>
 			<geometry>
-				<box size="0.6 0.4 0.438"/>
+				<mesh filename="package://my_mesh/meshes/stl/mobile_ds_res.stl"/>
 			</geometry>
 			<material name="metal_white"/>
-		</visual>
-		<visual>
-			<origin xyz="0.2 0.16 0.10" rpy="1.570796326795 0 0"/>
-			<geometry>
-				<cylinder length="0.1" radius="0.1"/>
-			</geometry>
-			<material name="metal"/>
-		</visual>
-		<visual>
-			<origin xyz="0.2 -0.16 0.10" rpy="1.570796326795 0 0"/>
-			<geometry>
-				<cylinder length="0.1" radius="0.1"/>
-			</geometry>
-			<material name="metal"/>
-		</visual>
-		<visual>
-			<origin xyz="-0.2 0.16 0.10" rpy="1.570796326795 0 0"/>
-			<geometry>
-				<cylinder length="0.1" radius="0.1"/>
-			</geometry>
-			<material name="metal"/>
-		</visual>
-		<visual>
-			<origin xyz="-0.2 -0.16 0.10" rpy="1.570796326795 0 0"/>
-			<geometry>
-				<cylinder length="0.1" radius="0.1"/>
-			</geometry>
-			<material name="metal"/>
 		</visual>
 		<collision>
 			<origin xyz="0   0  0.220" rpy="0.  0.  0."/>
 			<geometry>
-				<box size="0.7 0.5 0.438"/>
+				<box size="1.0 0.75 0.438"/>
+			</geometry>
+		</collision>
+		<collision>
+			<origin xyz="-0.25   0  0.5" rpy="0.  0.  0."/>
+			<geometry>
+				<box size="0.5 0.75 0.2"/>
 			</geometry>
 		</collision>

Commit message: pddlstream mobile PnP debugged

File: src/robots/kmb.xacro (robot description, xacro)
@@ -56,5 +56,5 @@
 		<origin xyz="0 0 0" rpy="0 0 0"/>
 		<axis xyz="0 0 1"/>
-    	<limit effort="10000" velocity="1.5708"/>
+    	<limit effort="10000" lower="-10000" upper="10000" velocity="1.5708"/>
 	</joint>
 	<joint name="kmb${robot_id}_joint3" type="revolute">

Commit message: demo implementation to bed sweep

File: src/robots/kmb.xacro (robot description, xacro)
@@ -24,4 +24,16 @@
 			<material name="metal_white"/>
 		</visual>
+		<collision>
+			<origin xyz="0.335   0  0.55" rpy="0.  0.  0."/>
+			<geometry>
+				<cylinder length="0.03" radius="0.06"/>
+			</geometry>
+		</collision>
+		<collision>
+			<origin xyz="0.45   0  0.45" rpy="0.  0.  0."/>
+			<geometry>
+				<box size="0.1 0.75 0.1"/>
+			</geometry>
+		</collision>
 		<collision>
 			<origin xyz="0   0  0.220" rpy="0.  0.  0."/>

Commit message: exp1006 fin

File: src/robots/kmb.xacro (robot description, xacro)
@@ -31,7 +31,7 @@
 		</collision>
 		<collision>
-			<origin xyz="0.45   0  0.45" rpy="0.  0.  0."/>
+			<origin xyz="0.525   0  0.525" rpy="0.  0.  0."/>
 			<geometry>
-				<box size="0.1 0.75 0.1"/>
+				<box size="0.25 1.05 0.25"/>
 			</geometry>
 		</collision>
@@ -39,5 +39,5 @@
 			<origin xyz="0   0  0.220" rpy="0.  0.  0."/>
 			<geometry>
-				<box size="1.0 0.75 0.438"/>
+				<box size="1.3 1.05 0.438"/>
 			</geometry>
 		</collision>

Commit message: up-sweeping done

File: src/robots/kmb.xacro (robot description, xacro)
@@ -31,7 +31,7 @@
 		</collision>
 		<collision>
-			<origin xyz="0.525   0  0.525" rpy="0.  0.  0."/>
+			<origin xyz="0.45   0  0.45" rpy="0.  0.  0."/>
 			<geometry>
-				<box size="0.25 1.05 0.25"/>
+				<box size="0.1 0.75 0.1"/>
 			</geometry>
 		</collision>
@@ -39,5 +39,5 @@
 			<origin xyz="0   0  0.220" rpy="0.  0.  0."/>
 			<geometry>
-				<box size="1.3 1.05 0.438"/>
+				<box size="1.0 0.75 0.438"/>
 			</geometry>
 		</collision>

Commit message: exp1022 fin

File: src/robots/kmb.xacro (robot description, xacro)
@@ -30,10 +30,11 @@
 			</geometry>
 		</collision>
-		<collision>
-			<origin xyz="0.525   0  0.525" rpy="0.  0.  0."/>
+	<!--<collision>
+			<origin xyz="0.625   0  0.525" rpy="0.  0.  0."/>
 			<geometry>
-				<box size="0.25 1.05 0.25"/>
+				<box size="0.05 1.05 0.1"/>
 			</geometry>
 		</collision>
+	-->
 		<collision>
 			<origin xyz="0   0  0.220" rpy="0.  0.  0."/>

Commit message: new collect

File: src/robots/kmb.xacro (robot description, xacro)
@@ -30,21 +30,20 @@
 			</geometry>
 		</collision>
-	<!--<collision>
-			<origin xyz="0.625   0  0.525" rpy="0.  0.  0."/>
+		<collision>
+			<origin xyz="0.5   0  0.55" rpy="0.  0.  0."/>
 			<geometry>
-				<box size="0.05 1.05 0.1"/>
+				<box size="0.10 0.9 0.23"/>
 			</geometry>
 		</collision>
-	-->
 		<collision>
 			<origin xyz="0   0  0.220" rpy="0.  0.  0."/>
 			<geometry>
-				<box size="1.3 1.05 0.438"/>
+				<box size="1.1 0.9 0.438"/>
 			</geometry>
 		</collision>
 		<collision>
-			<origin xyz="-0.25   0  0.5" rpy="0.  0.  0."/>
+			<origin xyz="-0.3   0  0.5" rpy="0.  0.  0."/>
 			<geometry>
-				<box size="0.5 0.75 0.2"/>
+				<box size="0.5 0.9 0.2"/>
 			</geometry>
 		</collision>

Commit message: exp 1027 fin

File: src/robots/kmb.xacro (robot description, xacro)
@@ -33,5 +33,5 @@
 			<origin xyz="0.5   0  0.55" rpy="0.  0.  0."/>
 			<geometry>
-				<box size="0.10 0.9 0.23"/>
+				<box size="0.10 0.7 0.23"/>
 			</geometry>
 		</collision>
@@ -39,5 +39,5 @@
 			<origin xyz="0   0  0.220" rpy="0.  0.  0."/>
 			<geometry>
-				<box size="1.1 0.9 0.438"/>
+				<box size="1.1 0.7 0.438"/>
 			</geometry>
 		</collision>
@@ -45,5 +45,5 @@
 			<origin xyz="-0.3   0  0.5" rpy="0.  0.  0."/>
 			<geometry>
-				<box size="0.5 0.9 0.2"/>
+				<box size="0.5 0.7 0.2"/>
 			</geometry>
 		</collision>

Commit message: mode switcher, etc

File: src/robots/kmb.xacro (robot description, xacro)
@@ -54,5 +54,5 @@
 		<origin xyz="0 0 0" rpy="0 0 0"/>
 		<axis xyz="1 0 0"/>
-    	<limit effort="10000" lower="-5" upper="5" velocity="1.0"/>
+    	<limit effort="10000" lower="-10" upper="10" velocity="1.0"/>
 	</joint>
 	<joint name="kmb${robot_id}_joint1" type="prismatic">
@@ -61,5 +61,5 @@
 		<origin xyz="0 0 0" rpy="0 0 0"/>
 		<axis xyz="0 1 0"/>
-    	<limit effort="10000" lower="-5" upper="5" velocity="1.0"/>
+    	<limit effort="10000" lower="-10" upper="10" velocity="1.0"/>
 	</joint>
 	<joint name="kmb${robot_id}_joint2" type="continuous">
@@ -68,5 +68,5 @@
 		<origin xyz="0 0 0" rpy="0 0 0"/>
 		<axis xyz="0 0 1"/>
-    	<limit effort="10000" lower="-10000" upper="10000" velocity="1.5708"/>
+    	<limit effort="10000" lower="-15.708" upper="15.708" velocity="1.5708"/>
 	</joint>
 	<joint name="kmb${robot_id}_joint3" type="revolute">

Commit message: sweep data collecting done

File: src/robots/kmb.xacro (robot description, xacro)
@@ -31,7 +31,7 @@
 		</collision>
 		<collision>
-			<origin xyz="0.5   0  0.47" rpy="0.  0.  0."/>
+			<origin xyz="0.5   0  0.50" rpy="0.  0.  0."/>
 			<geometry>
-				<box size="0.10 0.7 0.07"/>
+				<box size="0.10 0.7 0.13"/>
 			</geometry>
 		</collision>

Commit message: table and sofa model done

File: src/robots/kmb.xacro (robot description, xacro)
@@ -43,7 +43,7 @@
 		</collision>
 		<collision>
-			<origin xyz="-0.3   0  0.5" rpy="0.  0.  0."/>
+			<origin xyz="-0.3   0  0.45" rpy="0.  0.  0."/>
 			<geometry>
-				<box size="0.5 0.7 0.2"/>
+				<box size="0.5 0.7 0.1"/>
 			</geometry>
 		</collision>

Commit message: exp 1216 done

File: src/robots/kmb.xacro (robot description, xacro)
@@ -43,7 +43,19 @@
 		</collision>
 		<collision>
-			<origin xyz="-0.3   0  0.45" rpy="0.  0.  0."/>
+			<origin xyz="-0.3   0  0.55" rpy="0.  0.  0."/>
 			<geometry>
-				<box size="0.5 0.7 0.1"/>
+				<box size="0.5 0.7 0.2"/>
+			</geometry>
+		</collision>
+		<collision>
+			<origin xyz="0.05  0.3  0.55" rpy="0.  0.  0."/>
+			<geometry>
+				<box size="0.2 0.1 0.2"/>
+			</geometry>
+		</collision>
+		<collision>
+			<origin xyz="0.05  -0.3  0.55" rpy="0.  0.  0."/>
+			<geometry>
+				<box size="0.2 0.1 0.2"/>
 			</geometry>
 		</collision>

Commit message: exp 1220

File: src/robots/kmb.xacro (robot description, xacro)
@@ -60,4 +60,16 @@
 			</geometry>
 		</collision>
+		<collision>
+			<origin xyz="0.3  0.3  0.50" rpy="0.  0.  0."/>
+			<geometry>
+				<box size="0.3 0.1 0.1"/>
+			</geometry>
+		</collision>
+		<collision>
+			<origin xyz="0.3  -0.3  0.50" rpy="0.  0.  0."/>
+			<geometry>
+				<box size="0.3 0.1 0.1"/>
+			</geometry>
+		</collision>
 	</link>
 	<joint name="kmb${robot_id}_joint0" type="prismatic">

Commit message: add push script- basic hold and move

File: src/robots/kmb.xacro (robot description, xacro)
@@ -31,13 +31,25 @@
 		</collision>
 		<collision>
-			<origin xyz="0.5   0  0.50" rpy="0.  0.  0."/>
+			<origin xyz="0.5   0.3  0.28" rpy="0.  0.  0."/>
 			<geometry>
-				<box size="0.10 0.7 0.13"/>
+				<box size="0.10 0.1 0.56"/>
 			</geometry>
 		</collision>
 		<collision>
-			<origin xyz="0   0  0.220" rpy="0.  0.  0."/>
+			<origin xyz="0.5   -0.3  0.28" rpy="0.  0.  0."/>
 			<geometry>
-				<box size="1.1 0.7 0.438"/>
+				<box size="0.10 0.1 0.56"/>
+			</geometry>
+		</collision>
+		<collision>
+			<origin xyz="0.4   0.0  0.488" rpy="0.  0.  0."/>
+			<geometry>
+				<box size="0.10 0.5 0.1"/>
+			</geometry>
+		</collision>
+		<collision>
+			<origin xyz="-0.05   0  0.220" rpy="0.  0.  0."/>
+			<geometry>
+				<box size="1.0 0.7 0.438"/>
 			</geometry>
 		</collision>

Commit message: target reaching convergence checked

File: src/robots/kmb.xacro (robot description, xacro)
@@ -31,13 +31,13 @@
 		</collision>
 		<collision>
-			<origin xyz="0.5   0.3  0.28" rpy="0.  0.  0."/>
+			<origin xyz="0.4758   0.325  0.28" rpy="0.  0.  0."/>
 			<geometry>
-				<box size="0.10 0.1 0.56"/>
+				<box size="0.05 0.05 0.56"/>
 			</geometry>
 		</collision>
 		<collision>
-			<origin xyz="0.5   -0.3  0.28" rpy="0.  0.  0."/>
+			<origin xyz="0.475   -0.325  0.28" rpy="0.  0.  0."/>
 			<geometry>
-				<box size="0.10 0.1 0.56"/>
+				<box size="0.05 0.05 0.56"/>
 			</geometry>
 		</collision>
