Commit message: added: mobile dof

File: src/robots/custom_robots_src.urdf.xacro (robot description, xacro)
@@ -6,4 +6,5 @@
 <xacro:include filename="$(env RNB_PLANNING_DIR)/src/robots/indy7gripper.xacro"/>
 <xacro:include filename="$(env RNB_PLANNING_DIR)/src/robots/indy5dof.xacro"/>
+<xacro:include filename="$(env RNB_PLANNING_DIR)/src/robots/kmb.xacro"/>
 <link name="base_link"/>
 <!-- BODY BEGIN -->

File: src/robots/indy5dof.xacro (robot description, xacro)
@@ -10,5 +10,5 @@
     </xacro:unless>
 	<xacro:property name="PI" value="3.1415926535897931"/>
-	<xacro:property name="indy_material" value="metal_grey"/>
+	<xacro:property name="indy_material" value="metal_white"/>
 	<xacro:property name="tool_material" value="red"/>
 	<!-- <material name="grey"> <color rgba="0.5 0.5 0.5 1"/> </material> -->

File: src/robots/indy7.xacro (robot description, xacro)
@@ -10,5 +10,5 @@
     </xacro:unless>
 	<xacro:property name="PI" value="3.1415926535897931"/>
-	<xacro:property name="indy_material" value="metal_grey"/>
+	<xacro:property name="indy_material" value="metal_white"/>
 	<xacro:property name="tool_material" value="red"/>
 	<!-- <material name="grey"> <color rgba="0.5 0.5 0.5 1"/> </material> -->

File: src/robots/indy7gripper.xacro (robot description, xacro)
@@ -10,5 +10,5 @@
     </xacro:unless>
 	<xacro:property name="PI" value="3.1415926535897931"/>
-	<xacro:property name="indy_material" value="metal_grey"/>
+	<xacro:property name="indy_material" value="metal_white"/>
 	<xacro:property name="tool_material" value="red"/>
 	<!-- <material name="grey"> <color rgba="0.5 0.5 0.5 1"/> </material> -->

Commit message: 7dof added

File: src/robots/custom_robots_src.urdf.xacro (robot description, xacro)
@@ -7,4 +7,5 @@
 <xacro:include filename="$(env RNB_PLANNING_DIR)/src/robots/indy5dof.xacro"/>
 <xacro:include filename="$(env RNB_PLANNING_DIR)/src/robots/kmb.xacro"/>
+<xacro:include filename="$(env RNB_PLANNING_DIR)/src/robots/indy7kiro.xacro"/>
 <link name="base_link"/>
 <!-- BODY BEGIN -->

File: src/robots/indy7kiro.xacro (robot description, xacro)
@@ -1,5 +1,5 @@
 <?xml version="1.0" ?>
-<robot name="indy7gripper" xmlns:xacro="http://ros.org/wiki/xacro">
-  <xacro:macro name="indy7gripper" params="robot_id:='0' description_pkg:='indy7_description' connected_to:='' xyz:='0 0 0' rpy:='0 0 0'">
+<robot name="indy7kiro" xmlns:xacro="http://ros.org/wiki/xacro">
+  <xacro:macro name="indy7kiro" params="robot_id:='0' description_pkg:='indy7_description' connected_to:='' xyz:='0 0 0' rpy:='0 0 0'">
     <xacro:unless value="${not connected_to}">
       <joint name="indy${robot_id}_joint_${connected_to}" type="fixed">
@@ -147,8 +147,21 @@
 			<material name="${indy_material}"/>
 		</visual>
+		<visual>
+			<origin xyz="0 0 0.06" rpy="0 0 0"/>
+			<geometry>
+				<mesh filename="package://my_mesh/meshes/stl/kiro_indytool_link_res.stl"/>
+			</geometry>
+			<material name="${indy_material}"/>
+		</visual>
 		<collision>
 			<origin xyz="0 0 -0.058" rpy="0 0 0"/>
 			<geometry>
 				<cylinder length="0.26" radius="0.06"/>
+			</geometry>
+		</collision>
+		<collision>
+			<origin xyz="0.09 0 0.17" rpy="0 ${PI/4} 0"/>
+			<geometry>
+				<cylinder length="0.3" radius="0.05"/>
 			</geometry>
 		</collision>
@@ -159,42 +172,20 @@
 		</inertial>
 	</link>
+	<link name="indy${robot_id}_link7">
+		<visual>
+			<origin xyz="0 0 0" rpy="0 0 0"/>
+			<geometry>
+				<mesh filename="package://my_mesh/meshes/stl/kiro_indytool_mount_res.stl"/>
+			</geometry>
+			<material name="${indy_material}"/>
+		</visual>
+		<collision>
+			<origin xyz="-0.025 -0.0167 0.0" rpy="0 ${PI/2} 0"/>
+			<geometry>
+				<cylinder length="0.05" radius="0.05"/>
+			</geometry>
+		</collision>
+	</link>
 	<link name="indy${robot_id}_tcp">
-		<visual>
-			<origin xyz="0 0 0" rpy="0 0 1.570796"/>
-			<geometry>
-				<mesh filename="package://my_mesh/meshes/stl/indy_gripper_asm2_res.STL"/>
-			</geometry>
-			<material name="${indy_material}"/>
-		</visual>
-		<collision>
-			<origin xyz="0 0 0.04" rpy="0 0 0"/>
-			<geometry>
-				<box size="0.06 0.08 0.06"/>
-			</geometry>
-		</collision>
-		<collision>
-			<origin xyz="0.006 0.045 0.1" rpy="0 0 0"/>
-			<geometry>
-				<cylinder length="0.095" radius="0.015"/>
-			</geometry>
-		</collision>
-		<collision>
-			<origin xyz="-0.006  0.045  0.1" rpy="0 0 0"/>
-			<geometry>
-				<cylinder length="0.095" radius="0.015"/>
-			</geometry>
-		</collision>
-		<collision>
-			<origin xyz="0.006 -0.045  0.1" rpy="0 0 0"/>
-			<geometry>
-				<cylinder length="0.095" radius="0.015"/>
-			</geometry>
-		</collision>
-		<collision>
-			<origin xyz="-0.006 -0.045  0.1" rpy="0 0 0"/>
-			<geometry>
-				<cylinder length="0.095" radius="0.015"/>
-			</geometry>
-		</collision>
 	</link>
 	<joint name="indy${robot_id}_joint0" type="revolute">
@@ -240,8 +231,15 @@
 		<limit effort="10" velocity="1" lower="-${215*PI/180}" upper="${215*PI/180}"/>
 	</joint>
+	<joint name="indy${robot_id}_joint6" type="revolute">
+		<parent link="indy${robot_id}_link6"/>
+		<child link="indy${robot_id}_link7"/>
+		<origin xyz="+0.19605 +0.00000000 +0.27855" rpy="-${PI/2} ${PI/4} -${PI}"/>
+		<axis xyz="0 0 1"/>
+		<limit effort="10" velocity="1" lower="-${215*PI/180}" upper="${215*PI/180}"/>
+	</joint>
 	<joint name="indy${robot_id}_tcp" type="fixed">
-		<parent link="indy${robot_id}_link6"/>
+		<parent link="indy${robot_id}_link7"/>
 		<child link="indy${robot_id}_tcp"/>
-		<origin xyz="0 0 0.06" rpy="0 0 0"/>
+		<origin xyz="-0.04975 -0.0167 0" rpy="0 0 0"/>
 	</joint>
   </xacro:macro>

Commit message: apply panda, initial planning test

File: src/robots/custom_robots_src.urdf.xacro (robot description, xacro)
@@ -2,8 +2,10 @@
 <robot xmlns:xacro="http://www.ros.org/wiki/xacro" name="custom_robots">
 <xacro:include filename="$(find indy7_description)/urdf/materials.xacro"/>
+<xacro:include filename="$(env RNB_PLANNING_DIR)/src/robots/panda_arm.xacro"/>
 <xacro:include filename="$(env RNB_PLANNING_DIR)/src/robots/panda.xacro"/>
 <xacro:include filename="$(env RNB_PLANNING_DIR)/src/robots/indy7.xacro"/>
 <xacro:include filename="$(env RNB_PLANNING_DIR)/src/robots/indy7gripper.xacro"/>
 <xacro:include filename="$(env RNB_PLANNING_DIR)/src/robots/indy5dof.xacro"/>
+<xacro:include filename="$(env RNB_PLANNING_DIR)/src/robots/pmb.xacro"/>
 <xacro:include filename="$(env RNB_PLANNING_DIR)/src/robots/kmb.xacro"/>
 <xacro:include filename="$(env RNB_PLANNING_DIR)/src/robots/indy7kiro.xacro"/>

File: src/robots/panda_arm.xacro (robot description, xacro)
@@ -1,5 +1,9 @@
 <?xml version='1.0' encoding='utf-8'?>
 <robot xmlns:xacro="http://www.ros.org/wiki/xacro" name="panda">
-  <xacro:macro name="panda_arm" params="arm_id:='panda' description_pkg:='franka_description' connected_to:='' xyz:='0 0 0' rpy:='0 0 0'">
+  <xacro:macro name="panda_arm"
+               params="arm_id:='panda' robot_id:='' description_pkg:='franka_description' connected_to:='' xyz:='0 0 0' rpy:='0 0 0'">
+    <xacro:unless value="${robot_id == ''}">
+      <xacro:property name="arm_id" value="panda_arm${robot_id}" />
+    </xacro:unless>
     <xacro:unless value="${not connected_to}">
       <joint name="${arm_id}_joint_${connected_to}" type="fixed">

File: src/robots/pmb.xacro (robot description, xacro)
@@ -25,61 +25,43 @@
 		</visual>
 		<collision>
-			<origin xyz="0.335   0  0.55" rpy="0.  0.  0."/>
+			<origin xyz="-0.05   0.0  0.295" rpy="0.  0.  0."/>
 			<geometry>
-				<cylinder length="0.03" radius="0.06"/>
+				<box size="0.7 0.8 0.59"/>
 			</geometry>
 		</collision>
 		<collision>
-			<origin xyz="0.4758   0.325  0.28" rpy="0.  0.  0."/>
+			<origin xyz="-0.05   0.3  0.65" rpy="0.  0.  0."/>
 			<geometry>
-				<box size="0.05 0.05 0.56"/>
+				<box size="0.7 0.2 0.1"/>
 			</geometry>
 		</collision>
 		<collision>
-			<origin xyz="0.475   -0.325  0.28" rpy="0.  0.  0."/>
+			<origin xyz="-0.05   -0.3  0.65" rpy="0.  0.  0."/>
 			<geometry>
-				<box size="0.05 0.05 0.56"/>
+				<box size="0.7 0.2 0.1"/>
 			</geometry>
 		</collision>
 		<collision>
-			<origin xyz="0.4   0.0  0.488" rpy="0.  0.  0."/>
+			<origin xyz="-0.3   0.0  0.65" rpy="0.  0.  0."/>
 			<geometry>
-				<box size="0.10 0.5 0.1"/>
+				<box size="0.2 0.4 0.1"/>
 			</geometry>
 		</collision>
 		<collision>
-			<origin xyz="-0.05   0  0.220" rpy="0.  0.  0."/>
+			<origin xyz="0.25   0.0  0.65" rpy="0.  0.  0."/>
 			<geometry>
-				<box size="1.0 0.7 0.438"/>
+				<box size="0.1 0.4 0.1"/>
 			</geometry>
 		</collision>
 		<collision>
-			<origin xyz="-0.3   0  0.55" rpy="0.  0.  0."/>
+			<origin xyz="0.35  0.35  0.35" rpy="0.  0.  0."/>
 			<geometry>
-				<box size="0.5 0.7 0.2"/>
+				<box size="0.1 0.1 0.69"/>
 			</geometry>
 		</collision>
 		<collision>
-			<origin xyz="0.05  0.3  0.55" rpy="0.  0.  0."/>
+			<origin xyz="0.35  -0.35  0.35" rpy="0.  0.  0."/>
 			<geometry>
-				<box size="0.2 0.1 0.2"/>
-			</geometry>
-		</collision>
-		<collision>
-			<origin xyz="0.05  -0.3  0.55" rpy="0.  0.  0."/>
-			<geometry>
-				<box size="0.2 0.1 0.2"/>
-			</geometry>
-		</collision>
-		<collision>
-			<origin xyz="0.3  0.3  0.50" rpy="0.  0.  0."/>
-			<geometry>
-				<box size="0.3 0.1 0.1"/>
-			</geometry>
-		</collision>
-		<collision>
-			<origin xyz="0.3  -0.3  0.50" rpy="0.  0.  0."/>
-			<geometry>
-				<box size="0.3 0.1 0.1"/>
+				<box size="0.1 0.1 0.69"/>
 			</geometry>
 		</collision>
