Commit message: panda joint limit, collision boundary fix

File: src/robots/panda_arm.xacro (robot description, xacro)
@@ -148,5 +148,5 @@
         <origin xyz="0.   0 -0.037" rpy="0 0 0"/>
         <geometry>
-          <cylinder length="0.22" radius="0.06"/>
+          <cylinder length="0.22" radius="0.055"/>
         </geometry>
       </collision>

File: src/robots/panda_hand.xacro (robot description, xacro)
@@ -28,7 +28,7 @@
       </collision>
       <collision>
-        <origin xyz="0 0.06 -0.03" rpy="0 0 0"/>
+        <origin xyz="0 0.06 -0.028" rpy="0 0 0"/>
         <geometry>
-          <box size="0.08 0.07 0.04"/>
+          <box size="0.08 0.07 0.036"/>
         </geometry>
       </collision>

Commit message: add tool cam

File: src/robots/panda_arm.xacro (robot description, xacro)
@@ -179,5 +179,18 @@
       <limit effort="12" lower="-2.8973" upper="2.8973" velocity="2.6100"/>
     </joint>
-    <link name="${arm_id}_link8"/>
+    <link name="${arm_id}_link8">
+      <collision>
+        <origin xyz="0.0 0.0 -0.09" rpy="0.  0.  0."/>
+        <geometry>
+          <cylinder length="0.20" radius="0.05"/>
+        </geometry>
+      </collision>
+      <collision>
+        <origin xyz="0.042 0.042 -0.028" rpy="0 0 ${-pi/4}"/>
+        <geometry>
+          <box size="0.08 0.07 0.036"/>
+        </geometry>
+      </collision>
+    </link>
     <joint name="${arm_id}_joint8" type="fixed">
       <origin rpy="0 0 0" xyz="0 0 0.107"/>

File: src/robots/panda_hand.xacro (robot description, xacro)
@@ -16,19 +16,7 @@
       </visual>
       <collision>
-        <origin xyz="0.0 0.0 -0.09" rpy="0.  0.  0."/>
-        <geometry>
-          <cylinder length="0.20" radius="0.05"/>
-        </geometry>
-      </collision>
-      <collision>
         <origin xyz="0 0 0.028" rpy="0 0 0"/>
         <geometry>
           <box size="0.05 0.22 0.08"/>
-        </geometry>
-      </collision>
-      <collision>
-        <origin xyz="0 0.06 -0.028" rpy="0 0 0"/>
-        <geometry>
-          <box size="0.08 0.07 0.036"/>
         </geometry>
       </collision>
