Commit message: change mobile robot coordinates

File: src/robots/pmb.xacro (robot description, xacro)
@@ -18,5 +18,5 @@
 	<link name="pmb${robot_id}_platform">
 		<visual>
-			<origin xyz="0 0 0" rpy="0 0 0"/>
+			<origin xyz="-0.28 0 0" rpy="0 0 0"/>
 			<geometry>
 				<mesh filename="package://my_mesh/meshes/stl/rnb_mobile_res.stl"/>
@@ -25,5 +25,5 @@
 		</visual>
 		<collision>
-			<origin xyz="-0.05   0.0  0.295" rpy="0.  0.  0."/>
+			<origin xyz="-0.33   0.0  0.295" rpy="0.  0.  0."/>
 			<geometry>
 				<box size="0.7 0.8 0.59"/>
@@ -31,5 +31,5 @@
 		</collision>
 		<collision>
-			<origin xyz="-0.05   0.3  0.65" rpy="0.  0.  0."/>
+			<origin xyz="-0.33   0.3  0.65" rpy="0.  0.  0."/>
 			<geometry>
 				<box size="0.7 0.2 0.1"/>
@@ -37,5 +37,5 @@
 		</collision>
 		<collision>
-			<origin xyz="-0.05   -0.3  0.65" rpy="0.  0.  0."/>
+			<origin xyz="-0.33   -0.3  0.65" rpy="0.  0.  0."/>
 			<geometry>
 				<box size="0.7 0.2 0.1"/>
@@ -43,5 +43,5 @@
 		</collision>
 		<collision>
-			<origin xyz="-0.3   0.0  0.65" rpy="0.  0.  0."/>
+			<origin xyz="-0.58   0.0  0.65" rpy="0.  0.  0."/>
 			<geometry>
 				<box size="0.2 0.4 0.1"/>
@@ -49,5 +49,5 @@
 		</collision>
 		<collision>
-			<origin xyz="0.25   0.0  0.65" rpy="0.  0.  0."/>
+			<origin xyz="-0.03   0.0  0.65" rpy="0.  0.  0."/>
 			<geometry>
 				<box size="0.1 0.4 0.1"/>
@@ -55,5 +55,5 @@
 		</collision>
 		<collision>
-			<origin xyz="0.35  0.35  0.35" rpy="0.  0.  0."/>
+			<origin xyz="0.07  0.35  0.35" rpy="0.  0.  0."/>
 			<geometry>
 				<box size="0.1 0.1 0.69"/>
@@ -61,5 +61,5 @@
 		</collision>
 		<collision>
-			<origin xyz="0.35  -0.35  0.35" rpy="0.  0.  0."/>
+			<origin xyz="0.07  -0.35  0.35" rpy="0.  0.  0."/>
 			<geometry>
 				<box size="0.1 0.1 0.69"/>

Commit message: exp 0209 / add micp inlier thresh

File: src/robots/pmb.xacro (robot description, xacro)
@@ -49,7 +49,7 @@
 		</collision>
 		<collision>
-			<origin xyz="-0.03   0.0  0.65" rpy="0.  0.  0."/>
+			<origin xyz="0.02   0.0  0.65" rpy="0.  0.  0."/>
 			<geometry>
-				<box size="0.1 0.4 0.1"/>
+				<box size="0.2 0.6 0.1"/>
 			</geometry>
 		</collision>

Commit message: exp0210, planning well

File: src/robots/pmb.xacro (robot description, xacro)
@@ -31,37 +31,37 @@
 		</collision>
 		<collision>
-			<origin xyz="-0.33   0.3  0.65" rpy="0.  0.  0."/>
+			<origin xyz="-0.33   0.3  0.62" rpy="0.  0.  0."/>
 			<geometry>
-				<box size="0.7 0.2 0.1"/>
+				<box size="0.7 0.2 0.04"/>
 			</geometry>
 		</collision>
 		<collision>
-			<origin xyz="-0.33   -0.3  0.65" rpy="0.  0.  0."/>
+			<origin xyz="-0.33   -0.3  0.62" rpy="0.  0.  0."/>
 			<geometry>
-				<box size="0.7 0.2 0.1"/>
+				<box size="0.7 0.2 0.04"/>
 			</geometry>
 		</collision>
 		<collision>
-			<origin xyz="-0.58   0.0  0.65" rpy="0.  0.  0."/>
+			<origin xyz="-0.58   0.0  0.62" rpy="0.  0.  0."/>
 			<geometry>
-				<box size="0.2 0.4 0.1"/>
+				<box size="0.2 0.4 0.04"/>
 			</geometry>
 		</collision>
 		<collision>
-			<origin xyz="0.02   0.0  0.65" rpy="0.  0.  0."/>
+			<origin xyz="0.02   0.0  0.62" rpy="0.  0.  0."/>
 			<geometry>
-				<box size="0.2 0.6 0.1"/>
+				<box size="0.2 0.6 0.04"/>
 			</geometry>
 		</collision>
 		<collision>
-			<origin xyz="0.07  0.35  0.35" rpy="0.  0.  0."/>
+			<origin xyz="0.07  0.35  0.32" rpy="0.  0.  0."/>
 			<geometry>
-				<box size="0.1 0.1 0.69"/>
+				<box size="0.1 0.1 0.63"/>
 			</geometry>
 		</collision>
 		<collision>
-			<origin xyz="0.07  -0.35  0.35" rpy="0.  0.  0."/>
+			<origin xyz="0.07  -0.35  0.32" rpy="0.  0.  0."/>
 			<geometry>
-				<box size="0.1 0.1 0.69"/>
+				<box size="0.1 0.1 0.63"/>
 			</geometry>
 		</collision>
@@ -81,10 +81,10 @@
     	<limit effort="10000" lower="-10" upper="10" velocity="1.0"/>
 	</joint>
-	<joint name="pmb${robot_id}_joint2" type="continuous">
+	<joint name="pmb${robot_id}_joint2" type="revolute">
 		<parent link="pmb${robot_id}_link2"/>
 		<child link="pmb${robot_id}_link3"/>
 		<origin xyz="0 0 0" rpy="0 0 0"/>
 		<axis xyz="0 0 1"/>
-    	<limit effort="10000" lower="-15.708" upper="15.708" velocity="1.5708"/>
+    	<limit effort="10000" lower="-1.5" upper="1.5" velocity="1.5708"/>
 	</joint>
 	<joint name="pmb${robot_id}_joint3" type="revolute">

Commit message: 5 test done

File: src/robots/pmb.xacro (robot description, xacro)
@@ -55,13 +55,13 @@
 		</collision>
 		<collision>
-			<origin xyz="0.07  0.35  0.32" rpy="0.  0.  0."/>
+			<origin xyz="0.07  0.37  0.32" rpy="0.  0.  0."/>
 			<geometry>
-				<box size="0.1 0.1 0.63"/>
+				<box size="0.1 0.14 0.63"/>
 			</geometry>
 		</collision>
 		<collision>
-			<origin xyz="0.07  -0.35  0.32" rpy="0.  0.  0."/>
+			<origin xyz="0.07  -0.37  0.32" rpy="0.  0.  0."/>
 			<geometry>
-				<box size="0.1 0.1 0.63"/>
+				<box size="0.1 0.14 0.63"/>
 			</geometry>
 		</collision>

Commit message: exp finished

File: src/robots/pmb.xacro (robot description, xacro)
@@ -55,13 +55,13 @@
 		</collision>
 		<collision>
-			<origin xyz="0.07  0.37  0.32" rpy="0.  0.  0."/>
+			<origin xyz="0.02  0.365  0.32" rpy="0.  0.  0."/>
 			<geometry>
-				<box size="0.1 0.14 0.63"/>
+				<box size="0.2 0.13 0.63"/>
 			</geometry>
 		</collision>
 		<collision>
-			<origin xyz="0.07  -0.37  0.32" rpy="0.  0.  0."/>
+			<origin xyz="0.02  -0.365  0.32" rpy="0.  0.  0."/>
 			<geometry>
-				<box size="0.1 0.14 0.63"/>
+				<box size="0.2 0.13 0.63"/>
 			</geometry>
 		</collision>
