Commit message: mobile pnp planning done

File: lib/moveit_interface_py/test_assets/custom_robots.urdf (robot description, URDF)
Before this commit: robot custom_robots, 21 links, 20 joints
Links:
- removed link indy0_link0
- removed link indy0_link1
- removed link indy0_link2
- removed link indy0_link3
- removed link indy0_link4
- removed link indy0_link5
- removed link indy0_link6
- removed link indy0_tcp
- removed link panda1_hand
- removed link panda1_leftfinger
- removed link panda1_link0
- removed link panda1_link1
- removed link panda1_link2
- removed link panda1_link3
- removed link panda1_link4
- removed link panda1_link5
- removed link panda1_link6
- removed link panda1_link7
- removed link panda1_link8
- removed link panda1_rightfinger
- added link indy1_link0, mass 1.59306955; collision box size=0.14 0.1 0.08; visual mesh filename=package://indy7_description/meshes/stl/Indy7_0.stl
- added link indy1_link1, mass 11.8030102; collision cylinder length=0.3 radius=0.1; visual mesh filename=package://indy7_description/meshes/stl/Indy7_1.stl
- added link indy1_link2, mass 7.99292141; collision cylinder length=0.3 radius=0.085; collision cylinder length=0.5 radius=0.073
- added link indy1_link3, mass 2.99134127; collision cylinder length=0.25 radius=0.065; visual mesh filename=package://indy7_description/meshes/stl/Indy7_3.stl
- added link indy1_link4, mass 2.12317035; collision cylinder length=0.4 radius=0.06; visual mesh filename=package://indy7_description/meshes/stl/Indy7_4.stl
- added link indy1_link5, mass 2.28865091; collision cylinder length=0.23 radius=0.055; visual mesh filename=package://indy7_description/meshes/stl/Indy7_5.stl
- added link indy1_link6, mass 0.40083918; collision cylinder length=0.26 radius=0.06; visual mesh filename=package://indy7_description/meshes/stl/Indy7_6.stl
- added link indy1_tcp
- added link kmb0_link0
- added link kmb0_link1
- added link kmb0_link2
- added link kmb0_link3
- added link kmb0_link4
- added link kmb0_link5
- added link kmb0_platform; collision box size=0.5 0.75 0.2; collision box size=1.0 0.75 0.438
Joints:
- removed joint indy0_joint0
- removed joint indy0_joint1
- removed joint indy0_joint2
- removed joint indy0_joint3
- removed joint indy0_joint4
- removed joint indy0_joint5
- removed joint indy0_joint_base_link
- removed joint indy0_tcp
- removed joint panda1_finger_joint1
- removed joint panda1_finger_joint2
- removed joint panda1_hand_joint
- removed joint panda1_joint1
- removed joint panda1_joint2
- removed joint panda1_joint3
- removed joint panda1_joint4
- removed joint panda1_joint5
- removed joint panda1_joint6
- removed joint panda1_joint7
- removed joint panda1_joint8
- removed joint panda1_joint_base_link
- added joint indy1_joint0: type revolute, parent indy1_link0, child indy1_link1, origin xyz=0.0 0.0 0.0775 rpy=0.0 0.0 0.0, axis 0.0 0.0 1.0, limit lower=-2.09439510239 upper=2.09439510239 effort=0.7853981633974483 velocity=0.6544984694978736
- added joint indy1_joint1: type revolute, parent indy1_link1, child indy1_link2, origin xyz=0.0 -0.109 0.222 rpy=1.57079632679 1.57079632679 0.0, axis 0.0 0.0 1.0, limit lower=-1.57079632679 upper=1.57079632679 effort=0.7853981633974483 velocity=0.6544984694978736
- added joint indy1_joint2: type revolute, parent indy1_link2, child indy1_link3, origin xyz=-0.45 0.0 -0.0305 rpy=0.0 0.0 0.0, axis 0.0 0.0 1.0, limit lower=-3.05432619099 upper=3.05432619099 effort=0.7853981633974483 velocity=0.6544984694978736
- added joint indy1_joint3: type revolute, parent indy1_link3, child indy1_link4, origin xyz=-0.267 0.0 -0.075 rpy=-1.57079632679 0.0 1.57079632679, axis 0.0 0.0 1.0, limit lower=-3.05432619099 upper=3.05432619099 effort=0.7853981633974483 velocity=0.7853981633974483
- added joint indy1_joint4: type revolute, parent indy1_link4, child indy1_link5, origin xyz=0.0 -0.114 0.083 rpy=1.57079632679 1.57079632679 0.0, axis 0.0 0.0 1.0, limit lower=-3.05432619099 upper=3.05432619099 effort=0.7853981633974483 velocity=0.7853981633974483
- added joint indy1_joint5: type revolute, parent indy1_link5, child indy1_link6, origin xyz=-0.168 0.0 0.069 rpy=-1.57079632679 0.0 1.57079632679, axis 0.0 0.0 1.0, limit lower=-3.75245789179 upper=3.75245789179 effort=0.7853981633974483 velocity=0.7853981633974483
- added joint indy1_joint_kmb0_platform: type fixed, parent kmb0_platform, child indy1_link0, origin xyz=0.172 0.0 0.439 rpy=0.0 0.0 3.14159265359
- added joint indy1_tcp: type fixed, parent indy1_link6, child indy1_tcp, origin xyz=0.0 0.0 0.06 rpy=0.0 0.0 0.0
- added joint kmb0_joint0: type prismatic, parent kmb0_link0, child kmb0_link1, origin xyz=0.0 0.0 0.0 rpy=0.0 0.0 0.0, axis 1.0 0.0 0.0, limit lower=-5.0 upper=5.0 effort=10000.0 velocity=1.0
- added joint kmb0_joint1: type prismatic, parent kmb0_link1, child kmb0_link2, origin xyz=0.0 0.0 0.0 rpy=0.0 0.0 0.0, axis 0.0 1.0 0.0, limit lower=-5.0 upper=5.0 effort=10000.0 velocity=1.0
- added joint kmb0_joint2: type continuous, parent kmb0_link2, child kmb0_link3, origin xyz=0.0 0.0 0.0 rpy=0.0 0.0 0.0, axis 0.0 0.0 1.0, limit lower=0 upper=0 effort=10000.0 velocity=1.5708
- added joint kmb0_joint3: type revolute, parent kmb0_link3, child kmb0_link4, origin xyz=0.0 0.0 0.0 rpy=0.0 0.0 0.0, axis 1.0 0.0 0.0, limit lower=-0.001 upper=0.001 effort=0.0 velocity=0.0
- added joint kmb0_joint4: type revolute, parent kmb0_link4, child kmb0_link5, origin xyz=0.0 0.0 0.0 rpy=0.0 0.0 0.0, axis 0.0 1.0 0.0, limit lower=-0.001 upper=0.001 effort=0.0 velocity=0.0
- added joint kmb0_joint5: type prismatic, parent kmb0_link5, child kmb0_platform, origin xyz=0.0 0.0 0.0 rpy=0.0 0.0 0.0, axis 0.0 0.0 1.0, limit lower=-0.001 upper=0.001 effort=0.0 velocity=0.0
- added joint kmb0_joint_base_link: type fixed, parent base_link, child kmb0_link0, origin xyz=0.0 0.0 0.0 rpy=0.0 0.0 0.0

File: src/robots/kmb.xacro (robot description, xacro)
@@ -5,13 +5,16 @@
       <joint name="kmb${robot_id}_joint_${connected_to}" type="fixed">
         <parent link="${connected_to}"/>
-        <child link="kmb${robot_id}_link_0"/>
+        <child link="kmb${robot_id}_link0"/>
         <origin rpy="${rpy}" xyz="${xyz}"/>
       </joint>
     </xacro:unless>
 	<xacro:property name="PI" value="3.1415926535897931"/>
-	<link name="kmb${robot_id}_link_0"/>
-	<link name="kmb${robot_id}_link_x"/>
-	<link name="kmb${robot_id}_link_y"/>
-	<link name="kmb${robot_id}_link_r">
+	<link name="kmb${robot_id}_link0"/>
+	<link name="kmb${robot_id}_link1"/>
+	<link name="kmb${robot_id}_link2"/>
+	<link name="kmb${robot_id}_link3"/>
+	<link name="kmb${robot_id}_link4"/>
+	<link name="kmb${robot_id}_link5"/>
+	<link name="kmb${robot_id}_platform">
 		<visual>
 			<origin xyz="0 0 0" rpy="0 0 0"/>
@@ -35,6 +38,6 @@
 	</link>
 	<joint name="kmb${robot_id}_joint0" type="prismatic">
-		<parent link="kmb${robot_id}_link_0"/>
-		<child link="kmb${robot_id}_link_x"/>
+		<parent link="kmb${robot_id}_link0"/>
+		<child link="kmb${robot_id}_link1"/>
 		<origin xyz="0 0 0" rpy="0 0 0"/>
 		<axis xyz="1 0 0"/>
@@ -42,6 +45,6 @@
 	</joint>
 	<joint name="kmb${robot_id}_joint1" type="prismatic">
-		<parent link="kmb${robot_id}_link_x"/>
-		<child link="kmb${robot_id}_link_y"/>
+		<parent link="kmb${robot_id}_link1"/>
+		<child link="kmb${robot_id}_link2"/>
 		<origin xyz="0 0 0" rpy="0 0 0"/>
 		<axis xyz="0 1 0"/>
@@ -49,10 +52,31 @@
 	</joint>
 	<joint name="kmb${robot_id}_joint2" type="continuous">
-		<parent link="kmb${robot_id}_link_y"/>
-		<child link="kmb${robot_id}_link_r"/>
+		<parent link="kmb${robot_id}_link2"/>
+		<child link="kmb${robot_id}_link3"/>
 		<origin xyz="0 0 0" rpy="0 0 0"/>
 		<axis xyz="0 0 1"/>
     	<limit effort="10000" velocity="1.5708"/>
 	</joint>
+	<joint name="kmb${robot_id}_joint3" type="revolute">
+		<parent link="kmb${robot_id}_link3"/>
+		<child link="kmb${robot_id}_link4"/>
+		<origin xyz="0 0 0" rpy="0 0 0"/>
+		<axis xyz="1 0 0"/>
+    	<limit effort="0" lower="0" upper="0" velocity="0"/>
+	</joint>
+	<joint name="kmb${robot_id}_joint4" type="revolute">
+		<parent link="kmb${robot_id}_link4"/>
+		<child link="kmb${robot_id}_link5"/>
+		<origin xyz="0 0 0" rpy="0 0 0"/>
+		<axis xyz="0 1 0"/>
+    	<limit effort="0" lower="0" upper="0" velocity="0"/>
+	</joint>
+	<joint name="kmb${robot_id}_joint5" type="prismatic">
+		<parent link="kmb${robot_id}_link5"/>
+		<child link="kmb${robot_id}_platform"/>
+		<origin xyz="0 0 0" rpy="0 0 0"/>
+		<axis xyz="0 0 1"/>
+    	<limit effort="0" lower="0" upper="0" velocity="0.0"/>
+	</joint>
   </xacro:macro>
 </robot>
